File: boxpcb/Pro-Micro-v11.brd (EAGLE design)
At the start: 40 x 74 mm, 11 parts

Commit message: wip
Parts:
- added C5: 100uF, rcl:E3,5-8
- added C6, C7, C8, C9: 0.1uF, rcl:C025-024X044
- added EXT1, EXT2: (no value), con-phoenix-254:3POL254
- added JP2: (no value), microbuilder:1X08_OVAL
- added PWR: (no value), con-phoenix-254:2POL254
- added R1, R2, R3, R4, R5, R6: 47K, rcl:0204/5
- added S1: (no value), SparkFun-Electromechanical:TACTILE-PTH
- added U$5: EN11-VSM1AF20, rotary-encoder:EN11-VS*
- C1, C2, C3, C4: value (none) -> 0.1uF
Connections:
- new net RST: S1.3, S1.4
- net A3: now also C4.2
- net D10: now also JP2.6
- net D2: now also C6.2, R2.2, U$3.A
- net D3: now also C7.2, R1.2, U$3.B
- net D4: now also R3.1, U$3.E
- net D5: now also C8.2, R5.2, U$5.A
- net D6: now also C9.2, R4.2, U$5.B
- net D7: now also R6.1, U$5.E
- net D8: now also EXT1.2
- net D9: now also EXT2.2
- net GND: now also C4.1, C5.-, C6.1, C7.1, C8.1, C9.1, EXT1.3, EXT2.3, JP2.7, JP2.8, PWR.2, S1.1, S1.2, U$3.C, U$3.D, U$5.C, U$5.D
- net MISO: now also JP2.4
- net MOSI: now also JP2.5
- net SCK: now also JP2.3
- net VCC: now also C5.+, EXT1.1, EXT2.1, JP2.1, JP2.2, PWR.1, R1.1, R2.1, R3.2, R4.1, R5.1, R6.2

Commit message: before autorouter
Parts:
- added H1, H2, H3, H4: MOUNT-PAD-ROUND3.3, holes:3,3-PAD
- moved S1 220.2 mm to (10.7, 61.0)
- moved C7 211.6 mm to (26.7, 54.9), turned to 180 degrees
- moved C9 207.3 mm to (26.7, 39.4)
- moved C6 205.4 mm to (26.7, 52.3)
- moved C8 201.2 mm to (26.7, 36.8)
- moved JP2 189.3 mm to (21.1, 13.7), turned to 270 degrees
- moved R4 160.0 mm to (24.1, 29.2), turned to 90 degrees
- moved R3 158.1 mm to (23.1, 61.7), turned to 90 degrees
- moved R2 157.4 mm to (27.7, 61.7), turned to 270 degrees
- moved C5 156.4 mm to (11.9, 9.65), turned to 180 degrees
- moved R5 155.9 mm to (26.2, 29.2), turned to 90 degrees
- moved R1 153.2 mm to (25.4, 61.7), turned to 270 degrees
- moved EXT2 151.7 mm to (2.79, 19.1), turned to 90 degrees
- moved U$5 151.5 mm to (35.6, 35.6), turned to 90 degrees
- moved EXT1 149.4 mm to (2.79, 28.7), turned to 90 degrees
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Connections:
- removed net RST: S1.3, S1.4
- net RESET: now also S1.3, S1.4
Routing:
- net VCC: track 0.00 -> 65.2 mm
- net A1: track 0.00 -> 30.5 mm
- net D5: track 0.00 -> 19.1 mm
- net D7: track 0.00 -> 12.0 mm
- net D6: track 0.00 -> 11.2 mm
- added copper zone on layer 16, net GND
Other:
- board text removed: "3.3V Reg / 8MHz"
- board text removed: "5V Reg / 16MHz"
- board text removed: "Mark back accordingly"
- board text removed: "Valid combinations:"

Commit message: first ver routing
Parts:
- removed H1, H2, H3, H4: MOUNT-PAD-ROUND3.3, holes:3,3-PAD
- removed JP1: (no value), jumper:JP2W
- added A3: (no value), con-phoenix-254:3POL254
- moved C4 32.6 mm to (7.87, 36.3), turned to 90 degrees
- moved R4 15.3 mm to (25.1, 44.5), turned to 270 degrees
- moved R6 12.7 mm to (22.1, 41.9)
- moved JP2 11.3 mm to (26.4, 3.81), turned to 0 degrees
- moved JP6 9.07 mm to (19.6, 72.4)
- moved JP7 9.07 mm to (4.32, 44.5)
- moved R1 8.10 mm to (29.7, 68.6)
- moved R2 8.10 mm to (32.0, 68.6)
- moved R3 8.10 mm to (27.4, 68.6)
- moved S1 7.82 mm to (12.4, 68.6), flipped to the bottom, turned to 270 degrees
- moved C8 6.53 mm to (28.2, 30.5), turned to 90 degrees
- moved C6 6.10 mm to (26.4, 58.4)
- moved C7 6.10 mm to (26.4, 61.0), turned to 0 degrees
- moved C9 3.94 mm to (27.7, 43.2), turned to 270 degrees
- moved C1 3.82 mm to (27.2, 52.1)
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Connections:
- net A3: now also A3.2; no longer JP1.2
- net D2: now also C7.2, R1.2, U$3.B; no longer C6.2, R2.2, U$3.A
- net D3: now also C6.2, R2.2, U$3.A; no longer C7.2, R1.2, U$3.B
- net D5: now also C9.2, R4.2, U$5.B; no longer C8.2, R5.2, U$5.A
- net D6: now also R6.1, U$5.E; no longer C9.2, R4.2, U$5.B
- net D7: now also C8.2, R5.2, U$5.A; no longer R6.1, U$5.E
- net D8: now also EXT2.2; no longer EXT1.2
- net D9: now also EXT1.2; no longer EXT2.2
- net GND: now also A3.3; no longer JP1.3
- net VCC: now also A3.1; no longer JP1.1
Routing:
- net A2: track 0.00 -> 64.3 mm, vias 0 -> 2
- net D3: track 0.00 -> 63.2 mm, vias 0 -> 3
- net D4: track 0.00 -> 54.8 mm, vias 0 -> 3
- net D2: track 0.00 -> 52.1 mm, vias 0 -> 2
- net SCK: track 0.00 -> 51.4 mm
- net MISO: track 0.00 -> 49.5 mm
- net MOSI: track 0.00 -> 47.9 mm
- net D10: track 0.00 -> 45.1 mm
- net D7: track 12.0 -> 51.0 mm, vias 0 -> 2
- net A3: track 0.00 -> 37.2 mm, vias 0 -> 1
- net D8: track 0.00 -> 34.9 mm
- net D6: track 11.2 -> 42.8 mm, vias 0 -> 2
- net D5: track 19.1 -> 48.2 mm, vias 0 -> 2
- net VCC: track 65.2 -> 90.4 mm, vias 0 -> 2
- net D9: track 0.00 -> 19.2 mm
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- added copper zone on layer 1, net VCC

Commit message: wip
Parts:
- added H1, H2: MOUNT-HOLE3.0, holes:3,0
Routing:
- net D3: track 63.2 -> 57.1 mm
- net D2: track 52.1 -> 50.0 mm
Other:
- board text added: "BlinkyPants v1.0"
- board text added: "Eran Rundstein"
Changed lines of the file:
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@@
 <text x="4.699" y="65.405" size="0.8128" layer="21" ratio="15" rot="R90">J1</text>
 <wire x1="40" y1="0" x2="0" y2="0" width="0.2032" layer="20"/>
+<text x="17.526" y="13.97" size="1.778" layer="25" rot="R90">BlinkyPants v1.0</text>
+<text x="20.32" y="13.716" size="1.778" layer="25" rot="R90">Eran Rundstein</text>
 </plain>
 <attributes>
@@
 <attribute name="OC_FARNELL" value="unknown" x="4.572" y="37.592" size="1.778" layer="27" rot="R90" display="off"/>
 </element>
+<element name="H1" library="holes" package="3,0" value="MOUNT-HOLE3.0" x="3" y="3"/>
+<element name="H2" library="holes" package="3,0" value="MOUNT-HOLE3.0" x="37" y="71"/>
 </elements>
 <signals>
@@
 <wire x1="26.162" y1="27.432" x2="26.162" y2="26.67" width="0.3048" layer="1"/>
 <polygon width="0.3048" layer="1">
-<vertex x="0.508" y="73.406"/>
-<vertex x="39.116" y="73.406"/>
+<vertex x="0.508" y="73.66"/>
+<vertex x="39.37" y="73.66"/>
 <vertex x="39.116" y="1.27"/>
 <vertex x="0.508" y="1.27"/>
-<vertex x="0.508" y="73.152"/>
 </polygon>
 </signal>
@@
 <wire x1="36.81" y1="57.11" x2="37.552" y2="57.11" width="0.4064" layer="1"/>
 <wire x1="37.552" y1="57.11" x2="38.354" y2="57.912" width="0.4064" layer="1"/>
-<wire x1="38.354" y1="57.912" x2="38.354" y2="66.548" width="0.4064" layer="1"/>
-<wire x1="38.354" y1="66.548" x2="36.322" y2="68.58" width="0.4064" layer="1"/>
-<wire x1="36.322" y1="68.58" x2="32.258" y2="68.58" width="0.4064" layer="1"/>
-<wire x1="32.258" y1="68.58" x2="29.718" y2="66.04" width="0.4064" layer="1"/>
+<wire x1="38.354" y1="57.912" x2="38.354" y2="64.262" width="0.4064" layer="1"/>
 <wire x1="29.718" y1="66.04" x2="29.718" y2="62.992" width="0.4064" layer="1"/>
 <wire x1="29.718" y1="62.992" x2="27.686" y2="60.96" width="0.4064" layer="1"/>
@@
 <wire x1="24.13" y1="61.976" x2="26.67" y2="61.976" width="0.3048" layer="1"/>
 <wire x1="26.67" y1="61.976" x2="27.686" y2="60.96" width="0.3048" layer="1"/>
+<wire x1="32.512" y1="67.564" x2="31.242" y2="67.564" width="0.4064" layer="1"/>
+<wire x1="31.242" y1="67.564" x2="29.718" y2="66.04" width="0.4064" layer="1"/>
+<wire x1="38.354" y1="64.262" x2="37.338" y2="65.278" width="0.4064" layer="1"/>
+<wire x1="37.338" y1="65.278" x2="34.798" y2="65.278" width="0.4064" layer="1"/>
+<wire x1="34.798" y1="65.278" x2="32.512" y2="67.564" width="0.4064" layer="1"/>
 </signal>
 <signal name="D3">
@@
 <wire x1="36.81" y1="52.11" x2="38.394" y2="52.11" width="0.4064" layer="1"/>
 <wire x1="38.394" y1="52.11" x2="39.116" y2="52.832" width="0.4064" layer="1"/>
-<wire x1="39.116" y1="52.832" x2="39.116" y2="68.834" width="0.4064" layer="1"/>
-<wire x1="39.116" y1="68.834" x2="37.846" y2="70.104" width="0.4064" layer="1"/>
-<wire x1="37.846" y1="70.104" x2="35.052" y2="70.104" width="0.4064" layer="1"/>
-<wire x1="35.052" y1="70.104" x2="34.798" y2="69.85" width="0.4064" layer="1"/>
-<via x="34.798" y="69.85" extent="1-16" drill="0.6"/>
-<wire x1="34.798" y1="69.85" x2="34.798" y2="68.834" width="0.4064" layer="16"/>
-<wire x1="34.798" y1="68.834" x2="32.004" y2="66.04" width="0.4064" layer="16"/>
+<wire x1="39.116" y1="52.832" x2="39.116" y2="64.77" width="0.4064" layer="1"/>
 <wire x1="4.318" y1="59.69" x2="17.018" y2="59.69" width="0.3048" layer="1"/>
 <wire x1="17.018" y1="59.69" x2="18.288" y2="58.42" width="0.3048" layer="1"/>
@@
 <wire x1="24.638" y1="56.896" x2="26.162" y2="56.896" width="0.3048" layer="1"/>
 <wire x1="26.162" y1="56.896" x2="27.686" y2="58.42" width="0.3048" layer="1"/>
+<via x="37.592" y="66.294" extent="1-16" drill="0.6"/>
+<wire x1="37.592" y1="66.294" x2="39.116" y2="64.77" width="0.4064" layer="1"/>
+<wire x1="32.004" y1="66.04" x2="37.338" y2="66.04" width="0.4064" layer="16"/>
+<wire x1="37.338" y1="66.04" x2="37.592" y2="66.294" width="0.4064" layer="16"/>
 </signal>
 <signal name="D4">
