File: boxpcb/Pro-Micro-v11.sch (EAGLE design)
At the start: 11 parts

Commit message: wip
Parts:
- added C5: 100uF, rcl:CPOL-USE3.5-8
- added C6, C7, C8, C9: 0.1uF, rcl:C-EU025-024X044
- added EXT1, EXT2: (no value), con-phoenix-254:MPT3
- added JP2: (no value), microbuilder:HEADER-1X8
- added PWR: (no value), con-phoenix-254:MPT2
- added R1, R2, R3, R4, R5, R6: 47K, rcl:R-US_0204/5
- added S1: (no value), SparkFun-Electromechanical:TAC_SWITCHPTH
- added U$5: EN11-VSM1AF20, rotary-encoder:EN11
- C1, C2, C3, C4: value (none) -> 0.1uF
Connections:
- new net RST: S1.3, S1.4
- net A3: now also C4.2
- net D10: now also JP2.6
- net D2: now also C6.2, R2.2, U$3G$1.A
- net D3: now also C7.2, R1.2, U$3G$1.B
- net D4: now also R3.1, U$3SW.E
- net D5: now also C8.2, R5.2, U$5G$1.A
- net D6: now also C9.2, R4.2, U$5G$1.B
- net D7: now also R6.1, U$5SW.E
- net D8: now also EXT1-2.1
- net D9: now also EXT2-2.1
- net GND: now also C4.1, C5.-, C6.1, C7.1, C8.1, C9.1, EXT1-3.1, EXT2-3.1, JP2.7, JP2.8, PWR-2.1, S1.1, S1.2, U$3G$1.C, U$3SW.D, U$5G$1.C, U$5SW.D
- net MISO: now also JP2.4
- net MOSI: now also JP2.5
- net SCK: now also JP2.3
- net VCC: now also C5.+, EXT1-1.1, EXT2-1.1, JP2.1, JP2.2, PWR-1.1, R1.1, R2.1, R3.2, R4.1, R5.1, R6.2
Other:
- moved on the sheet: U$3SW

Commit message: before autorouter
Parts:
- added H1, H2, H3, H4: MOUNT-PAD-ROUND3.3, holes:MOUNT-PAD-ROUND3.3
Connections:
- removed net RST: S1.3, S1.4
- net RESET: now also S1.3, S1.4
Changed lines of the file:
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@@
 <part name="P+16" library="supply1" deviceset="VCC" device=""/>
 <part name="GND19" library="supply1" deviceset="GND" device=""/>
+<part name="H1" library="holes" deviceset="MOUNT-PAD-ROUND" device="3.3"/>
+<part name="H2" library="holes" deviceset="MOUNT-PAD-ROUND" device="3.3"/>
+<part name="H3" library="holes" deviceset="MOUNT-PAD-ROUND" device="3.3"/>
+<part name="H4" library="holes" deviceset="MOUNT-PAD-ROUND" device="3.3"/>
 </parts>
 <sheets>
@@
 <instance part="P+16" gate="VCC" x="254" y="152.4" rot="R90"/>
 <instance part="GND19" gate="1" x="254" y="137.16" rot="R270"/>
+<instance part="H1" gate="G$1" x="104.14" y="210.82"/>
+<instance part="H2" gate="G$1" x="104.14" y="203.2"/>
+<instance part="H3" gate="G$1" x="111.76" y="210.82"/>
+<instance part="H4" gate="G$1" x="111.76" y="203.2"/>
 </instances>
 <busses>
@@
 <label x="220.98" y="157.48" size="1.778" layer="95"/>
 <pinref part="JP6" gate="G$1" pin="3"/>
+</segment>
+<segment>
+<pinref part="S1" gate="S" pin="3"/>
+<pinref part="S1" gate="S" pin="4"/>
+<wire x1="243.84" y1="73.66" x2="243.84" y2="71.12" width="0.1524" layer="91"/>
+<wire x1="243.84" y1="71.12" x2="251.46" y2="71.12" width="0.1524" layer="91"/>
+<junction x="243.84" y="71.12"/>
+<label x="248.92" y="71.12" size="1.778" layer="95"/>
 </segment>
 </net>
@@
 </segment>
 </net>
-<net name="RST" class="0">
-<segment>
-<pinref part="S1" gate="S" pin="3"/>
-<pinref part="S1" gate="S" pin="4"/>
-<wire x1="243.84" y1="73.66" x2="243.84" y2="71.12" width="0.1524" layer="91"/>
-<wire x1="243.84" y1="71.12" x2="251.46" y2="71.12" width="0.1524" layer="91"/>
-<junction x="243.84" y="71.12"/>
-<label x="248.92" y="71.12" size="1.778" layer="95"/>
-</segment>
-</net>

Commit message: first ver routing
Parts:
- removed H1, H2, H3, H4: MOUNT-PAD-ROUND3.3, holes:MOUNT-PAD-ROUND3.3
- removed JP1: (no value), jumper:JP2W
- added A3: (no value), con-phoenix-254:MPT3
Connections:
- net A3: now also A3-2.1; no longer JP1.2
- net D2: now also C7.2, R1.2, U$3G$1.B; no longer C6.2, R2.2, U$3G$1.A
- net D3: now also C6.2, R2.2, U$3G$1.A; no longer C7.2, R1.2, U$3G$1.B
- net D5: now also C9.2, R4.2, U$5G$1.B; no longer C8.2, R5.2, U$5G$1.A
- net D6: now also R6.1, U$5SW.E; no longer C9.2, R4.2, U$5G$1.B
- net D7: now also C8.2, R5.2, U$5G$1.A; no longer R6.1, U$5SW.E
- net D8: now also EXT2-2.1; no longer EXT1-2.1
- net D9: now also EXT1-2.1; no longer EXT2-2.1
- net GND: now also A3-3.1; no longer JP1.3
- net VCC: now also A3-1.1; no longer JP1.1
Changed lines of the file:
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@@
 </variantdefs>
 <classes>
-<class number="0" name="default" width="0.2032" drill="0">
+<class number="0" name="default" width="0.254" drill="0">
 </class>
-<class number="1" name="vcc" width="0" drill="0">
+<class number="1" name="vcc" width="0.635" drill="0">
 </class>
 </classes>
@@
 <part name="P+4" library="supply1" deviceset="VCC" device=""/>
 <part name="GND4" library="supply1" deviceset="GND" device=""/>
-<part name="JP1" library="jumper" deviceset="JP2W" device=""/>
 <part name="C4" library="rcl" deviceset="C-EU" device="025-025X050" value="0.1uF"/>
 <part name="GND5" library="supply1" deviceset="GND" device=""/>
@@
 <part name="P+16" library="supply1" deviceset="VCC" device=""/>
 <part name="GND19" library="supply1" deviceset="GND" device=""/>
-<part name="H1" library="holes" deviceset="MOUNT-PAD-ROUND" device="3.3"/>
-<part name="H2" library="holes" deviceset="MOUNT-PAD-ROUND" device="3.3"/>
-<part name="H3" library="holes" deviceset="MOUNT-PAD-ROUND" device="3.3"/>
-<part name="H4" library="holes" deviceset="MOUNT-PAD-ROUND" device="3.3"/>
+<part name="A3" library="con-phoenix-254" deviceset="MPT3" device=""/>
 </parts>
 <sheets>
@@
 <instance part="P+4" gate="VCC" x="220.98" y="180.34"/>
 <instance part="GND4" gate="1" x="228.6" y="180.34" rot="R180"/>
-<instance part="JP1" gate="1" x="27.94" y="91.44" rot="R90"/>
 <instance part="C4" gate="G$1" x="38.1" y="96.52"/>
 <instance part="GND5" gate="1" x="45.72" y="99.06" rot="R90"/>
@@
 <instance part="P+16" gate="VCC" x="254" y="152.4" rot="R90"/>
 <instance part="GND19" gate="1" x="254" y="137.16" rot="R270"/>
-<instance part="H1" gate="G$1" x="104.14" y="210.82"/>
-<instance part="H2" gate="G$1" x="104.14" y="203.2"/>
-<instance part="H3" gate="G$1" x="111.76" y="210.82"/>
-<instance part="H4" gate="G$1" x="111.76" y="203.2"/>
+<instance part="A3" gate="-1" x="27.94" y="86.36" rot="R180"/>
+<instance part="A3" gate="-2" x="27.94" y="91.44" rot="R180"/>
+<instance part="A3" gate="-3" x="27.94" y="96.52" rot="R180"/>
 </instances>
 <busses>
@@
 </segment>
 <segment>
-<pinref part="JP1" gate="1" pin="3"/>
-<wire x1="30.48" y1="93.98" x2="30.48" y2="99.06" width="0.1524" layer="91"/>
+<wire x1="30.48" y1="96.52" x2="30.48" y2="99.06" width="0.1524" layer="91"/>
 <wire x1="30.48" y1="99.06" x2="38.1" y2="99.06" width="0.1524" layer="91"/>
 <pinref part="GND5" gate="1" pin="GND"/>
@@
 <junction x="38.1" y="99.06"/>
 <wire x1="38.1" y1="99.06" x2="43.18" y2="99.06" width="0.1524" layer="91"/>
+<pinref part="A3" gate="-3" pin="1"/>
 </segment>
 <segment>
@@
 </segment>
 <segment>
-<pinref part="JP1" gate="1" pin="1"/>
-<wire x1="30.48" y1="88.9" x2="30.48" y2="78.74" width="0.1524" layer="91"/>
 <pinref part="P+5" gate="VCC" pin="VCC"/>
+<pinref part="A3" gate="-1" pin="1"/>
+<wire x1="30.48" y1="86.36" x2="30.48" y2="78.74" width="0.1524" layer="91"/>
 </segment>
 <segment>
@@
 </segment>
 <segment>
+<pinref part="EXT1" gate="-2" pin="1"/>
+<wire x1="203.2" y1="114.3" x2="215.9" y2="114.3" width="0.1524" layer="91"/>
+<label x="218.44" y="116.84" size="1.778" layer="95" rot="R180"/>
+</segment>
+</net>
+<net name="D8" class="0">
+<segment>
+<wire x1="200.66" y1="137.16" x2="208.28" y2="137.16" width="0.1524" layer="91"/>
+<label x="203.2" y="137.16" size="1.778" layer="95"/>
+<pinref part="JP7" gate="G$1" pin="2"/>
+</segment>
+<segment>
 <pinref part="EXT2" gate="-2" pin="1"/>
 <wire x1="241.3" y1="114.3" x2="254" y2="114.3" width="0.1524" layer="91"/>
@@
 </segment>
 </net>
-<net name="D8" class="0">
-<segment>
-<wire x1="200.66" y1="137.16" x2="208.28" y2="137.16" width="0.1524" layer="91"/>
-<label x="203.2" y="137.16" size="1.778" layer="95"/>
-<pinref part="JP7" gate="G$1" pin="2"/>
-</segment>
-<segment>
-<pinref part="EXT1" gate="-2" pin="1"/>
-<wire x1="203.2" y1="114.3" x2="215.9" y2="114.3" width="0.1524" layer="91"/>
-<label x="218.44" y="116.84" size="1.778" layer="95" rot="R180"/>
-</segment>
-</net>
 <net name="A3" class="0">
 <segment>
@@
 </segment>
 <segment>
-<pinref part="JP1" gate="1" pin="2"/>
 <wire x1="30.48" y1="91.44" x2="38.1" y2="91.44" width="0.1524" layer="91"/>
 <label x="48.26" y="91.44" size="1.778" layer="95" rot="R180"/>
@@
 <junction x="38.1" y="91.44"/>
 <wire x1="38.1" y1="91.44" x2="48.26" y2="91.44" width="0.1524" layer="91"/>
+<pinref part="A3" gate="-2" pin="1"/>
 </segment>
 </net>
@@
 <label x="203.2" y="152.4" size="1.778" layer="95"/>
 <pinref part="JP7" gate="G$1" pin="8"/>
+</segment>
+<segment>
+<pinref part="U$3" gate="G$1" pin="B"/>
+<pinref part="R1" gate="G$1" pin="2"/>
+<wire x1="144.78" y1="144.78" x2="149.86" y2="144.78" width="0.1524" layer="91"/>
+<wire x1="149.86" y1="144.78" x2="149.86" y2="142.24" width="0.1524" layer="91"/>
+<wire x1="149.86" y1="144.78" x2="167.64" y2="144.78" width="0.1524" layer="91"/>
+<junction x="149.86" y="144.78"/>
+<label x="165.1" y="144.78" size="1.778" layer="95"/>
+<pinref part="C7" gate="G$1" pin="2"/>
+<wire x1="149.86" y1="154.94" x2="149.86" y2="144.78" width="0.1524" layer="91"/>
+</segment>
+</net>
+<net name="D3" class="0">
+<segment>
+<wire x1="200.66" y1="149.86" x2="208.28" y2="149.86" width="0.1524" layer="91"/>
+<label x="203.2" y="149.86" size="1.778" layer="95"/>
+<pinref part="JP7" gate="G$1" pin="7"/>
 </segment>
 <segment>
@@
 </segment>
 </net>
-<net name="D3" class="0">
-<segment>
-<wire x1="200.66" y1="149.86" x2="208.28" y2="149.86" width="0.1524" layer="91"/>
-<label x="203.2" y="149.86" size="1.778" layer="95"/>
-<pinref part="JP7" gate="G$1" pin="7"/>
-</segment>
-<segment>
-<pinref part="U$3" gate="G$1" pin="B"/>
-<pinref part="R1" gate="G$1" pin="2"/>
-<wire x1="144.78" y1="144.78" x2="149.86" y2="144.78" width="0.1524" layer="91"/>
-<wire x1="149.86" y1="144.78" x2="149.86" y2="142.24" width="0.1524" layer="91"/>
-<wire x1="149.86" y1="144.78" x2="167.64" y2="144.78" width="0.1524" layer="91"/>
-<junction x="149.86" y="144.78"/>
-<label x="165.1" y="144.78" size="1.778" layer="95"/>
-<pinref part="C7" gate="G$1" pin="2"/>
-<wire x1="149.86" y1="154.94" x2="149.86" y2="144.78" width="0.1524" layer="91"/>
-</segment>
-</net>
 <net name="D4" class="0">
 <segment>
@@
 <label x="203.2" y="144.78" size="1.778" layer="95"/>
 <pinref part="JP7" gate="G$1" pin="5"/>
+</segment>
+<segment>
+<pinref part="U$5" gate="G$1" pin="B"/>
+<pinref part="R4" gate="G$1" pin="2"/>
+<wire x1="147.32" y1="78.74" x2="152.4" y2="78.74" width="0.1524" layer="91"/>
+<wire x1="152.4" y1="78.74" x2="152.4" y2="76.2" width="0.1524" layer="91"/>
+<wire x1="152.4" y1="78.74" x2="170.18" y2="78.74" width="0.1524" layer="91"/>
+<junction x="152.4" y="78.74"/>
+<label x="167.64" y="78.74" size="1.778" layer="95"/>
+<pinref part="C9" gate="G$1" pin="2"/>
+<wire x1="152.4" y1="91.44" x2="152.4" y2="78.74" width="0.1524" layer="91"/>
+</segment>
+</net>
+<net name="D6" class="0">
+<segment>
+<wire x1="200.66" y1="142.24" x2="208.28" y2="142.24" width="0.1524" layer="91"/>
+<label x="203.2" y="142.24" size="1.778" layer="95"/>
+<pinref part="JP7" gate="G$1" pin="4"/>
+</segment>
+<segment>
+<pinref part="U$5" gate="SW" pin="E"/>
+<wire x1="111.76" y1="78.74" x2="111.76" y2="91.44" width="0.1524" layer="91"/>
+<pinref part="R6" gate="G$1" pin="1"/>
+<wire x1="111.76" y1="91.44" x2="111.76" y2="109.22" width="0.1524" layer="91"/>
+<wire x1="111.76" y1="91.44" x2="109.22" y2="91.44" width="0.1524" layer="91"/>
+<junction x="111.76" y="91.44"/>
+<label x="111.76" y="106.68" size="1.778" layer="95" rot="R90"/>
+</segment>
+</net>
+<net name="D7" class="0">
+<segment>
+<wire x1="200.66" y1="139.7" x2="208.28" y2="139.7" width="0.1524" layer="91"/>
+<label x="203.2" y="139.7" size="1.778" layer="95"/>
+<pinref part="JP7" gate="G$1" pin="3"/>
 </segment>
 <segment>
@@
 </segment>
 </net>
-<net name="D6" class="0">
-<segment>
-<wire x1="200.66" y1="142.24" x2="208.28" y2="142.24" width="0.1524" layer="91"/>
-<label x="203.2" y="142.24" size="1.778" layer="95"/>
-<pinref part="JP7" gate="G$1" pin="4"/>
-</segment>
-<segment>
-<pinref part="U$5" gate="G$1" pin="B"/>
-<pinref part="R4" gate="G$1" pin="2"/>
-<wire x1="147.32" y1="78.74" x2="152.4" y2="78.74" width="0.1524" layer="91"/>
-<wire x1="152.4" y1="78.74" x2="152.4" y2="76.2" width="0.1524" layer="91"/>
-<wire x1="152.4" y1="78.74" x2="170.18" y2="78.74" width="0.1524" layer="91"/>
-<junction x="152.4" y="78.74"/>
-<label x="167.64" y="78.74" size="1.778" layer="95"/>
-<pinref part="C9" gate="G$1" pin="2"/>
-<wire x1="152.4" y1="91.44" x2="152.4" y2="78.74" width="0.1524" layer="91"/>
-</segment>
-</net>
-<net name="D7" class="0">
-<segment>
-<wire x1="200.66" y1="139.7" x2="208.28" y2="139.7" width="0.1524" layer="91"/>
-<label x="203.2" y="139.7" size="1.778" layer="95"/>
-<pinref part="JP7" gate="G$1" pin="3"/>
-</segment>
-<segment>
-<pinref part="U$5" gate="SW" pin="E"/>
-<wire x1="111.76" y1="78.74" x2="111.76" y2="91.44" width="0.1524" layer="91"/>
-<pinref part="R6" gate="G$1" pin="1"/>
-<wire x1="111.76" y1="91.44" x2="111.76" y2="109.22" width="0.1524" layer="91"/>
-<wire x1="111.76" y1="91.44" x2="109.22" y2="91.44" width="0.1524" layer="91"/>
-<junction x="111.76" y="91.44"/>
-<label x="111.76" y="106.68" size="1.778" layer="95" rot="R90"/>
-</segment>
-</net>

Commit message: wip
Parts:
- added H1, H2: MOUNT-HOLE3.0, holes:MOUNT-HOLE3.0
Changed lines of the file:
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@@
 <part name="GND19" library="supply1" deviceset="GND" device=""/>
 <part name="A3" library="con-phoenix-254" deviceset="MPT3" device=""/>
+<part name="H1" library="holes" deviceset="MOUNT-HOLE" device="3.0"/>
+<part name="H2" library="holes" deviceset="MOUNT-HOLE" device="3.0"/>
 </parts>
 <sheets>
@@
 <instance part="A3" gate="-2" x="27.94" y="91.44" rot="R180"/>
 <instance part="A3" gate="-3" x="27.94" y="96.52" rot="R180"/>
+<instance part="H1" gate="G$1" x="73.66" y="203.2"/>
+<instance part="H2" gate="G$1" x="73.66" y="198.12"/>
 </instances>
 <busses>
