File: eagle/blinkybee/scarf.brd (EAGLE design)
At the start: 40 x 74 mm, 17 parts, among them IC1 TLC272P, M1 ELECTRET_MICROPHON-WM.64PN

Commit message: mic layout take 2
Parts:
- moved C1 22.7 mm to (22.6, 15.0), turned to 270 degrees
- moved R6 21.4 mm to (7.62, 18.8), turned to 180 degrees
- moved R7 13.9 mm to (23.6, 22.6), turned to 270 degrees
- moved C3 13.7 mm to (16.8, 15.0)
- moved R5 10.2 mm to (9.40, 16.5)
- moved R2 9.37 mm to (11.9, 31.8)
- moved R1 6.53 mm to (8.38, 24.6), turned to 90 degrees
- moved R4 4.10 mm to (23.1, 28.4)
- moved IC1 2.84 mm to (17.0, 22.6), turned to 180 degrees
- moved R3 2.51 mm to (21.3, 31.0), turned to 180 degrees
- moved C2 2.09 mm to (13.2, 28.7)
- moved M1 0.51 mm to (4.06, 27.7)
Routing:
- net N$2: track 6.76 -> 16.1 mm
- net N$3: track 12.1 -> 15.3 mm
- net N$1: track 7.62 -> 5.33 mm
- net N$6: track 42.8 -> 41.1 mm
- net MIC_OUT: track 3.81 -> 3.17 mm
- net N$5: track 4.57 -> 4.06 mm

Commit message: scarf pcb
Parts:
- removed PWR: (no value), con-phoenix-254:2POL254
- added C4, C6: 0.1uF, rcl:C025-025X050
- added CAP1, CAP2: (no value), pinhead:1X01
- added H1, H2, H3, H4: MOUNT-HOLE3.0, holes:3,0
- added LEDS1, LEDS2, MIC_SW: (no value), pinhead:1X03
- added PWR1, PWR2: (no value), con-phoenix-254:2POL254
- added R8, R9: 5M, rcl:0204/7
- moved C5 35.8 mm to (35.1, 26.7), turned to 0 degrees
- moved JP6 33.5 mm to (35.1, 42.7), turned to 0 degrees
- moved S1 23.0 mm to (25.7, 49.8)
- moved JP7 13.7 mm to (7.11, 57.9), turned to 180 degrees
- moved C3 8.95 mm to (21.8, 22.4)
- moved R3 8.74 mm to (26.4, 38.1)
- moved R7 8.74 mm to (28.7, 29.7)
- moved C2 8.74 mm to (18.3, 35.8)
- moved R1 8.74 mm to (13.5, 31.8)
- moved R2 8.74 mm to (17.0, 38.9)
- moved R4 8.74 mm to (28.2, 35.6)
- moved R5 8.74 mm to (14.5, 23.6)
- moved R6 8.74 mm to (12.7, 25.9)
- moved C1 8.74 mm to (27.7, 22.1)
- moved IC1 8.74 mm to (22.1, 29.7)
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Connections:
- net MIC_OUT renamed MIC_OUT_D
- net N$4 renamed MIC_OUT_A
- net D10: now also MIC_SW.2
- net D2: now also R8.2
- net D3: now also C4.2, CAP1.1, R8.1
- net D4: now also LEDS1.2, LEDS2.2
- net D6: now also R9.2
- net D9: now also C6.2, CAP2.1, R9.1
- net GND: now also C4.1, C6.1, LEDS1.1, LEDS2.1, MIC_SW.1, PWR1.2, PWR2.2; no longer PWR.2
- net VCC: now also LEDS1.3, LEDS2.3, MIC_SW.3, PWR1.1, PWR2.1; no longer PWR.1
Routing:
- net D4: track 0.00 -> 74.1 mm, vias 0 -> 4
- net D3: track 0.00 -> 42.6 mm, vias 0 -> 1
- net D2: track 0.00 -> 25.2 mm, vias 0 -> 3
- net RESET: track 0.00 -> 11.2 mm
- net D10: track 0.00 -> 9.58 mm, vias 0 -> 1
- net D9: track 0.00 -> 9.43 mm
- net D6: track 0.00 -> 2.79 mm
- added copper zone on layer 1, net VCC
Other:
- board size 40 x 74 mm -> 40.6 x 77 mm
- board text added: "CUT OFF"

Commit message: scarf pcb
Parts:
- moved MIC_SW 8.59 mm to (5.26, 28.5), turned to 45 degrees
Routing:
- net D10: track 9.58 -> 14.9 mm
- net D4: track 74.1 -> 73.3 mm
Changed lines of the file:
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@@
 <element name="H3" library="holes" package="3,0" value="MOUNT-HOLE3.0" x="3.81" y="50.8"/>
 <element name="H4" library="holes" package="3,0" value="MOUNT-HOLE3.0" x="3.81" y="19.05" smashed="yes"/>
-<element name="MIC_SW" library="pinhead" package="1X03" value="" x="2.286" y="36.576" rot="R270"/>
+<element name="MIC_SW" library="pinhead" package="1X03" value="" x="5.259603125" y="28.52239375" rot="R45"/>
 <element name="LEDS1" library="pinhead" package="1X03" value="" x="20.32" y="16.002"/>
 <element name="LEDS2" library="pinhead" package="1X03" value="" x="20.32" y="60.96"/>
@@
 <contactref element="C3" pad="-"/>
 <polygon width="0.8128" layer="16">
-<vertex x="39.37" y="75.692"/>
-<vertex x="39.37" y="0.254"/>
-<vertex x="1.27" y="0.254"/>
-<vertex x="1.27" y="75.692"/>
+<vertex x="40.386" y="75.692"/>
+<vertex x="40.386" y="0.254"/>
+<vertex x="0.254" y="0.254"/>
+<vertex x="0.254" y="75.692"/>
 </polygon>
 <contactref element="MIC_SW" pad="1"/>
@@
 <contactref element="PWR2" pad="1"/>
 <polygon width="0.8128" layer="1">
-<vertex x="39.37" y="75.692"/>
-<vertex x="39.37" y="0.254"/>
-<vertex x="1.27" y="0.254"/>
-<vertex x="1.27" y="75.692"/>
+<vertex x="40.386" y="75.692"/>
+<vertex x="40.386" y="0.254"/>
+<vertex x="0.254" y="0.254"/>
+<vertex x="0.254" y="75.692"/>
 </polygon>
 </signal>
@@
 <wire x1="6.858" y1="26.924" x2="12.192" y2="32.258" width="0.4064" layer="1"/>
 <wire x1="12.192" y1="32.258" x2="12.192" y2="36.83" width="0.4064" layer="1"/>
-<wire x1="12.192" y1="36.83" x2="9.144" y2="39.878" width="0.4064" layer="1"/>
-<via x="9.144" y="39.878" extent="1-16" drill="0.6"/>
-<wire x1="9.144" y1="39.878" x2="5.588" y2="39.878" width="0.4064" layer="16"/>
-<wire x1="5.588" y1="39.878" x2="4.826" y2="40.64" width="0.4064" layer="16"/>
-<via x="4.826" y="40.64" extent="1-16" drill="0.6"/>
-<wire x1="4.826" y1="40.64" x2="4.826" y2="42.926" width="0.4064" layer="1"/>
-<wire x1="4.826" y1="42.926" x2="6.35" y2="44.45" width="0.4064" layer="1"/>
+<wire x1="12.192" y1="36.83" x2="8.89" y2="40.132" width="0.4064" layer="1"/>
+<via x="8.89" y="40.132" extent="1-16" drill="0.6"/>
+<via x="5.334" y="40.894" extent="1-16" drill="0.6"/>
+<wire x1="5.334" y1="40.894" x2="5.334" y2="43.434" width="0.4064" layer="1"/>
+<wire x1="5.334" y1="43.434" x2="6.35" y2="44.45" width="0.4064" layer="1"/>
 <wire x1="6.35" y1="44.45" x2="15.748" y2="44.45" width="0.4064" layer="1"/>
 <wire x1="15.748" y1="44.45" x2="19.812" y2="48.514" width="0.4064" layer="1"/>
@@
 <via x="19.812" y="54.61" extent="1-16" drill="0.6"/>
 <wire x1="19.812" y1="54.61" x2="19.812" y2="57.912" width="0.4064" layer="1"/>
+<wire x1="8.89" y1="40.132" x2="5.842" y2="40.132" width="0.4064" layer="16"/>
+<wire x1="5.842" y1="40.132" x2="5.334" y2="40.894" width="0.4064" layer="16"/>
 </signal>
 <signal name="D5">
@@
 <contactref element="JP6" pad="12"/>
 <contactref element="MIC_SW" pad="2"/>
-<wire x1="2.286" y1="36.576" x2="4.826" y2="36.576" width="0.4064" layer="16"/>
-<wire x1="4.826" y1="36.576" x2="7.112" y2="38.862" width="0.4064" layer="16"/>
-<via x="7.112" y="38.862" extent="1-16" drill="0.6"/>
-<wire x1="7.112" y1="38.862" x2="7.112" y2="42.672" width="0.4064" layer="1"/>
+<wire x1="5.259603125" y1="28.52239375" x2="5.259603125" y2="36.755603125" width="0.4064" layer="16"/>
+<wire x1="5.259603125" y1="36.755603125" x2="7.112" y2="38.608" width="0.4064" layer="16"/>
+<via x="7.112" y="38.608" extent="1-16" drill="0.6"/>
+<wire x1="7.112" y1="38.608" x2="7.112" y2="42.672" width="0.4064" layer="1"/>
 </signal>
 <signal name="RXI">

Commit message: scarf v2014-03-22 sent to oshpark
Parts:
- removed H1, H2, H3, H4: MOUNT-HOLE3.0, holes:3,0
- added AIN0, AIN1: (no value), microbuilder:1X03_ROUND
- added C7, C8: 0.1uF, rcl:C025-025X050
- CAP1, CAP2: device pinhead:1X01 -> microbuilder:1X03_ROUND
- MIC_SW: device pinhead:1X03 -> microbuilder:1X03_ROUND
- moved CAP1 7.13 mm to (35.3, 28.2)
- moved C5 4.32 mm to (35.1, 22.4)
- moved CAP2 1.70 mm to (1.52, 61.5), turned to 90 degrees
- moved MIC_SW 0.74 mm to (5.45, 27.8)
- turned PWR1 to 0 degrees
Connections:
- removed net MIC_OUT_A: IC1.1, IC1.6, R4.1
- removed net MIC_OUT_D: C3.+, IC1.7
- net A0: now also AIN0.2, C8.1
- net A1: now also AIN1.2, C7.1
- net A2: now also IC1.1, IC1.6, R4.1
- net A3: now also C3.+, IC1.7
- net D3: now also CAP1.2; no longer CAP1.1
- net D9: now also CAP2.2; no longer CAP2.1
- net GND: now also AIN0.1, AIN1.1, C7.2, C8.2, CAP1.1, CAP2.1
- net VCC: now also AIN0.3, AIN1.3, CAP1.3, CAP2.3
Routing:
- net A1: track 0.00 -> 24.6 mm, vias 0 -> 1
- net A3: track 0.00 -> 22.4 mm
- net A2: track 0.00 -> 20.3 mm
- net A0: track 0.00 -> 19.1 mm, vias 0 -> 1
- net MIC_OUT_A: track 12.4 -> 0.00 mm
- net D3: track 42.6 -> 47.3 mm
- net GND: track 0.00 -> 3.64 mm
- net MIC_OUT_D: track 3.10 -> 0.00 mm
- net D10: track 14.9 -> 15.7 mm
Other:
- outline, holes or cut-outs redrawn
- board text added: "+"
- board text added: "2014-03-22"
- board text added: "blinkybee.com"
