File: eagle/blinkybee/scarf.sch (EAGLE design)
At the start: 17 parts, among them IC1 TLC272P, M1 ELECTRET_MICROPHON-WM.64PN

Commit message: scarf pcb
Parts:
- added C4, C6: 0.1uF, rcl:C-EU025-025X050
- added CAP1, CAP2: (no value), pinhead:PINHD-1X1
- added H1, H2, H3, H4: MOUNT-HOLE3.0, holes:MOUNT-HOLE3.0
- added LEDS1, LEDS2, MIC_SW: (no value), pinhead:PINHD-1X3
- added PWR2: (no value), con-phoenix-254:MPT2
- added R8, R9: 5M, rcl:R-US_0204/7
- renumbered PWR to PWR1
Connections:
- net MIC_OUT renamed MIC_OUT_D
- net N$4 renamed MIC_OUT_A
- net D10: now also MIC_SW.2
- net D2: now also R8.2
- net D3: now also C4.2, CAP1.1, R8.1
- net D4: now also LEDS1.2, LEDS2.2
- net D6: now also R9.2
- net D9: now also C6.2, CAP2.1, R9.1
- net GND: now also C4.1, C6.1, LEDS1.1, LEDS2.1, MIC_SW.1, PWR2-2.1
- net VCC: now also LEDS1.3, LEDS2.3, MIC_SW.3, PWR2-1.1

Commit message: scarf v2014-03-22 sent to oshpark
Parts:
- removed H1, H2, H3, H4: MOUNT-HOLE3.0, holes:MOUNT-HOLE3.0
- added AIN0, AIN1: (no value), microbuilder:HEADER-1X3ROUND
- added C7, C8: 0.1uF, rcl:C-EU025-025X050
- CAP1, CAP2: device pinhead:PINHD-1X1 -> microbuilder:HEADER-1X3ROUND
- MIC_SW: device pinhead:PINHD-1X3 -> microbuilder:HEADER-1X3ROUND
Connections:
- removed net MIC_OUT_A: IC1A.OUT, IC1B.-IN, R4.1
- removed net MIC_OUT_D: C3.+, IC1B.OUT
- net A0: now also AIN0.2, C8.1
- net A1: now also AIN1.2, C7.1
- net A2: now also IC1A.OUT, IC1B.-IN, R4.1
- net A3: now also C3.+, IC1B.OUT
- net D3: now also CAP1.2; no longer CAP1.1
- net D9: now also CAP2.2; no longer CAP2.1
- net GND: now also AIN0.1, AIN1.1, C7.2, C8.2, CAP1.1, CAP2.1
- net VCC: now also AIN0.3, AIN1.3, CAP1.3, CAP2.3
