File: eagle/blinkybee/scarf_no_mic.brd (EAGLE design)
At the start: 40.6 x 61.7 mm, 19 parts

Commit message: wip
Parts:
- added JP1: (no value), jumper:JP2Q
- moved UBEC_OUT 34.1 mm to (3.05, 18.8)
- moved BAT_IN 33.0 mm to (36.8, 17.3), turned to 90 degrees
- moved PWR_SW 29.4 mm to (34.8, 22.4), turned to 180 degrees
- moved UBEC_IN 24.9 mm to (32.8, 17.3), turned to 270 degrees
- moved C5 22.8 mm to (8.38, 16.3)
- moved AIN1 4.85 mm to (17.3, 20.3)
- moved AIN0 3.41 mm to (17.3, 22.4)
- moved C7 0.80 mm to (23.6, 24.6)
- moved C8 0.76 mm to (16.0, 24.9)
Connections:
- removed net D14: LEDS1.2
- net GND: now also JP1.4
- net MISO: now also LEDS1.2
- net N$2: now also JP1.1
- net N$3: now also JP1.3
- net RAW: now also JP1.2
Routing:
- net MISO: track 0.00 -> 18.4 mm, vias 0 -> 1
- net RAW: track 0.00 -> 14.3 mm
- net A2: track 6.71 -> 11.2 mm
- net N$3: track 4.06 -> 7.62 mm
- net N$2: track 4.13 -> 7.68 mm
- net A0: track 8.37 -> 6.35 mm
