File: eagle/blinkybee/scarf_no_mic.sch (EAGLE design)
At the start: 19 parts

Commit message: wip
Parts:
- added JP1: (no value), jumper:JP2Q
Connections:
- removed net D14: LEDS1.2
- net GND: now also JP1.4
- net MISO: now also LEDS1.2
- net N$2: now also JP1.1
- net N$3: now also JP1.3
- net RAW: now also JP1.2
Other:
- moved on the sheet: UBEC_IN-1, UBEC_IN-2
Changed lines of the file:
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@@
 <part name="PWR_SW" library="con-phoenix-254" deviceset="MPT2" device=""/>
 <part name="UBEC_IN" library="con-phoenix-254" deviceset="MPT2" device=""/>
+<part name="JP1" library="jumper" deviceset="JP2Q" device=""/>
+<part name="GND1" library="supply1" deviceset="GND" device=""/>
 </parts>
 <sheets>
@@
 <instance part="PWR_SW" gate="-1" x="271.78" y="101.6" rot="R90"/>
 <instance part="PWR_SW" gate="-2" x="276.86" y="101.6" rot="R90"/>
-<instance part="UBEC_IN" gate="-1" x="284.48" y="99.06"/>
-<instance part="UBEC_IN" gate="-2" x="284.48" y="93.98"/>
+<instance part="UBEC_IN" gate="-1" x="294.64" y="99.06"/>
+<instance part="UBEC_IN" gate="-2" x="294.64" y="93.98"/>
+<instance part="JP1" gate="B1" x="289.56" y="114.3" rot="MR0"/>
+<instance part="GND1" gate="1" x="287.02" y="129.54" rot="R180"/>
 </instances>
 <busses>
@@
 <wire x1="386.08" y1="193.04" x2="386.08" y2="203.2" width="0.1524" layer="91"/>
 </segment>
+<segment>
+<pinref part="GND1" gate="1" pin="GND"/>
+<pinref part="JP1" gate="B1" pin="4"/>
+<wire x1="287.02" y1="127" x2="287.02" y2="121.92" width="0.1524" layer="91"/>
+</segment>
 </net>
 <net name="RESET" class="0">
@@
 <pinref part="JP6" gate="G$1" pin="10"/>
 </segment>
+<segment>
+<pinref part="LEDS1" gate="A" pin="2"/>
+<wire x1="299.72" y1="187.96" x2="279.4" y2="187.96" width="0.1524" layer="91"/>
+<label x="279.4" y="187.96" size="1.778" layer="95"/>
+</segment>
 </net>
 <net name="MOSI" class="0">
@@
 <label x="220.98" y="162.56" size="1.778" layer="95"/>
 <pinref part="JP6" gate="G$1" pin="1"/>
+</segment>
+<segment>
+<pinref part="JP1" gate="B1" pin="2"/>
+<wire x1="289.56" y1="121.92" x2="289.56" y2="127" width="0.1524" layer="91"/>
+<label x="289.56" y="127" size="1.778" layer="95"/>
 </segment>
 </net>
@@
 <pinref part="PWR_SW" gate="-2" pin="1"/>
 <pinref part="UBEC_IN" gate="-1" pin="1"/>
-<wire x1="276.86" y1="99.06" x2="281.94" y2="99.06" width="0.1524" layer="91"/>
+<wire x1="276.86" y1="99.06" x2="289.56" y2="99.06" width="0.1524" layer="91"/>
+<pinref part="JP1" gate="B1" pin="1"/>
+<wire x1="289.56" y1="99.06" x2="292.1" y2="99.06" width="0.1524" layer="91"/>
+<wire x1="289.56" y1="99.06" x2="289.56" y2="106.68" width="0.1524" layer="91"/>
+<junction x="289.56" y="99.06"/>
 </segment>
 </net>
@@
 <pinref part="BAT_IN" gate="-1" pin="1"/>
 <pinref part="UBEC_IN" gate="-2" pin="1"/>
-<wire x1="266.7" y1="93.98" x2="281.94" y2="93.98" width="0.1524" layer="91"/>
-</segment>
-</net>
-<net name="D14" class="0">
-<segment>
-<pinref part="LEDS1" gate="A" pin="2"/>
-<wire x1="299.72" y1="187.96" x2="279.4" y2="187.96" width="0.1524" layer="91"/>
-<label x="279.4" y="187.96" size="1.778" layer="95"/>
-</segment>
-</net>
+<wire x1="266.7" y1="93.98" x2="287.02" y2="93.98" width="0.1524" layer="91"/>
+<pinref part="JP1" gate="B1" pin="3"/>
+<wire x1="287.02" y1="93.98" x2="292.1" y2="93.98" width="0.1524" layer="91"/>
+<wire x1="287.02" y1="106.68" x2="287.02" y2="93.98" width="0.1524" layer="91"/>
+<junction x="287.02" y="93.98"/>
+</segment>
+</net>
