File: eagle/mutebox/mutebox.brd (EAGLE design)
At the start: 127 x 63.5 mm, 60 parts, among them IC1 74HCT595D, IC2 74HC165D

Commit message: mutebox
Parts:
- IC3, IC4: value 21298E -> MCP3208
- renumbered JP2 to P_CONN, JP3 to B_CONN, U$29 to IC3, U$47 to IC4
Connections:
- net B_PB3: now also IC2.4; no longer IC2.3
- net B_PB4: now also IC2.3; no longer IC2.4
- net P10: now also IC3.P$3; no longer IC3.P$4
- net P11: now also IC3.P$2; no longer IC3.P$5
- net P12: now also IC3.P$1; no longer IC3.P$2
- net P15: now also IC4.P$3; no longer IC4.P$4
- net P16: now also IC4.P$1; no longer IC4.P$2
- net P2: now also IC3.P$7; no longer IC3.P$6
- net P3: now also IC3.P$6; no longer IC3.P$3
- net P4: now also IC3.P$5; no longer IC3.P$1
- net P7: now also IC4.P$4; no longer IC4.P$3
- net P8: now also IC4.P$2; no longer IC4.P$1
- net P9: now also IC3.P$4; no longer IC3.P$7
Routing:
- net P9: track 34.1 -> 46.4 mm, vias 0 -> 1
- net P12: track 42.3 -> 53.2 mm
- net P4: track 26.8 -> 32.4 mm
- net P3: track 13.8 -> 18.9 mm
- net P11: track 29.8 -> 34.2 mm, vias 0 -> 1
- net B_PB4: track 74.0 -> 69.6 mm
- net B_PB3: track 84.1 -> 86.4 mm
- net P10: track 31.2 -> 32.6 mm, vias 0 -> 1
- net P8: track 25.7 -> 24.4 mm
- net P15: track 31.7 -> 31.0 mm, vias 0 -> 1
- net P16: track 35.2 -> 34.6 mm, vias 0 -> 1
- net P2: track 13.6 -> 13.0 mm
- net P7: track 14.7 -> 15.2 mm
Other:
- board text added: "Designed by Eran Rundstein, Nov 2014"

Commit message: wip
Parts:
- R1: value 10kB -> 10kB (688-RK09D1130C2P)
Changed lines of the file:
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@@
 <element name="U$6" library="keves" package="B3J-XX00-1LED" value="B3J-XX00-1LED" x="84.328" y="9.906"/>
 <element name="U$1" library="keves" package="B3J-XX00-1LED" value="B3J-XX00-1LED" x="14.478" y="9.906"/>
-<element name="R1" library="pot-alps" package="ALPS_POT_VERTICAL_PS" value="10kB" x="14.478" y="48.006" rot="R180"/>
+<element name="R1" library="pot-alps" package="ALPS_POT_VERTICAL_PS" value="10kB (688-RK09D1130C2P)" x="14.478" y="48.006" rot="R180"/>
 <element name="R12" library="pot-alps" package="ALPS_POT_VERTICAL_PS" value="10kB" x="84.328" y="32.766" rot="R180"/>
 <element name="R10" library="pot-alps" package="ALPS_POT_VERTICAL_PS" value="10kB" x="70.358" y="32.766" rot="R180"/>

Commit message: muteboxwip
Parts:
- B_CONN, P_CONN: device pinhead:2X05 -> microbuilder:2X05
Changed lines of the file:
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@@
 <element name="C7" library="microbuilder" package="0603" value="100nF" x="2.794" y="24.892" rot="MR270"/>
 <element name="C8" library="microbuilder" package="0603" value="100nF" x="122.936" y="11.176" rot="MR180"/>
-<element name="P_CONN" library="pinhead" package="2X05" value="" x="3.81" y="46.99" rot="MR90"/>
+<element name="P_CONN" library="microbuilder" package="2X05" value="" x="3.81" y="46.99" rot="MR90"/>
 <element name="R33" library="microbuilder" package="_0805" value="10" x="8.128" y="43.434" rot="R270"/>
-<element name="B_CONN" library="pinhead" package="2X05" value="" x="123.19" y="31.75" rot="R90"/>
+<element name="B_CONN" library="microbuilder" package="2X05" value="" x="123.19" y="31.75" rot="R90"/>
 <element name="R34" library="microbuilder" package="_0603" value="10K" x="125.984" y="24.384" rot="R90"/>
 </elements>
