File: eagle/mutebox/mutebox.brd (EAGLE design)
At the start: 127 x 63.5 mm, 60 parts, among them IC1 74HCT595D, IC2 74HC165D, IC3 MCP3208, IC4 MCP3208

Commit message: mutebox rearrange buttons
Parts:
- B_CONN, P_CONN: device microbuilder:2X05 -> con-harting-ml:ML10
- moved R25 4.58 mm to (22.4, 6.35)
- moved R1 4.57 mm to (19.1, 48.0)
- moved R2 4.57 mm to (19.1, 32.8)
- moved U$1 4.57 mm to (19.1, 9.91)
- moved R24 4.35 mm to (108.5, 21.1)
- moved R15 4.32 mm to (108.0, 48.0)
- moved R16 4.32 mm to (108.0, 32.8)
- moved U$8 4.32 mm to (108.0, 9.91)
- moved R26 3.34 mm to (35.1, 6.60)
- moved R18 3.31 mm to (35.1, 20.1)
- moved R3 3.30 mm to (31.8, 48.0)
- moved R6 3.30 mm to (31.8, 32.8)
- moved U$2 3.30 mm to (31.8, 9.91)
- moved R13 3.05 mm to (95.2, 48.0)
- moved R14 3.05 mm to (95.2, 32.8)
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Routing:
- net P13: track 38.3 -> 47.3 mm
- net P12: track 53.2 -> 46.2 mm
- net P10: track 32.6 -> 37.5 mm
- net AVCC: track 28.0 -> 32.6 mm
- net B_PB1: track 125.8 -> 121.5 mm
- net B_LED8: track 117.3 -> 113.2 mm
- net P9: track 46.4 -> 42.9 mm
- net B_PB8: track 27.1 -> 30.5 mm
- net B_LED2: track 29.0 -> 32.2 mm
- net B_LED6: track 86.4 -> 83.5 mm
- net B_PB2: track 109.3 -> 106.5 mm
- net VCC: track 27.0 -> 29.5 mm
- net B_LED3: track 40.5 -> 42.8 mm
- net B_LED7: track 107.1 -> 105.1 mm
- net B_PB7: track 39.4 -> 41.4 mm
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
Commit message: wip
Other:
- board text added: "MuteBox UI 1.0 (c) Eran Rundstein, 2014"
- board text removed: "Designed by Eran Rundstein, Nov 2014"

Commit message: wip
Parts:
- added H5, H6: MOUNT-HOLE3.2, holes:3,2
- moved B_CONN 11.0 mm to (121.7, 42.7)
- moved R34 4.93 mm to (123.2, 20.3), turned to 180 degrees
- moved C7 4.89 mm to (7.62, 24.1), turned to 0 degrees
Routing:
- net B_RC1: track 27.7 -> 46.0 mm
- net B_SI: track 11.4 -> 24.2 mm
- net B_SC: track 146.7 -> 155.9 mm
- net B_RC2: track 148.8 -> 157.8 mm
- net B_SO: track 140.0 -> 148.2 mm
- net VCC: track 29.5 -> 35.8 mm

Commit message: wip
Parts:
- moved B_CONN 1.37 mm to (122.2, 43.9), flipped to the bottom, turned to 270 degrees
Routing:
- net B_RC1: track 46.0 -> 32.8 mm
- net B_RC2: track 157.8 -> 148.3 mm, vias 3 -> 4
- net B_SC: track 155.9 -> 151.7 mm
- net B_SI: track 24.2 -> 26.7 mm
- net B_SO: track 148.2 -> 150.5 mm
Changed lines of the file:
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@@
 <attribute name="VALUE" x="6.477" y="45.0214" size="0.4064" layer="27" ratio="10" rot="R270"/>
 </element>
-<element name="B_CONN" library="con-harting-ml" package="ML10" value="" x="121.666" y="42.672" smashed="yes" rot="R90">
-<attribute name="OC_NEWARK" value="unknown" x="121.666" y="42.672" size="1.778" layer="27" rot="R90" display="off"/>
-<attribute name="MPN" value="" x="121.666" y="42.672" size="1.778" layer="27" rot="R90" display="off"/>
-<attribute name="MF" value="" x="121.666" y="42.672" size="1.778" layer="27" rot="R90" display="off"/>
-<attribute name="OC_FARNELL" value="unknown" x="121.666" y="42.672" size="1.778" layer="27" rot="R90" display="off"/>
-<attribute name="NAME" x="116.586" y="32.512" size="1.778" layer="25" ratio="10" rot="R90"/>
-<attribute name="VALUE" x="116.586" y="42.672" size="1.778" layer="27" ratio="10" rot="R90"/>
+<element name="B_CONN" library="con-harting-ml" package="ML10" value="" x="122.174" y="43.942" smashed="yes" rot="MR270">
+<attribute name="OC_NEWARK" value="unknown" x="122.174" y="43.942" size="1.778" layer="28" rot="MR270" display="off"/>
+<attribute name="MPN" value="" x="122.174" y="43.942" size="1.778" layer="28" rot="MR270" display="off"/>
+<attribute name="MF" value="" x="122.174" y="43.942" size="1.778" layer="28" rot="MR270" display="off"/>
+<attribute name="OC_FARNELL" value="unknown" x="122.174" y="43.942" size="1.778" layer="28" rot="MR270" display="off"/>
+<attribute name="NAME" x="117.094" y="54.102" size="1.778" layer="26" ratio="10" rot="MR270"/>
+<attribute name="VALUE" x="117.094" y="43.942" size="1.778" layer="28" ratio="10" rot="MR270"/>
 </element>
 <element name="R34" library="microbuilder" package="_0603" value="10K" x="123.19" y="20.32" smashed="yes" rot="R180">
@@
 <contactref element="B_CONN" pad="1"/>
 <contactref element="B_CONN" pad="2"/>
-<wire x1="122.936" y1="37.592" x2="120.396" y2="37.592" width="1.778" layer="1"/>
+<wire x1="123.444" y1="49.022" x2="120.904" y2="49.022" width="1.778" layer="16"/>
 </signal>
 <signal name="B_LED1">
@@
 <contactref element="IC2" pad="9"/>
 <contactref element="B_CONN" pad="5"/>
-<wire x1="122.936" y1="42.672" x2="122.428" y2="42.672" width="0.254" layer="16"/>
-<wire x1="122.428" y1="42.672" x2="121.666" y2="41.91" width="0.254" layer="16"/>
-<wire x1="121.666" y1="41.91" x2="121.666" y2="31.75" width="0.254" layer="16"/>
-<wire x1="121.666" y1="31.75" x2="120.269" y2="30.353" width="0.254" layer="16"/>
-<wire x1="120.269" y1="30.353" x2="120.142" y2="30.226" width="0.254" layer="16"/>
 <wire x1="123.9774" y1="21.717" x2="123.9774" y2="22.0726" width="0.254" layer="16"/>
 <wire x1="123.9774" y1="22.0726" x2="119.888" y2="26.162" width="0.254" layer="16"/>
 <wire x1="119.888" y1="26.162" x2="119.888" y2="29.972" width="0.254" layer="16"/>
-<wire x1="119.888" y1="29.972" x2="120.142" y2="30.226" width="0.254" layer="16"/>
+<wire x1="119.888" y1="29.972" x2="124.968" y2="35.052" width="0.254" layer="16"/>
+<wire x1="124.968" y1="35.052" x2="124.968" y2="42.418" width="0.254" layer="16"/>
+<wire x1="124.968" y1="42.418" x2="123.444" y2="43.942" width="0.254" layer="16"/>
 </signal>
 <signal name="B_SC">
@@
 <contactref element="B_CONN" pad="7"/>
 <contactref element="B_CONN" pad="8"/>
-<wire x1="116.078" y1="20.32" x2="116.078" y2="15.24" width="0.254" layer="16"/>
+<wire x1="116.078" y1="20.066" x2="116.078" y2="15.24" width="0.254" layer="16"/>
 <wire x1="117.8306" y1="14.097" x2="117.221" y2="14.097" width="0.254" layer="16"/>
 <wire x1="117.221" y1="14.097" x2="116.078" y2="15.24" width="0.254" layer="16"/>
@@
 <wire x1="114.808" y1="13.462" x2="116.586" y2="13.462" width="0.254" layer="16"/>
 <wire x1="116.586" y1="13.462" x2="117.221" y2="14.097" width="0.254" layer="16"/>
-<wire x1="116.84" y1="21.082" x2="116.078" y2="20.32" width="0.254" layer="1"/>
-<via x="116.078" y="20.32" extent="1-16" drill="0.6"/>
+<via x="116.078" y="20.066" extent="1-16" drill="0.6"/>
 <wire x1="109.728" y1="11.938" x2="109.982" y2="12.192" width="0.254" layer="16"/>
-<wire x1="116.84" y1="21.082" x2="118.11" y2="21.082" width="0.254" layer="1"/>
-<wire x1="118.11" y1="21.082" x2="118.618" y2="21.59" width="0.254" layer="1"/>
-<wire x1="118.618" y1="21.59" x2="118.618" y2="43.434" width="0.254" layer="1"/>
-<wire x1="118.618" y1="43.434" x2="120.396" y2="45.212" width="0.254" layer="1"/>
-<wire x1="120.396" y1="45.212" x2="122.936" y2="45.212" width="0.254" layer="1"/>
+<wire x1="116.078" y1="20.066" x2="116.078" y2="21.336" width="0.254" layer="1"/>
+<wire x1="116.078" y1="21.336" x2="118.364" y2="23.622" width="0.254" layer="1"/>
+<wire x1="118.364" y1="23.622" x2="118.364" y2="39.116" width="0.254" layer="1"/>
+<wire x1="118.364" y1="39.116" x2="120.65" y2="41.402" width="0.254" layer="1"/>
+<wire x1="120.65" y1="41.402" x2="120.904" y2="41.402" width="0.254" layer="1"/>
+<wire x1="120.904" y1="41.402" x2="123.444" y2="41.402" width="0.254" layer="1"/>
 </signal>
 <signal name="B_SO">
@@
 <via x="108.458" y="12.954" extent="1-16" drill="0.6"/>
 <wire x1="109.982" y1="14.478" x2="113.792" y2="14.478" width="0.254" layer="1"/>
-<wire x1="113.792" y1="14.478" x2="119.126" y2="19.812" width="0.254" layer="1"/>
-<wire x1="119.126" y1="19.812" x2="119.126" y2="41.402" width="0.254" layer="1"/>
-<wire x1="119.126" y1="41.402" x2="120.396" y2="42.672" width="0.254" layer="1"/>
+<wire x1="113.792" y1="14.478" x2="115.316" y2="16.002" width="0.254" layer="1"/>
+<wire x1="115.316" y1="16.002" x2="115.316" y2="21.336" width="0.254" layer="1"/>
+<wire x1="117.856" y1="23.876" x2="117.856" y2="42.418" width="0.254" layer="1"/>
+<wire x1="117.856" y1="42.418" x2="119.38" y2="43.942" width="0.254" layer="1"/>
+<wire x1="119.38" y1="43.942" x2="120.904" y2="43.942" width="0.254" layer="1"/>
+<wire x1="115.316" y1="21.336" x2="117.856" y2="23.876" width="0.254" layer="1"/>
 </signal>
 <signal name="N$9">
@@
 <wire x1="113.284" y1="13.716" x2="112.268" y2="12.7" width="0.254" layer="16"/>
 <via x="112.268" y="12.7" extent="1-16" drill="0.6"/>
-<wire x1="115.824" y1="21.59" x2="115.062" y2="20.828" width="0.254" layer="1"/>
-<wire x1="115.062" y1="20.828" x2="115.062" y2="18.796" width="0.254" layer="1"/>
-<wire x1="115.062" y1="18.796" x2="113.284" y2="17.018" width="0.254" layer="1"/>
 <via x="113.284" y="17.018" extent="1-16" drill="0.6"/>
 <wire x1="113.284" y1="17.018" x2="113.284" y2="13.716" width="0.254" layer="16"/>
-<wire x1="115.824" y1="21.59" x2="117.348" y2="21.59" width="0.254" layer="1"/>
-<wire x1="117.348" y1="21.59" x2="118.11" y2="22.352" width="0.254" layer="1"/>
-<wire x1="118.11" y1="22.352" x2="118.11" y2="45.466" width="0.254" layer="1"/>
-<wire x1="118.11" y1="45.466" x2="120.396" y2="47.752" width="0.254" layer="1"/>
+<wire x1="113.284" y1="17.018" x2="114.554" y2="18.288" width="0.254" layer="1"/>
+<wire x1="114.554" y1="18.288" x2="114.554" y2="21.336" width="0.254" layer="1"/>
+<wire x1="116.84" y1="23.622" x2="116.84" y2="32.258" width="0.254" layer="1"/>
+<via x="116.84" y="32.258" extent="1-16" drill="0.3302"/>
+<wire x1="116.84" y1="32.258" x2="116.84" y2="34.798" width="0.254" layer="16"/>
+<wire x1="116.84" y1="34.798" x2="120.904" y2="38.862" width="0.254" layer="16"/>
+<wire x1="116.84" y1="23.622" x2="114.554" y2="21.336" width="0.254" layer="1"/>
 </signal>
 <signal name="B_RC1">
@@
 <wire x1="121.158" y1="13.97" x2="121.158" y2="16.51" width="0.254" layer="16"/>
 <wire x1="121.158" y1="16.51" x2="121.666" y2="17.018" width="0.254" layer="16"/>
-<wire x1="119.634" y1="49.276" x2="122.174" y2="49.276" width="0.254" layer="16"/>
-<wire x1="122.174" y1="49.276" x2="122.936" y2="48.514" width="0.254" layer="16"/>
-<wire x1="122.936" y1="48.514" x2="122.936" y2="47.752" width="0.254" layer="16"/>
 <wire x1="121.666" y1="17.018" x2="121.666" y2="20.32" width="0.254" layer="16"/>
 <wire x1="121.666" y1="20.32" x2="117.856" y2="24.13" width="0.254" layer="16"/>
-<wire x1="117.856" y1="24.13" x2="117.856" y2="47.498" width="0.254" layer="16"/>
-<wire x1="117.856" y1="47.498" x2="119.634" y2="49.276" width="0.254" layer="16"/>
+<wire x1="117.856" y1="24.13" x2="117.856" y2="29.718" width="0.254" layer="16"/>
+<wire x1="123.444" y1="38.862" x2="123.444" y2="35.306" width="0.254" layer="16"/>
+<wire x1="123.444" y1="35.306" x2="117.856" y2="29.718" width="0.254" layer="16"/>
 </signal>
 <signal name="N$10">
