File: eagle/mutebox/mutebox.sch (EAGLE design)
At the start: 39 parts

Commit message: mutebox
Parts:
- added C7, C8: 100nF, microbuilder:CAP_CERAMIC0603
- added IC1: 74HCT595D, 74xx-eu:74HCT595D
- added IC2: 74HC165D, 74xx-eu:74HC165D
- added JP4: (no value), pinhead:PINHD-2X6
- added JP5: (no value), microbuilder:HEADER-1X3ROUND
- added R17, R18, R19, R20, R21, R22, R23, R24: 220, microbuilder:RESISTOR_0603
- added R25, R26, R27, R28, R29, R30, R31, R32: 10K, microbuilder:RESISTOR_0603
- JP1: device pinhead:PINHD-2X10 -> pinhead:PINHD-2X6
Connections:
- removed net P10-: JP1.12
- removed net P11-: JP1.13
- removed net P12-: JP1.14
- removed net P13-: JP1.15
- removed net P14-: JP1.16
- removed net P15-: JP1.17
- removed net P16-: JP1.18
- removed net P9-: JP1.11
- new net B_LED1: IC1A.QA, R17.1
- new net B_LED2: IC1A.QB, R18.1
- new net B_LED3: IC1A.QC, R19.1
- new net B_LED4: IC1A.QD, R20.1
- new net B_LED5: IC1A.QE, R21.1
- new net B_LED6: IC1A.QF, R22.1
- new net B_LED7: IC1A.QG, R23.1
- new net B_LED8: IC1A.QH, R24.1
- new net B_PB1: IC2A.H, R25.1, U$1.SW2
- new net B_PB2: IC2A.G, R26.1, U$2.SW2
- new net B_PB3: IC2A.F, R27.1, U$3.SW2
- new net B_PB4: IC2A.E, R28.1, U$4.SW2
- new net B_PB5: IC2A.D, R29.1, U$5.SW2
- new net B_PB6: IC2A.C, R30.1, U$6.SW2
- new net B_PB7: IC2A.B, R31.1, U$7.SW2
- new net B_PB8: IC2A.A, R32.1, U$8.SW2
- new net B_RC: IC1A.RCK, IC2A.SH/!LD, JP5.2
- new net B_RC_1: JP1.7, JP1.8, JP5.1
- new net B_RC_2: JP1.10, JP1.9, JP5.3
- new net B_SC: IC1A.SCK, IC2A.CLK, JP1.5, JP1.6
- new net B_SO: IC1A.SER, JP1.3, JP1.4
- new net GND: C7.P$1, C8.P$1, IC1A.G, IC1P.GND, IC2A.INH, IC2P.GND, JP1.11, JP1.12, U$1.LED-, U$1.SW1, U$2.LED-, U$2.SW1, U$3.LED-, U$3.SW1, U$4.LED-, U$4.SW1, U$5.LED-, U$5.SW1, U$6.LED-, U$6.SW1, U$7.LED-, U$7.SW1, U$8.LED-, U$8.SW1
- new net N$1: R17.2, U$1.LED+
- new net N$2: R18.2, U$2.LED+
- new net N$3: R19.2, U$3.LED+
- new net N$4: R20.2, U$4.LED+
- new net N$5: R21.2, U$5.LED+
- new net N$6: R22.2, U$6.LED+
- new net N$7: R23.2, U$7.LED+
- new net N$8: R24.2, U$8.LED+
- new net N$9: IC1A.QH*, IC2A.QH
- new net VCC: C7.P$2, C8.P$2, IC1A.SCL, IC1P.VCC, IC2P.VCC, JP1.1, JP1.2, R25.2, R26.2, R27.2, R28.2, R29.2, R30.2, R31.2, R32.2
- net AGND: now also JP4.11, JP4.12; no longer JP1.19, JP1.20
- net AVCC: now also JP4.1, JP4.2; no longer JP1.1, JP1.2
- net P_CLK: now also JP4.10, JP4.9; no longer JP1.10, JP1.9
- net P_CS1: now also JP4.4; no longer JP1.3
- net P_CS2: now also JP4.3; no longer JP1.4
- net P_CS3: now also JP4.6; no longer JP1.5
- net P_CS4: now also JP4.5; no longer JP1.6
- net P_DIN: now also JP4.8; no longer JP1.7
- net P_DOUT: now also JP4.7; no longer JP1.8

Commit message: mutebox
Parts:
- removed JP5: (no value), microbuilder:HEADER-1X3ROUND
Connections:
- removed net B_RC_1: JP1.7, JP1.8, JP5.1
- removed net B_RC_2: JP1.10, JP1.9, JP5.3
- removed net N$9: IC1A.QH*, IC2A.QH
- new net B_SI: IC2A.QH, JP1.10, JP1.9
- net B_LED1: now also IC1A.QE; no longer IC1A.QA
- net B_LED2: now also IC1A.QD; no longer IC1A.QB
- net B_LED4: now also IC1A.QB; no longer IC1A.QD
- net B_LED5: now also IC1A.QA; no longer IC1A.QE
- net B_PB3: now also IC2A.E; no longer IC2A.F
- net B_PB4: now also IC2A.F; no longer IC2A.E
- net B_RC: now also JP1.7, JP1.8; no longer JP5.2
Changed lines of the file:
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@@
 <part name="U$77" library="microbuilder" deviceset="GND" device=""/>
 <part name="P+12" library="microbuilder" deviceset="VCC" device=""/>
-<part name="JP5" library="microbuilder" deviceset="HEADER-1X3" device="ROUND"/>
 </parts>
 <sheets>
@@
 <instance part="U$77" gate="G$1" x="144.78" y="45.72"/>
 <instance part="P+12" gate="VCC" x="144.78" y="76.2"/>
-<instance part="JP5" gate="A" x="119.38" y="50.8" rot="R90"/>
 </instances>
 <busses>
@@
 </segment>
 <segment>
+<pinref part="IC1" gate="A" pin="QE"/>
+<wire x1="15.24" y1="58.42" x2="7.62" y2="58.42" width="0.1524" layer="91"/>
+<label x="5.08" y="58.42" size="1.778" layer="95"/>
+</segment>
+</net>
+<net name="B_LED2" class="0">
+<segment>
+<pinref part="R18" gate="G$1" pin="1"/>
+<wire x1="38.1" y1="-15.24" x2="38.1" y2="-20.32" width="0.1524" layer="91"/>
+<label x="38.1" y="-20.32" size="1.778" layer="95"/>
+</segment>
+<segment>
+<pinref part="IC1" gate="A" pin="QD"/>
+<wire x1="15.24" y1="55.88" x2="7.62" y2="55.88" width="0.1524" layer="91"/>
+<label x="5.08" y="55.88" size="1.778" layer="95"/>
+</segment>
+</net>
+<net name="B_LED3" class="0">
+<segment>
+<pinref part="R19" gate="G$1" pin="1"/>
+<wire x1="63.5" y1="-15.24" x2="63.5" y2="-20.32" width="0.1524" layer="91"/>
+<label x="63.5" y="-20.32" size="1.778" layer="95"/>
+</segment>
+<segment>
+<pinref part="IC1" gate="A" pin="QC"/>
+<wire x1="15.24" y1="53.34" x2="7.62" y2="53.34" width="0.1524" layer="91"/>
+<label x="5.08" y="53.34" size="1.778" layer="95"/>
+</segment>
+</net>
+<net name="B_LED4" class="0">
+<segment>
+<pinref part="R20" gate="G$1" pin="1"/>
+<wire x1="91.44" y1="-15.24" x2="91.44" y2="-20.32" width="0.1524" layer="91"/>
+<label x="91.44" y="-20.32" size="1.778" layer="95"/>
+</segment>
+<segment>
+<pinref part="IC1" gate="A" pin="QB"/>
+<wire x1="15.24" y1="50.8" x2="7.62" y2="50.8" width="0.1524" layer="91"/>
+<label x="5.08" y="50.8" size="1.778" layer="95"/>
+</segment>
+</net>
+<net name="B_LED5" class="0">
+<segment>
+<pinref part="R21" gate="G$1" pin="1"/>
+<wire x1="119.38" y1="-15.24" x2="119.38" y2="-20.32" width="0.1524" layer="91"/>
+<label x="119.38" y="-20.32" size="1.778" layer="95"/>
+</segment>
+<segment>
 <pinref part="IC1" gate="A" pin="QA"/>
 <wire x1="15.24" y1="48.26" x2="7.62" y2="48.26" width="0.1524" layer="91"/>
 <label x="5.08" y="48.26" size="1.778" layer="95"/>
-</segment>
-</net>
-<net name="B_LED2" class="0">
-<segment>
-<pinref part="R18" gate="G$1" pin="1"/>
-<wire x1="38.1" y1="-15.24" x2="38.1" y2="-20.32" width="0.1524" layer="91"/>
-<label x="38.1" y="-20.32" size="1.778" layer="95"/>
-</segment>
-<segment>
-<pinref part="IC1" gate="A" pin="QB"/>
-<wire x1="15.24" y1="50.8" x2="7.62" y2="50.8" width="0.1524" layer="91"/>
-<label x="5.08" y="50.8" size="1.778" layer="95"/>
-</segment>
-</net>
-<net name="B_LED3" class="0">
-<segment>
-<pinref part="R19" gate="G$1" pin="1"/>
-<wire x1="63.5" y1="-15.24" x2="63.5" y2="-20.32" width="0.1524" layer="91"/>
-<label x="63.5" y="-20.32" size="1.778" layer="95"/>
-</segment>
-<segment>
-<pinref part="IC1" gate="A" pin="QC"/>
-<wire x1="15.24" y1="53.34" x2="7.62" y2="53.34" width="0.1524" layer="91"/>
-<label x="5.08" y="53.34" size="1.778" layer="95"/>
-</segment>
-</net>
-<net name="B_LED4" class="0">
-<segment>
-<pinref part="R20" gate="G$1" pin="1"/>
-<wire x1="91.44" y1="-15.24" x2="91.44" y2="-20.32" width="0.1524" layer="91"/>
-<label x="91.44" y="-20.32" size="1.778" layer="95"/>
-</segment>
-<segment>
-<pinref part="IC1" gate="A" pin="QD"/>
-<wire x1="15.24" y1="55.88" x2="7.62" y2="55.88" width="0.1524" layer="91"/>
-<label x="5.08" y="55.88" size="1.778" layer="95"/>
-</segment>
-</net>
-<net name="B_LED5" class="0">
-<segment>
-<pinref part="R21" gate="G$1" pin="1"/>
-<wire x1="119.38" y1="-15.24" x2="119.38" y2="-20.32" width="0.1524" layer="91"/>
-<label x="119.38" y="-20.32" size="1.778" layer="95"/>
-</segment>
-<segment>
-<pinref part="IC1" gate="A" pin="QE"/>
-<wire x1="15.24" y1="58.42" x2="7.62" y2="58.42" width="0.1524" layer="91"/>
-<label x="5.08" y="58.42" size="1.778" layer="95"/>
 </segment>
 </net>
@@
 </segment>
 <segment>
-<pinref part="IC2" gate="A" pin="F"/>
-<wire x1="88.9" y1="58.42" x2="81.28" y2="58.42" width="0.1524" layer="91"/>
-<label x="78.74" y="58.42" size="1.778" layer="95"/>
+<pinref part="IC2" gate="A" pin="E"/>
+<wire x1="88.9" y1="60.96" x2="81.28" y2="60.96" width="0.1524" layer="91"/>
+<label x="78.74" y="60.96" size="1.778" layer="95"/>
 </segment>
 </net>
@@
 </segment>
 <segment>
-<pinref part="IC2" gate="A" pin="E"/>
-<wire x1="88.9" y1="60.96" x2="81.28" y2="60.96" width="0.1524" layer="91"/>
-<label x="78.74" y="60.96" size="1.778" layer="95"/>
+<pinref part="IC2" gate="A" pin="F"/>
+<wire x1="88.9" y1="58.42" x2="81.28" y2="58.42" width="0.1524" layer="91"/>
+<label x="78.74" y="58.42" size="1.778" layer="95"/>
 </segment>
 </net>
@@
 </segment>
 </net>
-<net name="B_RC_2" class="0">
+<net name="B_SI" class="0">
+<segment>
+<pinref part="IC2" gate="A" pin="QH"/>
+<wire x1="114.3" y1="71.12" x2="119.38" y2="71.12" width="0.1524" layer="91"/>
+<label x="116.84" y="71.12" size="1.778" layer="95"/>
+</segment>
 <segment>
 <pinref part="JP1" gate="A" pin="9"/>
 <wire x1="144.78" y1="55.88" x2="134.62" y2="55.88" width="0.1524" layer="91"/>
-<label x="134.62" y="55.88" size="1.778" layer="95"/>
+<label x="132.08" y="55.88" size="1.778" layer="95"/>
 <pinref part="JP1" gate="A" pin="10"/>
 <wire x1="152.4" y1="55.88" x2="144.78" y2="55.88" width="0.1524" layer="91"/>
 <junction x="144.78" y="55.88"/>
 </segment>
-<segment>
-<pinref part="JP5" gate="A" pin="3"/>
-<wire x1="121.92" y1="48.26" x2="121.92" y2="38.1" width="0.1524" layer="91"/>
-<label x="121.92" y="33.02" size="1.778" layer="95" rot="R90"/>
-</segment>
-</net>
-<net name="N$9" class="0">
-<segment>
-<pinref part="IC1" gate="A" pin="QH*"/>
-<wire x1="15.24" y1="71.12" x2="12.7" y2="71.12" width="0.1524" layer="91"/>
-<wire x1="12.7" y1="71.12" x2="12.7" y2="81.28" width="0.1524" layer="91"/>
-<wire x1="12.7" y1="81.28" x2="116.84" y2="81.28" width="0.1524" layer="91"/>
-<wire x1="116.84" y1="81.28" x2="116.84" y2="71.12" width="0.1524" layer="91"/>
-<pinref part="IC2" gate="A" pin="QH"/>
-<wire x1="116.84" y1="71.12" x2="114.3" y2="71.12" width="0.1524" layer="91"/>
-</segment>
 </net>
 <net name="B_SC" class="0">
@@
 </segment>
 <segment>
+<pinref part="IC1" gate="A" pin="SCK"/>
+<wire x1="40.64" y1="53.34" x2="48.26" y2="53.34" width="0.1524" layer="91"/>
+<label x="45.72" y="53.34" size="1.778" layer="95"/>
+</segment>
+<segment>
 <pinref part="JP1" gate="A" pin="5"/>
 <wire x1="144.78" y1="60.96" x2="134.62" y2="60.96" width="0.1524" layer="91"/>
-<label x="134.62" y="60.96" size="1.778" layer="95"/>
+<label x="132.08" y="60.96" size="1.778" layer="95"/>
 <pinref part="JP1" gate="A" pin="6"/>
 <wire x1="152.4" y1="60.96" x2="144.78" y2="60.96" width="0.1524" layer="91"/>
 <junction x="144.78" y="60.96"/>
 </segment>
-<segment>
-<pinref part="IC1" gate="A" pin="SCK"/>
-<wire x1="40.64" y1="53.34" x2="48.26" y2="53.34" width="0.1524" layer="91"/>
-<label x="45.72" y="53.34" size="1.778" layer="95"/>
-</segment>
 </net>
 <net name="B_SO" class="0">
@@
 <pinref part="JP1" gate="A" pin="3"/>
 <wire x1="144.78" y1="63.5" x2="134.62" y2="63.5" width="0.1524" layer="91"/>
-<label x="134.62" y="63.5" size="1.778" layer="95"/>
+<label x="132.08" y="63.5" size="1.778" layer="95"/>
 <pinref part="JP1" gate="A" pin="4"/>
 <wire x1="152.4" y1="63.5" x2="144.78" y2="63.5" width="0.1524" layer="91"/>
@@
 </segment>
 <segment>
-<pinref part="JP5" gate="A" pin="2"/>
-<wire x1="119.38" y1="48.26" x2="119.38" y2="38.1" width="0.1524" layer="91"/>
-<label x="119.38" y="33.02" size="1.778" layer="95" rot="R90"/>
-</segment>
-</net>
-<net name="B_RC_1" class="0">
-<segment>
 <pinref part="JP1" gate="A" pin="7"/>
 <wire x1="144.78" y1="58.42" x2="134.62" y2="58.42" width="0.1524" layer="91"/>
-<label x="134.62" y="58.42" size="1.778" layer="95"/>
+<label x="132.08" y="58.42" size="1.778" layer="95"/>
 <pinref part="JP1" gate="A" pin="8"/>
 <wire x1="152.4" y1="58.42" x2="144.78" y2="58.42" width="0.1524" layer="91"/>
 <junction x="144.78" y="58.42"/>
 </segment>
-<segment>
-<pinref part="JP5" gate="A" pin="1"/>
-<wire x1="116.84" y1="48.26" x2="116.84" y2="38.1" width="0.1524" layer="91"/>
-<label x="116.84" y="33.02" size="1.778" layer="95" rot="R90"/>
-</segment>
-</net>
+</net>

Commit message: mutebox
Parts:
- removed JP2, JP3: (no value), microbuilder:HEADER-1X3ROUND
Connections:
- removed net P_CS3: JP3.1, JP4.6
- removed net P_CS4: JP3.3, JP4.5
- removed net P_CS_A: JP2.2, U$29.!CS
- removed net P_CS_B: JP3.2, U$47.!CS
- net P_CLK: now also JP4.7, JP4.8; no longer JP4.10, JP4.9
- net P_CS1: now also U$29.!CS; no longer JP2.1
- net P_CS2: now also U$47.!CS; no longer JP2.3
- net P_DIN: now also JP4.6; no longer JP4.8
- net P_DOUT: now also JP4.5; no longer JP4.7
Changed lines of the file:
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@@
 <part name="U$50" library="microbuilder" deviceset="AVCC" device=""/>
 <part name="U$51" library="microbuilder" deviceset="AGND" device=""/>
-<part name="JP2" library="microbuilder" deviceset="HEADER-1X3" device="ROUND"/>
-<part name="JP3" library="microbuilder" deviceset="HEADER-1X3" device="ROUND"/>
 <part name="U$29" library="MCP3208" deviceset="21298E" device=""/>
 <part name="C1" library="microbuilder" deviceset="CAP_CERAMIC" device="0603" value="100nF"/>
@@
 <instance part="U$50" gate="G$1" x="121.92" y="10.16"/>
 <instance part="U$51" gate="G$1" x="116.84" y="17.78" rot="R90"/>
-<instance part="JP2" gate="A" x="33.02" y="55.88" rot="R90"/>
-<instance part="JP3" gate="A" x="48.26" y="55.88" rot="R90"/>
 <instance part="U$29" gate="G$1" x="93.98" y="63.5" rot="R270"/>
 <instance part="C1" gate="G$1" x="124.46" y="55.88"/>
@@
 </segment>
 <segment>
-<pinref part="JP2" gate="A" pin="1"/>
-<wire x1="30.48" y1="53.34" x2="30.48" y2="45.72" width="0.1524" layer="91"/>
-<label x="30.48" y="40.64" size="1.778" layer="95" rot="R90"/>
+<pinref part="U$29" gate="G$1" pin="!CS"/>
+<wire x1="78.74" y1="66.04" x2="71.12" y2="66.04" width="0.1524" layer="91"/>
+<label x="68.58" y="66.04" size="1.778" layer="95"/>
 </segment>
 </net>
@@
 </segment>
 <segment>
+<pinref part="U$29" gate="G$1" pin="DIN"/>
+<wire x1="78.74" y1="60.96" x2="71.12" y2="60.96" width="0.1524" layer="91"/>
+<label x="68.58" y="60.96" size="1.778" layer="95"/>
+</segment>
+<segment>
+<wire x1="25.4" y1="17.78" x2="38.1" y2="17.78" width="0.1524" layer="91"/>
+<label x="35.56" y="17.78" size="1.778" layer="95"/>
+<pinref part="JP4" gate="A" pin="6"/>
+</segment>
+</net>
+<net name="P_CLK" class="0">
+<segment>
+<pinref part="U$47" gate="G$1" pin="CLK"/>
+<wire x1="78.74" y1="7.62" x2="71.12" y2="7.62" width="0.1524" layer="91"/>
+<label x="68.58" y="7.62" size="1.778" layer="95"/>
+</segment>
+<segment>
+<pinref part="U$29" gate="G$1" pin="CLK"/>
+<wire x1="78.74" y1="55.88" x2="71.12" y2="55.88" width="0.1524" layer="91"/>
+<label x="68.58" y="55.88" size="1.778" layer="95"/>
+</segment>
+<segment>
+<wire x1="2.54" y1="15.24" x2="17.78" y2="15.24" width="0.1524" layer="91"/>
+<label x="2.54" y="15.24" size="1.778" layer="95"/>
+<pinref part="JP4" gate="A" pin="7"/>
+</segment>
+<segment>
 <wire x1="38.1" y1="15.24" x2="25.4" y2="15.24" width="0.1524" layer="91"/>
 <label x="35.56" y="15.24" size="1.778" layer="95"/>
 <pinref part="JP4" gate="A" pin="8"/>
 </segment>
-<segment>
-<pinref part="U$29" gate="G$1" pin="DIN"/>
-<wire x1="78.74" y1="60.96" x2="71.12" y2="60.96" width="0.1524" layer="91"/>
-<label x="68.58" y="60.96" size="1.778" layer="95"/>
-</segment>
-</net>
-<net name="P_CLK" class="0">
-<segment>
-<pinref part="U$47" gate="G$1" pin="CLK"/>
-<wire x1="78.74" y1="7.62" x2="71.12" y2="7.62" width="0.1524" layer="91"/>
-<label x="68.58" y="7.62" size="1.778" layer="95"/>
-</segment>
-<segment>
-<wire x1="38.1" y1="12.7" x2="25.4" y2="12.7" width="0.1524" layer="91"/>
-<label x="35.56" y="12.7" size="1.778" layer="95"/>
-<pinref part="JP4" gate="A" pin="10"/>
-</segment>
-<segment>
-<wire x1="17.78" y1="12.7" x2="2.54" y2="12.7" width="0.1524" layer="91"/>
-<label x="2.54" y="12.7" size="1.778" layer="95"/>
-<pinref part="JP4" gate="A" pin="9"/>
-</segment>
-<segment>
-<pinref part="U$29" gate="G$1" pin="CLK"/>
-<wire x1="78.74" y1="55.88" x2="71.12" y2="55.88" width="0.1524" layer="91"/>
-<label x="68.58" y="55.88" size="1.778" layer="95"/>
-</segment>
 </net>
 <net name="P_DOUT" class="0">
@@
 </segment>
 <segment>
-<wire x1="2.54" y1="15.24" x2="17.78" y2="15.24" width="0.1524" layer="91"/>
-<label x="2.54" y="15.24" size="1.778" layer="95"/>
-<pinref part="JP4" gate="A" pin="7"/>
-</segment>
-<segment>
 <pinref part="U$29" gate="G$1" pin="DOUT"/>
 <wire x1="78.74" y1="50.8" x2="71.12" y2="50.8" width="0.1524" layer="91"/>
 <label x="68.58" y="50.8" size="1.778" layer="95"/>
 </segment>
+<segment>
+<wire x1="17.78" y1="17.78" x2="2.54" y2="17.78" width="0.1524" layer="91"/>
+<label x="2.54" y="17.78" size="1.778" layer="95"/>
+<pinref part="JP4" gate="A" pin="5"/>
+</segment>
 </net>
 <net name="P_CS2" class="0">
@@
 </segment>
 <segment>
-<pinref part="JP2" gate="A" pin="3"/>
-<wire x1="35.56" y1="53.34" x2="35.56" y2="45.72" width="0.1524" layer="91"/>
-<label x="35.56" y="40.64" size="1.778" layer="95" rot="R90"/>
-</segment>
-</net>
-<net name="P_CS3" class="0">
-<segment>
-<wire x1="25.4" y1="17.78" x2="38.1" y2="17.78" width="0.1524" layer="91"/>
-<label x="35.56" y="17.78" size="1.778" layer="95"/>
-<pinref part="JP4" gate="A" pin="6"/>
-</segment>
-<segment>
-<pinref part="JP3" gate="A" pin="1"/>
-<wire x1="45.72" y1="53.34" x2="45.72" y2="45.72" width="0.1524" layer="91"/>
-<label x="45.72" y="40.64" size="1.778" layer="95" rot="R90"/>
-</segment>
-</net>
-<net name="P_CS4" class="0">
-<segment>
-<wire x1="17.78" y1="17.78" x2="2.54" y2="17.78" width="0.1524" layer="91"/>
-<label x="2.54" y="17.78" size="1.778" layer="95"/>
-<pinref part="JP4" gate="A" pin="5"/>
-</segment>
-<segment>
-<pinref part="JP3" gate="A" pin="3"/>
-<wire x1="50.8" y1="53.34" x2="50.8" y2="45.72" width="0.1524" layer="91"/>
-<label x="50.8" y="40.64" size="1.778" layer="95" rot="R90"/>
-</segment>
-</net>
-<net name="P_CS_A" class="0">
-<segment>
-<pinref part="JP2" gate="A" pin="2"/>
-<wire x1="33.02" y1="53.34" x2="33.02" y2="45.72" width="0.1524" layer="91"/>
-<label x="33.02" y="38.1" size="1.778" layer="95" rot="R90"/>
-</segment>
-<segment>
-<pinref part="U$29" gate="G$1" pin="!CS"/>
-<wire x1="78.74" y1="66.04" x2="71.12" y2="66.04" width="0.1524" layer="91"/>
-<label x="68.58" y="66.04" size="1.778" layer="95"/>
-</segment>
-</net>
-<net name="P_CS_B" class="0">
-<segment>
-<pinref part="JP3" gate="A" pin="2"/>
-<wire x1="48.26" y1="53.34" x2="48.26" y2="45.72" width="0.1524" layer="91"/>
-<label x="48.26" y="38.1" size="1.778" layer="95" rot="R90"/>
-</segment>
-<segment>
