File: eagle/mutebox/mutebox.sch (EAGLE design)
At the start: 60 parts, among them IC1 74HCT595D, IC2 74HC165D, IC3 MCP3208, IC4 MCP3208

Commit message: mutebox rearrange buttons
Parts:
- B_CONN, P_CONN: device microbuilder:HEADER-2X5 -> con-harting-ml:ML10
Changed lines of the file:
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@@
 <part name="U$9" library="microbuilder" deviceset="AGND" device=""/>
 <part name="U$10" library="microbuilder" deviceset="AGND" device=""/>
-<part name="P_CONN" library="microbuilder" deviceset="HEADER-2X5" device=""/>
+<part name="P_CONN" library="con-harting-ml" deviceset="ML10" device=""/>
 <part name="R33" library="microbuilder" deviceset="RESISTOR" device="_0805" value="10"/>
 <part name="U$27" library="microbuilder" deviceset="AVCC" device=""/>
-<part name="B_CONN" library="microbuilder" deviceset="HEADER-2X5" device=""/>
+<part name="B_CONN" library="con-harting-ml" deviceset="ML10" device=""/>
 <part name="U$28" library="microbuilder" deviceset="GND" device=""/>
 <part name="U$78" library="microbuilder" deviceset="GND" device=""/>
@@
 <instance part="U$9" gate="G$1" x="-2.54" y="22.86" rot="R270"/>
 <instance part="U$10" gate="G$1" x="40.64" y="22.86" rot="R90"/>
-<instance part="P_CONN" gate="A" x="20.32" y="17.78"/>
+<instance part="P_CONN" gate="G$1" x="20.32" y="17.78" rot="R180"/>
 <instance part="R33" gate="G$1" x="48.26" y="20.32"/>
 <instance part="U$27" gate="G$1" x="58.42" y="20.32" rot="R270"/>
@@
 </segment>
 <segment>
-<wire x1="0" y1="22.86" x2="17.78" y2="22.86" width="0.1524" layer="91"/>
+<wire x1="0" y1="22.86" x2="12.7" y2="22.86" width="0.1524" layer="91"/>
 <pinref part="U$9" gate="G$1" pin="AGND"/>
-<pinref part="P_CONN" gate="A" pin="1"/>
-</segment>
-<segment>
-<wire x1="38.1" y1="22.86" x2="25.4" y2="22.86" width="0.1524" layer="91"/>
+<pinref part="P_CONN" gate="G$1" pin="1"/>
+</segment>
+<segment>
+<wire x1="38.1" y1="22.86" x2="27.94" y2="22.86" width="0.1524" layer="91"/>
 <pinref part="U$10" gate="G$1" pin="AGND"/>
-<pinref part="P_CONN" gate="A" pin="2"/>
+<pinref part="P_CONN" gate="G$1" pin="2"/>
 </segment>
 </net>
@@
 </segment>
 <segment>
-<pinref part="P_CONN" gate="A" pin="10"/>
-<wire x1="25.4" y1="12.7" x2="35.56" y2="12.7" width="0.1524" layer="91"/>
+<pinref part="P_CONN" gate="G$1" pin="10"/>
+<wire x1="27.94" y1="12.7" x2="35.56" y2="12.7" width="0.1524" layer="91"/>
 <label x="33.02" y="12.7" size="1.778" layer="95"/>
 </segment>
@@
 </segment>
 <segment>
-<pinref part="P_CONN" gate="A" pin="6"/>
-<wire x1="25.4" y1="17.78" x2="35.56" y2="17.78" width="0.1524" layer="91"/>
+<pinref part="P_CONN" gate="G$1" pin="6"/>
+<wire x1="27.94" y1="17.78" x2="35.56" y2="17.78" width="0.1524" layer="91"/>
 <label x="33.02" y="17.78" size="1.778" layer="95"/>
 </segment>
@@
 </segment>
 <segment>
-<pinref part="P_CONN" gate="A" pin="7"/>
-<wire x1="7.62" y1="15.24" x2="17.78" y2="15.24" width="0.1524" layer="91"/>
+<pinref part="P_CONN" gate="G$1" pin="7"/>
+<wire x1="7.62" y1="15.24" x2="12.7" y2="15.24" width="0.1524" layer="91"/>
 <label x="2.54" y="15.24" size="1.778" layer="95"/>
 </segment>
 <segment>
-<pinref part="P_CONN" gate="A" pin="8"/>
-<wire x1="25.4" y1="15.24" x2="35.56" y2="15.24" width="0.1524" layer="91"/>
+<pinref part="P_CONN" gate="G$1" pin="8"/>
+<wire x1="27.94" y1="15.24" x2="35.56" y2="15.24" width="0.1524" layer="91"/>
 <label x="33.02" y="15.24" size="1.778" layer="95"/>
 </segment>
@@
 </segment>
 <segment>
-<pinref part="P_CONN" gate="A" pin="5"/>
-<wire x1="17.78" y1="17.78" x2="7.62" y2="17.78" width="0.1524" layer="91"/>
+<pinref part="P_CONN" gate="G$1" pin="5"/>
+<wire x1="12.7" y1="17.78" x2="7.62" y2="17.78" width="0.1524" layer="91"/>
 <label x="2.54" y="17.78" size="1.778" layer="95"/>
 </segment>
@@
 </segment>
 <segment>
-<pinref part="P_CONN" gate="A" pin="9"/>
-<wire x1="17.78" y1="12.7" x2="7.62" y2="12.7" width="0.1524" layer="91"/>
+<pinref part="P_CONN" gate="G$1" pin="9"/>
+<wire x1="12.7" y1="12.7" x2="7.62" y2="12.7" width="0.1524" layer="91"/>
 <label x="2.54" y="12.7" size="1.778" layer="95"/>
 </segment>
@@
 <segment>
 <pinref part="R33" gate="G$1" pin="1"/>
-<wire x1="43.18" y1="20.32" x2="25.4" y2="20.32" width="0.1524" layer="91"/>
-<pinref part="P_CONN" gate="A" pin="4"/>
-<pinref part="P_CONN" gate="A" pin="3"/>
-<wire x1="17.78" y1="20.32" x2="25.4" y2="20.32" width="0.1524" layer="91"/>
-<junction x="25.4" y="20.32"/>
+<wire x1="43.18" y1="20.32" x2="27.94" y2="20.32" width="0.1524" layer="91"/>
+<pinref part="P_CONN" gate="G$1" pin="4"/>
+<pinref part="P_CONN" gate="G$1" pin="3"/>
+<wire x1="12.7" y1="20.32" x2="27.94" y2="20.32" width="0.1524" layer="91"/>
+<junction x="27.94" y="20.32"/>
 </segment>
 </net>
@@
 <instance part="U$75" gate="G$1" x="38.1" y="35.56" rot="R90"/>
 <instance part="U$76" gate="G$1" x="111.76" y="30.48" rot="R90"/>
-<instance part="B_CONN" gate="A" x="182.88" y="60.96"/>
+<instance part="B_CONN" gate="G$1" x="185.42" y="60.96" rot="R180"/>
 <instance part="U$28" gate="G$1" x="195.58" y="66.04" rot="R90"/>
 <instance part="U$78" gate="G$1" x="172.72" y="66.04" rot="R270"/>
@@
 </segment>
 <segment>
-<pinref part="B_CONN" gate="A" pin="1"/>
+<pinref part="B_CONN" gate="G$1" pin="1"/>
 <pinref part="U$78" gate="G$1" pin="GND"/>
-<wire x1="180.34" y1="66.04" x2="175.26" y2="66.04" width="0.1524" layer="91"/>
+<wire x1="177.8" y1="66.04" x2="175.26" y2="66.04" width="0.1524" layer="91"/>
 </segment>
 <segment>
 <pinref part="U$28" gate="G$1" pin="GND"/>
-<pinref part="B_CONN" gate="A" pin="2"/>
-<wire x1="193.04" y1="66.04" x2="187.96" y2="66.04" width="0.1524" layer="91"/>
+<pinref part="B_CONN" gate="G$1" pin="2"/>
 </segment>
 </net>
@@
 <segment>
 <pinref part="P+13" gate="VCC" pin="VCC"/>
-<pinref part="B_CONN" gate="A" pin="3"/>
-<wire x1="175.26" y1="63.5" x2="180.34" y2="63.5" width="0.1524" layer="91"/>
+<pinref part="B_CONN" gate="G$1" pin="3"/>
+<wire x1="175.26" y1="63.5" x2="177.8" y2="63.5" width="0.1524" layer="91"/>
 </segment>
 <segment>
 <pinref part="P+14" gate="VCC" pin="VCC"/>
-<pinref part="B_CONN" gate="A" pin="4"/>
-<wire x1="193.04" y1="63.5" x2="187.96" y2="63.5" width="0.1524" layer="91"/>
+<pinref part="B_CONN" gate="G$1" pin="4"/>
 </segment>
 <segment>
@@
 </segment>
 <segment>
-<pinref part="B_CONN" gate="A" pin="5"/>
-<wire x1="180.34" y1="60.96" x2="172.72" y2="60.96" width="0.1524" layer="91"/>
+<pinref part="B_CONN" gate="G$1" pin="5"/>
+<wire x1="177.8" y1="60.96" x2="172.72" y2="60.96" width="0.1524" layer="91"/>
 <label x="170.18" y="60.96" size="1.778" layer="95"/>
 </segment>
@@
 </segment>
 <segment>
-<pinref part="B_CONN" gate="A" pin="7"/>
-<wire x1="180.34" y1="58.42" x2="172.72" y2="58.42" width="0.1524" layer="91"/>
+<pinref part="B_CONN" gate="G$1" pin="7"/>
+<wire x1="177.8" y1="58.42" x2="172.72" y2="58.42" width="0.1524" layer="91"/>
 <label x="170.18" y="58.42" size="1.778" layer="95"/>
 </segment>
 <segment>
-<pinref part="B_CONN" gate="A" pin="8"/>
-<wire x1="187.96" y1="58.42" x2="195.58" y2="58.42" width="0.1524" layer="91"/>
+<pinref part="B_CONN" gate="G$1" pin="8"/>
+<wire x1="193.04" y1="58.42" x2="195.58" y2="58.42" width="0.1524" layer="91"/>
 <label x="195.58" y="58.42" size="1.778" layer="95"/>
 </segment>
@@
 </segment>
 <segment>
-<pinref part="B_CONN" gate="A" pin="6"/>
-<wire x1="187.96" y1="60.96" x2="195.58" y2="60.96" width="0.1524" layer="91"/>
+<pinref part="B_CONN" gate="G$1" pin="6"/>
+<wire x1="193.04" y1="60.96" x2="195.58" y2="60.96" width="0.1524" layer="91"/>
 <label x="195.58" y="60.96" size="1.778" layer="95"/>
 </segment>
@@
 <net name="B_RC2" class="0">
 <segment>
-<pinref part="B_CONN" gate="A" pin="10"/>
-<wire x1="187.96" y1="55.88" x2="195.58" y2="55.88" width="0.1524" layer="91"/>
+<pinref part="B_CONN" gate="G$1" pin="10"/>
+<wire x1="193.04" y1="55.88" x2="195.58" y2="55.88" width="0.1524" layer="91"/>
 <label x="195.58" y="55.88" size="1.778" layer="95"/>
 </segment>
@@
 <net name="B_RC1" class="0">
 <segment>
-<pinref part="B_CONN" gate="A" pin="9"/>
-<wire x1="180.34" y1="55.88" x2="172.72" y2="55.88" width="0.1524" layer="91"/>
+<pinref part="B_CONN" gate="G$1" pin="9"/>
+<wire x1="177.8" y1="55.88" x2="172.72" y2="55.88" width="0.1524" layer="91"/>
 <label x="170.18" y="55.88" size="1.778" layer="95"/>
 </segment>

Commit message: wip
Parts:
- added H5, H6: MOUNT-HOLE3.2, holes:MOUNT-HOLE3.2
Changed lines of the file:
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@@
 <part name="R34" library="microbuilder" deviceset="RESISTOR" device="_0603" value="10K"/>
 <part name="P+12" library="microbuilder" deviceset="VCC" device=""/>
+<part name="H5" library="holes" deviceset="MOUNT-HOLE" device="3.2"/>
+<part name="H6" library="holes" deviceset="MOUNT-HOLE" device="3.2"/>
 </parts>
 <sheets>
@@
 <instance part="R33" gate="G$1" x="48.26" y="20.32"/>
 <instance part="U$27" gate="G$1" x="58.42" y="20.32" rot="R270"/>
+<instance part="H5" gate="G$1" x="109.22" y="-86.36"/>
+<instance part="H6" gate="G$1" x="109.22" y="-91.44"/>
 </instances>
 <busses>
