File: eagle/mutebox/main.brd (EAGLE design)
At the start: 127 x 88.9 mm, 48 parts, among them IC1 6N138S-TA1, IC2 6N138S-TA1, IC3 74HCT541DW, IC4 74HCT541DW, IC5 74HC595D, Q1 BC337

Commit message: wip
Parts:
- flipped CONN_SCS to the top
Routing:
- net SCS_D2: track 58.7 -> 66.3 mm, vias 1 -> 2
- net SCS_D4: track 95.9 -> 91.8 mm
- net SCS_D3: track 55.7 -> 52.9 mm
- net SCS_D7: track 57.2 -> 54.6 mm
- net SCS_D6: track 57.8 -> 60.3 mm, vias 2 -> 3
- net SCS_D5: track 56.8 -> 54.3 mm
- net SCS_D0: track 57.5 -> 60.0 mm
- net SCS_D1: track 56.3 -> 53.8 mm
- net 3.3V: track 143.4 -> 142.4 mm, vias 1 -> 2
Other:
- board text added: "3.3V"
- board text added: "5V"
Changed lines of the file:
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@@
 <text x="105.156" y="46.736" size="1.778" layer="22" rot="MR0">MuteBox Main PCB v1.0
 (c) Eran Rundstein, 2014</text>
+<text x="78.232" y="46.482" size="1.778" layer="22">MuteBox Main PCB v1.0
+(c) Eran Rundstein, 2014</text>
+<text x="22.352" y="24.638" size="0.762" layer="22" rot="MR0">5V</text>
+<text x="23.114" y="30.48" size="0.762" layer="22" rot="MR0">3.3V</text>
 </plain>
 <attributes>
@@
 <element name="H3" library="holes" package="3,3" value="MOUNT-HOLE3.3" x="2.54" y="2.54"/>
 <element name="H4" library="holes" package="3,3" value="MOUNT-HOLE3.3" x="124.46" y="2.54"/>
-<element name="CONN_SCS" library="con-harting-ml" package="ML10" value="" x="119.761" y="63.119" rot="MR90">
-<attribute name="OC_NEWARK" value="unknown" x="119.761" y="63.119" size="1.778" layer="28" rot="MR90" display="off"/>
-<attribute name="MPN" value="" x="119.761" y="63.119" size="1.778" layer="28" rot="MR90" display="off"/>
-<attribute name="MF" value="" x="119.761" y="63.119" size="1.778" layer="28" rot="MR90" display="off"/>
-<attribute name="OC_FARNELL" value="unknown" x="119.761" y="63.119" size="1.778" layer="28" rot="MR90" display="off"/>
+<element name="CONN_SCS" library="con-harting-ml" package="ML10" value="" x="119.761" y="63.119" rot="R90">
+<attribute name="OC_NEWARK" value="unknown" x="119.761" y="63.119" size="1.778" layer="27" rot="R90" display="off"/>
+<attribute name="MPN" value="" x="119.761" y="63.119" size="1.778" layer="27" rot="R90" display="off"/>
+<attribute name="MF" value="" x="119.761" y="63.119" size="1.778" layer="27" rot="R90" display="off"/>
+<attribute name="OC_FARNELL" value="unknown" x="119.761" y="63.119" size="1.778" layer="27" rot="R90" display="off"/>
 </element>
 <element name="U$1" library="STM32F4-DISCOVERY" package="STM32F4-DISCOVERY" value="STM32F4-DISCOVERY" x="38.608" y="55.626" rot="R180"/>
@@
 <wire x1="81.28" y1="64.77" x2="65.532" y2="64.77" width="0.1524" layer="16"/>
 <wire x1="116.967" y1="69.723" x2="92.964" y2="69.723" width="0.1524" layer="16"/>
-<wire x1="118.491" y1="68.199" x2="116.967" y2="69.723" width="0.1524" layer="16"/>
 <via x="81.28" y="64.77" extent="1-16" drill="0.3302"/>
 <via x="92.964" y="69.723" extent="1-16" drill="0.3302"/>
@@
 <wire x1="84.074" y1="64.77" x2="89.027" y2="69.723" width="0.1524" layer="1"/>
 <wire x1="89.027" y1="69.723" x2="92.964" y2="69.723" width="0.1524" layer="1"/>
+<via x="116.967" y="69.723" extent="1-16" drill="0.3302"/>
+<wire x1="116.967" y1="69.723" x2="119.507" y2="69.723" width="0.1524" layer="1"/>
+<wire x1="119.507" y1="69.723" x2="121.031" y2="68.199" width="0.1524" layer="1"/>
 </signal>
 <signal name="SCS_D5">
@@
 <wire x1="67.691" y1="62.103" x2="66.548" y2="63.246" width="0.1524" layer="16"/>
 <wire x1="90.932" y1="62.103" x2="67.691" y2="62.103" width="0.1524" layer="16"/>
-<wire x1="121.031" y1="65.659" x2="121.031" y2="65.024" width="0.1524" layer="16"/>
-<wire x1="121.031" y1="65.024" x2="120.142" y2="64.135" width="0.1524" layer="16"/>
-<wire x1="120.142" y1="64.135" x2="118.11" y2="64.135" width="0.1524" layer="16"/>
-<wire x1="118.11" y1="64.135" x2="116.332" y2="62.357" width="0.1524" layer="16"/>
-<wire x1="116.332" y1="62.357" x2="91.186" y2="62.357" width="0.1524" layer="16"/>
+<wire x1="115.824" y1="62.357" x2="91.186" y2="62.357" width="0.1524" layer="16"/>
 <wire x1="91.186" y1="62.357" x2="90.932" y2="62.103" width="0.1524" layer="16"/>
+<wire x1="118.491" y1="65.659" x2="118.491" y2="65.024" width="0.1524" layer="16"/>
+<wire x1="118.491" y1="65.024" x2="115.824" y2="62.357" width="0.1524" layer="16"/>
 </signal>
 <signal name="SCS_D4">
@@
 <wire x1="121.412" y1="59.563" x2="118.618" y2="59.563" width="0.1524" layer="16"/>
 <wire x1="122.047" y1="60.198" x2="121.412" y2="59.563" width="0.1524" layer="16"/>
-<wire x1="118.491" y1="65.659" x2="119.507" y2="66.675" width="0.1524" layer="16"/>
 <via x="79.375" y="41.783" extent="1-16" drill="0.3302"/>
 <wire x1="79.375" y1="41.783" x2="98.425" y2="41.783" width="0.1524" layer="1"/>
@@
 <wire x1="98.425" y1="41.783" x2="100.838" y2="41.783" width="0.1524" layer="16"/>
 <wire x1="63.119" y1="59.817" x2="64.008" y2="60.706" width="0.1524" layer="16"/>
-<wire x1="119.507" y1="66.675" x2="121.539" y2="66.675" width="0.1524" layer="16"/>
-<wire x1="121.539" y1="66.675" x2="122.047" y2="66.167" width="0.1524" layer="16"/>
-<wire x1="122.047" y1="66.167" x2="122.047" y2="60.198" width="0.1524" layer="16"/>
+<wire x1="122.047" y1="65.024" x2="122.047" y2="60.198" width="0.1524" layer="16"/>
 <wire x1="63.119" y1="42.037" x2="63.373" y2="41.783" width="0.1524" layer="16"/>
+<wire x1="121.031" y1="65.659" x2="121.412" y2="65.659" width="0.1524" layer="16"/>
+<wire x1="121.412" y1="65.659" x2="122.047" y2="65.024" width="0.1524" layer="16"/>
 </signal>
 <signal name="SCS_D3">
@@
 <wire x1="67.564" y1="61.722" x2="66.548" y2="60.706" width="0.1524" layer="16"/>
 <wire x1="91.313" y1="61.722" x2="67.564" y2="61.722" width="0.1524" layer="16"/>
-<wire x1="121.031" y1="63.119" x2="121.031" y2="62.738" width="0.1524" layer="16"/>
-<wire x1="121.031" y1="62.738" x2="120.269" y2="61.976" width="0.1524" layer="16"/>
-<wire x1="120.269" y1="61.976" x2="91.567" y2="61.976" width="0.1524" layer="16"/>
+<wire x1="117.348" y1="61.976" x2="91.567" y2="61.976" width="0.1524" layer="16"/>
 <wire x1="91.567" y1="61.976" x2="91.313" y2="61.722" width="0.1524" layer="16"/>
+<wire x1="118.491" y1="63.119" x2="117.348" y2="61.976" width="0.1524" layer="16"/>
 </signal>
 <signal name="SCS_D2">
@@
 <via x="102.235" y="57.023" extent="1-16" drill="0.3302"/>
 <wire x1="102.235" y1="57.023" x2="108.331" y2="63.119" width="0.1524" layer="1"/>
-<wire x1="108.331" y1="63.119" x2="118.491" y2="63.119" width="0.1524" layer="1"/>
+<via x="108.331" y="63.119" extent="1-16" drill="0.3302"/>
+<wire x1="108.331" y1="63.119" x2="115.824" y2="63.119" width="0.1524" layer="16"/>
+<wire x1="121.031" y1="63.119" x2="119.888" y2="64.262" width="0.1524" layer="16"/>
+<wire x1="119.888" y1="64.262" x2="119.888" y2="66.294" width="0.1524" layer="16"/>
+<wire x1="119.888" y1="66.294" x2="119.38" y2="66.802" width="0.1524" layer="16"/>
+<wire x1="119.38" y1="66.802" x2="118.11" y2="66.802" width="0.1524" layer="16"/>
+<wire x1="118.11" y1="66.802" x2="117.094" y2="65.786" width="0.1524" layer="16"/>
+<wire x1="117.094" y1="65.786" x2="117.094" y2="64.389" width="0.1524" layer="16"/>
+<wire x1="117.094" y1="64.389" x2="115.824" y2="63.119" width="0.1524" layer="16"/>
 </signal>
 <signal name="SCS_D1">
@@
 <wire x1="69.469" y1="61.087" x2="66.548" y2="58.166" width="0.1524" layer="16"/>
 <wire x1="91.186" y1="61.087" x2="69.469" y2="61.087" width="0.1524" layer="16"/>
-<wire x1="121.031" y1="60.579" x2="120.015" y2="61.595" width="0.1524" layer="16"/>
-<wire x1="120.015" y1="61.595" x2="91.694" y2="61.595" width="0.1524" layer="16"/>
+<wire x1="117.348" y1="61.595" x2="91.694" y2="61.595" width="0.1524" layer="16"/>
 <wire x1="91.694" y1="61.595" x2="91.186" y2="61.087" width="0.1524" layer="16"/>
+<wire x1="118.491" y1="60.579" x2="118.364" y2="60.579" width="0.1524" layer="16"/>
+<wire x1="118.364" y1="60.579" x2="117.348" y2="61.595" width="0.1524" layer="16"/>
 </signal>
 <signal name="SCS_D0">
@@
 <contactref element="U$1" pad="P$26"/>
 <wire x1="64.897" y1="56.515" x2="64.008" y2="55.626" width="0.1524" layer="16"/>
-<wire x1="114.3" y1="56.388" x2="115.8875" y2="57.9755" width="0.1524" layer="1"/>
-<wire x1="115.8875" y1="57.9755" x2="118.491" y2="60.579" width="0.1524" layer="1"/>
 <wire x1="64.897" y1="56.515" x2="74.676" y2="56.515" width="0.1524" layer="16"/>
 <wire x1="74.676" y1="56.515" x2="75.692" y2="55.499" width="0.1524" layer="16"/>
@@
 <via x="102.489" y="55.372" extent="1-16" drill="0.3302"/>
 <wire x1="102.489" y1="55.372" x2="113.284" y2="55.372" width="0.1524" layer="1"/>
-<wire x1="113.284" y1="55.372" x2="114.3" y2="56.388" width="0.1524" layer="1"/>
+<wire x1="121.031" y1="60.579" x2="119.888" y2="59.436" width="0.1524" layer="1"/>
+<wire x1="119.888" y1="59.436" x2="117.348" y2="59.436" width="0.1524" layer="1"/>
+<wire x1="117.348" y1="59.436" x2="113.284" y2="55.372" width="0.1524" layer="1"/>
 </signal>
 <signal name="SCS_D7">
 <contactref element="CONN_SCS" pad="10"/>
 <contactref element="U$1" pad="P$33"/>
-<wire x1="116.459" y1="65.024" x2="86.233" y2="65.024" width="0.1524" layer="16"/>
-<wire x1="118.618" y1="67.183" x2="116.459" y2="65.024" width="0.1524" layer="16"/>
-<wire x1="120.015" y1="67.183" x2="118.618" y2="67.183" width="0.1524" layer="16"/>
-<wire x1="121.031" y1="68.199" x2="120.015" y2="67.183" width="0.1524" layer="16"/>
+<wire x1="115.316" y1="65.024" x2="86.233" y2="65.024" width="0.1524" layer="16"/>
 <via x="75.565" y="65.532" extent="1-16" drill="0.6" shape="octagon"/>
 <wire x1="75.565" y1="65.532" x2="78.359" y2="65.532" width="0.1524" layer="1"/>
@@
 <wire x1="75.565" y1="65.532" x2="66.802" y2="65.532" width="0.1524" layer="16"/>
 <wire x1="66.802" y1="65.532" x2="66.548" y2="65.786" width="0.1524" layer="16"/>
+<wire x1="115.316" y1="65.024" x2="118.491" y2="68.199" width="0.1524" layer="16"/>
 </signal>
 <signal name="3.3V">
@@
 <contactref element="U$1" pad="P$56"/>
 <contactref element="JP2" pad="3"/>
-<wire x1="102.489" y1="39.497" x2="121.031" y2="58.039" width="0.1524" layer="16"/>
 <wire x1="92.202" y1="39.497" x2="102.489" y2="39.497" width="0.1524" layer="16"/>
 <wire x1="85.852" y1="33.147" x2="92.202" y2="39.497" width="0.1524" layer="16"/>
@@
 <via x="57.785" y="27.686" extent="1-16" drill="0.3302"/>
 <wire x1="57.785" y1="27.686" x2="39.116" y2="27.686" width="0.254" layer="16"/>
+<via x="102.489" y="39.497" extent="1-16" drill="0.3302"/>
+<wire x1="102.489" y1="39.497" x2="118.491" y2="55.499" width="0.1524" layer="1"/>
+<wire x1="118.491" y1="55.499" x2="118.491" y2="58.039" width="0.1524" layer="1"/>
 </signal>
 <signal name="LCD_D6">
@@
 </signal>
 </signals>
-<errors>
-</errors>
 </board>
 </drawing>
