File: eagle/mutebox/main.brd (EAGLE design)
At the start: 127 x 88.9 mm, 48 parts, among them IC1 6N138S-TA1, IC2 6N138S-TA1, IC3 74HCT541DW, IC4 74HCT541DW, IC5 74HC595D, Q1 BC337

Commit message: wip
Parts:
- moved B_CONN1 5.59 mm to (105.9, 5.21)
- moved P_CONN1 5.59 mm to (85.2, 5.21)
- moved U$1 1.27 mm to (39.9, 55.6)
Routing:
- net PB4: track 171.4 -> 178.6 mm
- net PB14: track 151.3 -> 145.7 mm
- net MOD1_BTN_CS1: track 45.0 -> 50.6 mm
- net MOD1_BTN_SO: track 41.7 -> 47.3 mm
- net MOD1_BTN_CS2: track 49.1 -> 54.6 mm
- net MOD1_POT_SC: track 22.0 -> 27.5 mm
- net MOD1_POT_SO: track 16.1 -> 21.7 mm
- net MOD1_POT_CS2: track 22.4 -> 28.0 mm
- net MOD1_POT_CS1: track 27.0 -> 32.6 mm
- net MOD1_BTN_SC: track 44.7 -> 50.2 mm

Commit message: WTF CHANGES IN BOARD???
Parts:
- moved C1 3.43 mm to (70.0, 5.21)
- moved D2 3.43 mm to (62.1, 70.9)
- moved IC3 3.43 mm to (65.8, 13.5)
- moved IC5 3.43 mm to (27.2, 64.0)
- moved MIDI_IN2 3.43 mm to (54.2, 88.9)
- moved R7 3.43 mm to (23.5, 75.7)
- moved R8 3.43 mm to (42.5, 73.2)
- moved U$1 3.43 mm to (43.3, 55.6)
- moved VR1 3.43 mm to (26.8, 16.0)
- moved C3 3.43 mm to (28.2, 57.8)
- moved JP2 3.43 mm to (22.9, 27.7)
- moved MIDI_OUT2 3.43 mm to (33.9, 88.9)
- moved Q1 3.43 mm to (33.1, 18.3)
- moved R11 3.43 mm to (23.7, 21.8)
- moved R12 3.43 mm to (29.5, 16.8)
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Routing:
- net LCD_RW: track 48.6 -> 55.4 mm
- net PB14: track 145.7 -> 139.4 mm
- net PB15: track 93.7 -> 88.9 mm
- net PB3: track 105.0 -> 100.7 mm
- net PC13: track 81.0 -> 77.5 mm
- net SCS_D2: track 66.3 -> 62.9 mm
- net LCD_D7: track 27.7 -> 31.1 mm
- net SCS_D6: track 60.3 -> 56.9 mm
- net SCS_D5: track 54.3 -> 50.8 mm
- net SCS_D3: track 52.9 -> 49.5 mm
- net SCS_D1: track 53.8 -> 50.4 mm
- net SCS_D0: track 60.0 -> 56.6 mm
- net PB5: track 105.6 -> 102.2 mm
- net MIDI_IN2: track 18.4 -> 15.0 mm
- net LCD_RS: track 43.3 -> 46.8 mm
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