File: eagle/mutebox/scs.brd (EAGLE design)
At the start: 127 x 50.8 mm, 31 parts, among them IC1 6N138S-TA1, IC2 6N138S-TA1, SW1 RK09D1130C2P

Commit message: wip
Parts:
- added JP1: (no value), microbuilder:2X08
- R10, R5: value 4.7K -> 1K
- R4, R9: value 1K -> 4.7K
- moved CONN_SCS 205.6 mm to (123.2, 32.3), flipped to the bottom, turned to 270 degrees
- moved CONN_MIDI 204.5 mm to (123.2, 18.0), flipped to the bottom, turned to 270 degrees
- moved IC1 200.9 mm to (107.7, 6.86), turned to 90 degrees
- moved R10 183.6 mm to (91.2, 6.86), flipped to the bottom, turned to 180 degrees
- moved R5 183.1 mm to (109.7, 6.86), flipped to the bottom, turned to 180 degrees
- moved R9 176.6 mm to (87.1, 6.86), flipped to the bottom
- moved R4 176.1 mm to (105.7, 6.86), flipped to the bottom
- moved IC2 142.0 mm to (89.2, 6.35), turned to 90 degrees
- moved R1 138.2 mm to (88.6, 35.1), flipped to the bottom
- moved D1 130.8 mm to (88.4, 33.0), flipped to the bottom
- moved R3 126.7 mm to (68.3, 35.1), flipped to the bottom
- moved R6 118.5 mm to (47.8, 35.1), flipped to the bottom
- moved R2 108.3 mm to (51.3, 35.1), flipped to the bottom, turned to 180 degrees
- moved R8 107.9 mm to (27.9, 35.1), flipped to the bottom
- moved D2 99.8 mm to (47.5, 33.0), flipped to the bottom
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Connections:
- new net LCD_B+: JP1.1, LCD1.A
- new net LCD_B-: JP1.2, LCD1.K
- new net LCD_D0: JP1.9, LCD1.DB0
- new net LCD_D1: JP1.10, LCD1.DB1
- new net LCD_D2: JP1.7, LCD1.DB2
- new net LCD_D3: JP1.8, LCD1.DB3
- new net LCD_D4: JP1.5, LCD1.DB4
- new net LCD_D5: JP1.6, LCD1.DB5
- new net LCD_D6: JP1.3, LCD1.DB6
- new net LCD_D7: JP1.4, LCD1.DB7
- new net LCD_E: JP1.12, LCD1.E
- new net LCD_RS: JP1.14, LCD1.RS
- new net LCD_RW: JP1.11, LCD1.R/W
- new net LCD_V0: JP1.13, LCD1.V5
- new net LCD_VD: JP1.16, LCD1.VDD
- new net LCD_VS: JP1.15, LCD1.GND
Routing:
- added copper zone on layer 1, net 5.0V
- added copper zone on layer 16, net GND

Commit message: wip
Parts:
- removed CONN_MIDI: (no value), microbuilder:2X05
- removed D1, D2: 1N4148WS, microbuilder:SOD-323
- removed IC1, IC2: 6N138S-TA1, 6n138:SO8-GW300
- removed MIDI_IN1, MIDI_IN2, MIDI_OUT1, MIDI_OUT2: MIDIJACK, keves:CP-2350
- removed R1, R2, R3, R6, R7, R8: 220, microbuilder:_0603
- removed R10, R5: 1K, microbuilder:_0603
- removed R4, R9: 4.7K, microbuilder:_0603
Connections:
- removed net 5.0V: CONN_MIDI.2, IC1.8, IC2.8, R10.2, R3.1, R5.2, R8.1
- removed net MIDI_IN1: CONN_MIDI.4, IC1.6, R5.1
- removed net MIDI_IN2: CONN_MIDI.3, IC2.6, R10.1
- removed net MIDI_IN3: CONN_MIDI.6
- removed net MIDI_IN4: CONN_MIDI.5
- removed net MIDI_OUT1: CONN_MIDI.8, R2.1
- removed net MIDI_OUT2: CONN_MIDI.7, R7.1
- removed net MIDI_OUT3: CONN_MIDI.10
- removed net MIDI_OUT4: CONN_MIDI.9
- removed net N$1: MIDI_OUT1.5, R2.2
- removed net N$10: MIDI_IN2.4, R6.2
- removed net N$11: D2.C, IC2.2, R6.1
- removed net N$12: D2.A, IC2.3, MIDI_IN2.5
- removed net N$13: IC2.7, R9.1
- removed net N$2: MIDI_OUT1.4, R3.2
- removed net N$3: MIDI_IN1.4, R1.2
- removed net N$4: D1.C, IC1.2, R1.1
- removed net N$5: D1.A, IC1.3, MIDI_IN1.5
- removed net N$6: IC1.7, R4.1
- removed net N$8: MIDI_OUT2.5, R7.2
- removed net N$9: MIDI_OUT2.4, R8.2
- net GND: no longer CONN_MIDI.1, IC1.5, IC2.5, MIDI_OUT1.2, MIDI_OUT2.2, R4.2, R9.2
Changed lines of the file:
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@@
 </autorouter>
 <elements>
-<element name="MIDI_IN1" library="keves" package="CP-2350" value="MIDIJACK" x="80.01" y="50.8" smashed="yes" rot="MR180">
-<attribute name="NAME" x="73.914" y="33.956" size="1.778" layer="26" ratio="10" rot="MR180"/>
-</element>
-<element name="MIDI_OUT1" library="keves" package="CP-2350" value="MIDIJACK" x="59.69" y="50.8" smashed="yes" rot="MR180">
-<attribute name="NAME" x="53.594" y="33.956" size="1.778" layer="26" ratio="10" rot="MR180"/>
-</element>
-<element name="R1" library="microbuilder" package="_0603" value="220" x="88.646" y="35.052" rot="MR0"/>
-<element name="R2" library="microbuilder" package="_0603" value="220" x="51.308" y="35.052" rot="MR180"/>
-<element name="R3" library="microbuilder" package="_0603" value="220" x="68.326" y="35.052" rot="MR0"/>
-<element name="D1" library="microbuilder" package="SOD-323" value="1N4148WS" x="88.392" y="33.02" rot="MR0"/>
-<element name="IC1" library="6n138" package="SO8-GW300" value="6N138S-TA1" x="107.696" y="6.858" rot="R90"/>
-<element name="R4" library="microbuilder" package="_0603" value="4.7K" x="105.664" y="6.858" rot="MR0"/>
-<element name="R5" library="microbuilder" package="_0603" value="1K" x="109.728" y="6.858" rot="MR180"/>
-<element name="MIDI_IN2" library="keves" package="CP-2350" value="MIDIJACK" x="39.37" y="50.8" smashed="yes" rot="MR180">
-<attribute name="NAME" x="33.274" y="33.956" size="1.778" layer="26" ratio="10" rot="MR180"/>
-</element>
-<element name="MIDI_OUT2" library="keves" package="CP-2350" value="MIDIJACK" x="19.05" y="50.8" smashed="yes" rot="MR180">
-<attribute name="NAME" x="12.954" y="33.956" size="1.778" layer="26" ratio="10" rot="MR180"/>
-</element>
-<element name="R6" library="microbuilder" package="_0603" value="220" x="47.752" y="35.052" rot="MR0"/>
-<element name="R7" library="microbuilder" package="_0603" value="220" x="10.414" y="35.052" rot="MR180"/>
-<element name="R8" library="microbuilder" package="_0603" value="220" x="27.94" y="35.052" rot="MR0"/>
-<element name="D2" library="microbuilder" package="SOD-323" value="1N4148WS" x="47.498" y="33.02" rot="MR0"/>
-<element name="IC2" library="6n138" package="SO8-GW300" value="6N138S-TA1" x="89.154" y="6.35" rot="R90"/>
-<element name="R9" library="microbuilder" package="_0603" value="4.7K" x="87.122" y="6.858" rot="MR0"/>
-<element name="R10" library="microbuilder" package="_0603" value="1K" x="91.186" y="6.858" rot="MR180"/>
 <element name="H1" library="holes" package="3,3" value="MOUNT-HOLE3.3" x="2.54" y="48.26"/>
 <element name="H2" library="holes" package="3,3" value="MOUNT-HOLE3.3" x="124.46" y="48.26"/>
@@
 <element name="S5" library="og-switch" package="B3F-40XX" value="" x="102.87" y="20.32"/>
 <element name="CONN_SCS" library="microbuilder" package="2X05" value="" x="123.19" y="32.258" rot="MR270"/>
-<element name="CONN_MIDI" library="microbuilder" package="2X05" value="" x="123.19" y="18.034" rot="MR270"/>
 <element name="JP1" library="microbuilder" package="2X08" value="" x="45.212" y="3.556" rot="MR180"/>
 </elements>
 <signals>
 <signal name="GND">
-<contactref element="MIDI_OUT1" pad="2"/>
-<contactref element="R4" pad="2"/>
-<contactref element="IC1" pad="5"/>
-<contactref element="MIDI_OUT2" pad="2"/>
-<contactref element="R9" pad="2"/>
-<contactref element="IC2" pad="5"/>
 <contactref element="SW1" pad="D"/>
 <contactref element="SW1" pad="C"/>
@@
 <contactref element="S5" pad="4"/>
 <contactref element="CONN_SCS" pad="1"/>
-<contactref element="CONN_MIDI" pad="1"/>
 <polygon width="0.254" layer="16">
 <vertex x="0.254" y="50.546"/>
@@
 <vertex x="0.254" y="0.254"/>
 </polygon>
-<wire x1="109.1184" y1="17.8308" x2="111.633" y2="11.548" width="0" layer="19" extent="1-1"/>
-<wire x1="93.091" y1="11.04" x2="96.6216" y2="17.8308" width="0" layer="19" extent="1-1"/>
-</signal>
-<signal name="N$1">
-<contactref element="R2" pad="2"/>
-<contactref element="MIDI_OUT1" pad="5"/>
-<wire x1="52.07" y1="35.052" x2="54.61" y2="35.78" width="0" layer="19" extent="16-16"/>
-</signal>
-<signal name="N$2">
-<contactref element="R3" pad="2"/>
-<contactref element="MIDI_OUT1" pad="4"/>
-<wire x1="64.77" y1="35.78" x2="67.564" y2="35.052" width="0" layer="19" extent="16-16"/>
 </signal>
 <signal name="5.0V">
-<contactref element="R3" pad="1"/>
-<contactref element="IC1" pad="8"/>
-<contactref element="R5" pad="2"/>
-<contactref element="R8" pad="1"/>
-<contactref element="IC2" pad="8"/>
-<contactref element="R10" pad="2"/>
-<contactref element="CONN_MIDI" pad="2"/>
 <polygon width="0.254" layer="1">
 <vertex x="0.254" y="50.546"/>
@@
 <vertex x="0.254" y="0.254"/>
 </polygon>
-<wire x1="85.217" y1="11.04" x2="69.088" y2="35.052" width="0" layer="19" extent="1-16"/>
-<wire x1="91.948" y1="6.858" x2="85.217" y2="11.04" width="0" layer="19" extent="1-16"/>
-<wire x1="110.49" y1="6.858" x2="91.948" y2="6.858" width="0" layer="19" extent="16-16"/>
-<wire x1="28.702" y1="35.052" x2="69.088" y2="35.052" width="0" layer="19" extent="16-16"/>
-</signal>
-<signal name="MIDI_OUT1">
-<contactref element="R2" pad="1"/>
-<contactref element="CONN_MIDI" pad="8"/>
-<wire x1="50.546" y1="35.052" x2="121.92" y2="15.494" width="0" layer="19" extent="16-16"/>
-</signal>
-<signal name="N$3">
-<contactref element="R1" pad="2"/>
-<contactref element="MIDI_IN1" pad="4"/>
-<wire x1="85.09" y1="35.78" x2="87.884" y2="35.052" width="0" layer="19" extent="16-16"/>
-</signal>
-<signal name="N$4">
-<contactref element="R1" pad="1"/>
-<contactref element="D1" pad="C"/>
-<contactref element="IC1" pad="2"/>
-<wire x1="89.662" y1="33.02" x2="89.408" y2="35.052" width="0" layer="19" extent="16-16"/>
-<wire x1="106.426" y1="2.168" x2="89.662" y2="33.02" width="0" layer="19" extent="1-16"/>
-</signal>
-<signal name="N$5">
-<contactref element="MIDI_IN1" pad="5"/>
-<contactref element="D1" pad="A"/>
-<contactref element="IC1" pad="3"/>
-<wire x1="74.93" y1="35.78" x2="87.122" y2="33.02" width="0" layer="19" extent="16-16"/>
-<wire x1="108.966" y1="2.168" x2="87.122" y2="33.02" width="0" layer="19" extent="1-16"/>
-</signal>
-<signal name="N$6">
-<contactref element="R4" pad="1"/>
-<contactref element="IC1" pad="7"/>
-<wire x1="106.426" y1="6.858" x2="106.426" y2="11.548" width="0" layer="19" extent="1-16"/>
-</signal>
-<signal name="MIDI_IN1">
-<contactref element="IC1" pad="6"/>
-<contactref element="R5" pad="1"/>
-<contactref element="CONN_MIDI" pad="4"/>
-<wire x1="108.966" y1="11.548" x2="121.92" y2="20.574" width="0" layer="19" extent="1-1"/>
-<wire x1="108.966" y1="6.858" x2="108.966" y2="11.548" width="0" layer="19" extent="1-16"/>
-</signal>
-<signal name="N$8">
-<contactref element="R7" pad="2"/>
-<contactref element="MIDI_OUT2" pad="5"/>
-<wire x1="11.176" y1="35.052" x2="13.97" y2="35.78" width="0" layer="19" extent="16-16"/>
-</signal>
-<signal name="N$9">
-<contactref element="R8" pad="2"/>
-<contactref element="MIDI_OUT2" pad="4"/>
-<wire x1="24.13" y1="35.78" x2="27.178" y2="35.052" width="0" layer="19" extent="16-16"/>
-</signal>
-<signal name="N$10">
-<contactref element="R6" pad="2"/>
-<contactref element="MIDI_IN2" pad="4"/>
-<wire x1="44.45" y1="35.78" x2="46.99" y2="35.052" width="0" layer="19" extent="16-16"/>
-</signal>
-<signal name="N$11">
-<contactref element="R6" pad="1"/>
-<contactref element="D2" pad="C"/>
-<contactref element="IC2" pad="2"/>
-<wire x1="48.768" y1="33.02" x2="87.884" y2="1.66" width="0" layer="19" extent="1-16"/>
-<wire x1="48.514" y1="35.052" x2="48.768" y2="33.02" width="0" layer="19" extent="16-16"/>
-</signal>
-<signal name="N$12">
-<contactref element="MIDI_IN2" pad="5"/>
-<contactref element="D2" pad="A"/>
-<contactref element="IC2" pad="3"/>
-<wire x1="46.228" y1="33.02" x2="90.424" y2="1.66" width="0" layer="19" extent="1-16"/>
-<wire x1="34.29" y1="35.78" x2="46.228" y2="33.02" width="0" layer="19" extent="16-16"/>
-</signal>
-<signal name="N$13">
-<contactref element="R9" pad="1"/>
-<contactref element="IC2" pad="7"/>
-<wire x1="87.884" y1="6.858" x2="87.884" y2="11.04" width="0" layer="19" extent="1-16"/>
-</signal>
-<signal name="MIDI_IN2">
-<contactref element="IC2" pad="6"/>
-<contactref element="R10" pad="1"/>
-<contactref element="CONN_MIDI" pad="3"/>
-<wire x1="90.424" y1="11.04" x2="124.46" y2="20.574" width="0" layer="19" extent="1-1"/>
-<wire x1="90.424" y1="6.858" x2="90.424" y2="11.04" width="0" layer="19" extent="1-16"/>
-</signal>
-<signal name="MIDI_OUT2">
-<contactref element="R7" pad="1"/>
-<contactref element="CONN_MIDI" pad="7"/>
-<wire x1="9.652" y1="35.052" x2="124.46" y2="15.494" width="0" layer="19" extent="16-16"/>
 </signal>
 <signal name="SCS_D6">
@@
 <contactref element="CONN_SCS" pad="2"/>
 </signal>
-<signal name="MIDI_IN3">
-<contactref element="CONN_MIDI" pad="6"/>
-</signal>
-<signal name="MIDI_IN4">
-<contactref element="CONN_MIDI" pad="5"/>
-</signal>
-<signal name="MIDI_OUT3">
-<contactref element="CONN_MIDI" pad="10"/>
-</signal>
-<signal name="MIDI_OUT4">
-<contactref element="CONN_MIDI" pad="9"/>
-</signal>
 <signal name="LCD_B+">

Commit message: route mutebox scs
Parts:
- removed JP1: (no value), microbuilder:2X08
- added SV1: (no value), con-harting-ml:ML16
- CONN_SCS: device microbuilder:2X05 -> con-harting-ml:ML10
- moved CONN_SCS 0.80 mm to (122.4, 32.0)
Connections:
- net LCD_B+: now also SV1.1; no longer JP1.1
- net LCD_B-: now also SV1.2; no longer JP1.2
- net LCD_D0: now also SV1.9; no longer JP1.9
- net LCD_D1: now also SV1.10; no longer JP1.10
- net LCD_D2: now also SV1.7; no longer JP1.7
- net LCD_D3: now also SV1.8; no longer JP1.8
- net LCD_D4: now also SV1.5; no longer JP1.5
- net LCD_D5: now also SV1.6; no longer JP1.6
- net LCD_D6: now also SV1.3; no longer JP1.3
- net LCD_D7: now also SV1.4; no longer JP1.4
- net LCD_E: now also SV1.12; no longer JP1.12
- net LCD_RS: now also SV1.14; no longer JP1.14
- net LCD_RW: now also SV1.11; no longer JP1.11
- net LCD_V0: now also SV1.13; no longer JP1.13
- net LCD_VD: now also SV1.16; no longer JP1.16
- net LCD_VS: now also SV1.15; no longer JP1.15
Routing:
- net SCS_D6: track 0.00 -> 138.0 mm
- net SCS_D5: track 0.00 -> 92.1 mm, vias 0 -> 1
- net SCS_D4: track 0.00 -> 76.8 mm, vias 0 -> 1
- net SCS_D3: track 0.00 -> 57.6 mm
- net LCD_B-: track 0.00 -> 57.1 mm
- net LCD_B+: track 0.00 -> 48.3 mm
- net LCD_V0: track 0.00 -> 45.5 mm
- net SCS_D7: track 0.00 -> 43.7 mm
- net SCS_D2: track 0.00 -> 33.9 mm
- net LCD_VS: track 0.00 -> 32.6 mm
- net LCD_RW: track 0.00 -> 30.4 mm
- net LCD_D2: track 0.00 -> 28.3 mm
- net LCD_D0: track 0.00 -> 28.1 mm
- net LCD_E: track 0.00 -> 28.1 mm
- net LCD_D6: track 0.00 -> 28.0 mm
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