File: eagle/mutebox/scs.sch (EAGLE design)
At the start: 31 parts, among them IC1 6N138S-TA1, IC2 6N138S-TA1, SW1 RK09D1130C2P

Commit message: wip
Parts:
- added JP1: (no value), microbuilder:HEADER-2X8
- R10, R5: value 4.7K -> 1K
- R4, R9: value 1K -> 4.7K
Connections:
- new net LCD_B+: JP1.1, LCD1.A
- new net LCD_B-: JP1.2, LCD1.K
- new net LCD_D0: JP1.9, LCD1.DB0
- new net LCD_D1: JP1.10, LCD1.DB1
- new net LCD_D2: JP1.7, LCD1.DB2
- new net LCD_D3: JP1.8, LCD1.DB3
- new net LCD_D4: JP1.5, LCD1.DB4
- new net LCD_D5: JP1.6, LCD1.DB5
- new net LCD_D6: JP1.3, LCD1.DB6
- new net LCD_D7: JP1.4, LCD1.DB7
- new net LCD_E: JP1.12, LCD1.E
- new net LCD_RS: JP1.14, LCD1.RS
- new net LCD_RW: JP1.11, LCD1.R/W
- new net LCD_V0: JP1.13, LCD1.V5
- new net LCD_VD: JP1.16, LCD1.VDD
- new net LCD_VS: JP1.15, LCD1.GND
Other:
- moved on the sheet: LCD1

Commit message: wip
Parts:
- removed CONN_MIDI: (no value), microbuilder:HEADER-2X5
- removed D1, D2: 1N4148WS, microbuilder:DIODESOD-323
- removed IC1, IC2: 6N138S-TA1, 6n138:6N138SMD
- removed MIDI_IN1, MIDI_IN2, MIDI_OUT1, MIDI_OUT2: MIDIJACK, keves:MIDIJACK
- removed R1, R2, R3, R6, R7, R8: 220, microbuilder:RESISTOR_0603
- removed R10, R5: 1K, microbuilder:RESISTOR_0603
- removed R4, R9: 4.7K, microbuilder:RESISTOR_0603
Connections:
- removed net 5.0V: CONN_MIDI.2, IC1.VCC, IC2.VCC, R10.2, R3.1, R5.2, R8.1
- removed net MIDI_IN1: CONN_MIDI.4, IC1.VO, R5.1
- removed net MIDI_IN2: CONN_MIDI.3, IC2.VO, R10.1
- removed net MIDI_IN3: CONN_MIDI.6
- removed net MIDI_IN4: CONN_MIDI.5
- removed net MIDI_OUT1: CONN_MIDI.8, R2.1
- removed net MIDI_OUT2: CONN_MIDI.7, R7.1
- removed net MIDI_OUT3: CONN_MIDI.10
- removed net MIDI_OUT4: CONN_MIDI.9
- removed net N$1: MIDI_OUT1.5, R2.2
- removed net N$10: MIDI_IN2.4, R6.2
- removed net N$11: D2.C, IC2.A, R6.1
- removed net N$12: D2.A, IC2.C, MIDI_IN2.5
- removed net N$13: IC2.VB, R9.1
- removed net N$2: MIDI_OUT1.4, R3.2
- removed net N$3: MIDI_IN1.4, R1.2
- removed net N$4: D1.C, IC1.A, R1.1
- removed net N$5: D1.A, IC1.C, MIDI_IN1.5
- removed net N$6: IC1.VB, R4.1
- removed net N$8: MIDI_OUT2.5, R7.2
- removed net N$9: MIDI_OUT2.4, R8.2
- net GND: no longer CONN_MIDI.1, IC1.GND, IC2.GND, MIDI_OUT1.2, MIDI_OUT2.2, R4.2, R9.2

Commit message: route mutebox scs
Parts:
- removed JP1: (no value), microbuilder:HEADER-2X8
- added SV1: (no value), con-harting-ml:ML16
- CONN_SCS: device microbuilder:HEADER-2X5 -> con-harting-ml:ML10
Connections:
- net LCD_B+: now also SV1.1; no longer JP1.1
- net LCD_B-: now also SV1.2; no longer JP1.2
- net LCD_D0: now also SV1.9; no longer JP1.9
- net LCD_D1: now also SV1.10; no longer JP1.10
- net LCD_D2: now also SV1.7; no longer JP1.7
- net LCD_D3: now also SV1.8; no longer JP1.8
- net LCD_D4: now also SV1.5; no longer JP1.5
- net LCD_D5: now also SV1.6; no longer JP1.6
- net LCD_D6: now also SV1.3; no longer JP1.3
- net LCD_D7: now also SV1.4; no longer JP1.4
- net LCD_E: now also SV1.12; no longer JP1.12
- net LCD_RS: now also SV1.14; no longer JP1.14
- net LCD_RW: now also SV1.11; no longer JP1.11
- net LCD_V0: now also SV1.13; no longer JP1.13
- net LCD_VD: now also SV1.16; no longer JP1.16
- net LCD_VS: now also SV1.15; no longer JP1.15
