File: midimixer-channel.sch (EAGLE design)
At the start: 29 parts, among them U1 LM1117IMPX-3.3/NOPB, Y1 8MHz 695-HCM49-8-U

Commit message: wip
Parts:
- added C14, C15: 0.1uF, microbuilder:CAP_CERAMIC0603
- added D1: DC7G3HWA, SparkFun-LED:LED_BARGRAPH_10
- added JP4: (no value), microbuilder:HEADER-1X670MIL
- added R5, R6: 330, microbuilder:RESISTOR0603
- added RN1, RN2: 4606X-101-101LF, resistor-sil:G05R
- added U$36: B3W-9000-RG2N, keves:B3W-9000-RG2N
Connections:
- new net LCD_CLK: JP4.3
- new net LCD_DC: JP4.6
- new net LCD_MOSI: JP4.4
- new net LCS_CS: JP4.5
- new net N$10: R6.1, U$36.LED2-
- new net N$11: C15.P$2, U$36.SW2_A, U$36.SW2_B
- new net N$12: U$36.LED1+
- new net N$13: U$36.LED2+
- new net N$14: D1A.C, RN1.2
- new net N$15: D1B.C, RN1.3
- new net N$16: D1C.C, RN1.4
- new net N$17: D1D.C, RN1.5
- new net N$18: D1E.C, RN1.6
- new net N$19: D1F.C, RN2.2
- new net N$20: D1G.C, RN2.3
- new net N$21: D1H.C, RN2.4
- new net N$22: D1I.C, RN2.5
- new net N$23: D1J.C, RN2.6
- new net N$9: R5.1, U$36.LED1-
- net 3.3V: now also C14.P$2, JP4.1
- net GND: now also C14.P$1, C15.P$1, JP4.2, R5.2, R6.2, RN1.1, RN2.1, U$36.SW1_A, U$36.SW1_B
- net PB2: now also B2.S

Commit message: wip
Parts:
- added C16, C17, C18, C19, C20, C21, C22, C23, C24: 0.1uF, microbuilder:CAP_CERAMIC0603
- added H1, H2, H3, H4: STAND-OFF, SparkFun-Electromechanical:STAND-OFF
- added IC1, IC2, IC3, IC4: 74LS595D, SparkFun-DigitalIC:74LS595D
- added R10, R11, R12, R13, R14, R15, R16, R7, R8, R9: 330, microbuilder:RESISTOR0603
- added R17, R19, R20, R21, R22, R23, R24, R25, R26: 10k, microbuilder:RESISTOR_0603
- added U$42: PTA6043-2015CPB103, keves:PTA6043-2015CPB103
- added U$43, U$47, U$51, U$55, U$59: B3W-9000-RG2N, keves:B3W-9000-RG2N
- added U$63, U$64: PEC11-4215K-S0024, keves:PEC11-4215K-S0024
- added U$65, U$66, U$67, U$68, U$69, U$70, U$71: PTV111-4220A-B104, keves:PTV111-4220A-B104
- added U$87: 74165D, SparkFun-DigitalIC:74165D
Connections:
- new net BTN_LED1: IC3.QC, U$55.LED1+
- new net BTN_LED10: IC4.QD
- new net BTN_LED11: IC4.QE
- new net BTN_LED12: IC4.QF
- new net BTN_LED2: IC3.QD, U$55.LED2+
- new net BTN_LED3: IC3.QE, U$43.LED1+
- new net BTN_LED4: IC3.QF, U$43.LED2+
- new net BTN_LED5: IC3.QG, U$36.LED1+
- new net BTN_LED6: IC3.QH, U$36.LED2+
- new net BTN_LED7: IC4.QA
- new net BTN_LED8: IC4.QB
- new net BTN_LED9: IC4.QC
- new net N$24: R7.1, U$43.LED1-
- new net N$25: R8.1, U$43.LED2-
- new net N$26: C16.P$2, U$43.SW2_A, U$43.SW2_B
- new net N$27: U$87.QH
- new net N$28: R17.1, U$87.SER
- new net N$29: R9.1, U$47.LED1-
- new net N$30: R10.1, U$47.LED2-
- new net N$31: C17.P$2, U$47.SW2_A, U$47.SW2_B
- new net N$32: U$47.LED1+
- new net N$33: U$47.LED2+
- new net N$34: R11.1, U$51.LED1-
- new net N$35: R12.1, U$51.LED2-
- new net N$36: C18.P$2, U$51.SW2_A, U$51.SW2_B
- new net N$37: U$51.LED1+
- new net N$38: U$51.LED2+
- new net N$39: R13.1, U$55.LED1-
- new net N$40: R14.1, U$55.LED2-
- new net N$41: C19.P$2, U$55.SW2_A, U$55.SW2_B
- new net N$42: R26.1, U$87.A
- new net N$43: R25.1, U$87.B
- new net N$44: R15.1, U$59.LED1-
- new net N$45: R16.1, U$59.LED2-
- new net N$46: C20.P$2, U$59.SW2_A, U$59.SW2_B
- new net N$47: U$59.LED1+
- new net N$48: U$59.LED2+
- new net N$49: D1J.A, IC1.QA
- new net N$50: D1I.A, IC1.QB
- new net N$51: D1H.A, IC1.QC
- new net N$52: D1G.A, IC1.QD
- new net N$53: D1F.A, IC1.QE
- new net N$54: D1E.A, IC1.QF
- new net N$55: D1D.A, IC1.QG
- new net N$56: D1C.A, IC1.QH
- new net N$57: IC1.QH*, IC3.SER
- new net N$58: IC1.SCK, IC3.SCK, IC4.SCK, U$87.CLK
- new net N$59: IC1.RCK, IC3.RCK, IC4.RCK, U$87.SH/!LD
- new net N$60: D1B.A, IC3.QA
- new net N$61: D1A.A, IC3.QB
- new net N$62: R24.1, U$87.C
- new net N$63: IC4.QG
- new net N$64: IC4.QH
- new net N$65: IC4.QH*
- new net N$66: R23.1, U$87.D
- new net N$67: R22.1, U$87.E
- new net N$68: R21.1, U$87.F
- new net N$69: R20.1, U$87.G
- new net N$70: R19.1, U$87.H
- net 3.3V: now also C21.P$2, C22.P$2, C23.P$1, C24.P$2, IC1.SCL, IC1.VCC, IC3.SCL, IC3.VCC, IC4.SCL, IC4.VCC, R17.2, R19.2, R20.2, R21.2, R22.2, R23.2, R24.2, R25.2, R26.2, U$87.VCC
- net GND: now also C16.P$1, C17.P$1, C18.P$1, C19.P$1, C20.P$1, C21.P$1, C22.P$1, C23.P$2, C24.P$1, IC1.G, IC1.GND, IC3.G, IC3.GND, IC4.G, IC4.GND, R10.2, R11.2, R12.2, R13.2, R14.2, R15.2, R16.2, R7.2, R8.2, R9.2, U$43.SW1_A, U$43.SW1_B, U$47.SW1_A, U$47.SW1_B, U$51.SW1_A, U$51.SW1_B, U$55.SW1_A, U$55.SW1_B, U$59.SW1_A, U$59.SW1_B, U$87.CLK_INH, U$87.GND
- net N$12: now also IC3.QH*, IC4.SER; no longer U$36.LED1+
- net N$13: now also IC1.SER; no longer U$36.LED2+

Commit message: wip
Parts:
- added C25: 0.1uF, microbuilder:CAP_CERAMIC0603
- added D2: SN65HVD230, omc:SN65HVD230
- added R18: 0, microbuilder:RESISTOR_0603
- added R27: 120, microbuilder:RESISTOR_0603
Connections:
- removed net N$13: IC1.SER
- removed net N$27: U$87.QH
- removed net N$58: IC1.SCK, IC3.SCK, IC4.SCK, U$87.CLK
- removed net N$59: IC1.RCK, IC3.RCK, IC4.RCK, U$87.SH/!LD
- new net CAN_H: D2.CANH, R27.1
- new net CAN_L: D2.CANL, R27.2
- new net CAN_RX: D2.RXD
- new net CAN_TX: D2.TXD
- new net N$73: D2.RS, R18.1
- new net SPI2_CLK: IC1.SCK, IC3.SCK, IC4.SCK, U$1.PB13/I2S2_CK, U$87.CLK
- new net SPI2_MISO: U$1.PB14/I2S2_XD, U$87.QH
- new net SPI2_MOSI: IC1.SER, U$1.PB15/I2S2_SD
- new net SPI2_RC1: IC1.RCK, IC3.RCK, IC4.RCK, U$1.PB12/I2S2_WS
- new net SPI2_RC2: U$1.PC6/I2S2_MCK, U$87.SH/!LD
- net 3.3V: now also C25.P$1, D2.VCC
- net GND: now also C25.P$2, D2.GND, R18.2
Other:
- note added: "PD10 in Midibox!!"
- moved on the sheet: C14, JP4

Commit message: wip
Connections:
- removed net N$32: U$47.LED1+
- removed net N$33: U$47.LED2+
- removed net N$37: U$51.LED1+
- removed net N$38: U$51.LED2+
- removed net N$47: U$59.LED1+
- removed net N$48: U$59.LED2+
- net 3.3V: now also U$42.E, U$65.E, U$66.E, U$67.E, U$68.E
- net BTN_LED10: now also U$51.LED2+
- net BTN_LED11: now also U$59.LED1+
- net BTN_LED12: now also U$59.LED2+
- net BTN_LED7: now also U$47.LED1+
- net BTN_LED8: now also U$47.LED2+
- net BTN_LED9: now also U$51.LED1+
- net GND: now also U$42.A, U$65.A, U$66.A, U$67.A, U$68.A, U$69.A, U$70.A, U$71.A
Changed lines of the file:
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@@
 <part name="U$96" library="microbuilder" deviceset="GND" device=""/>
 <part name="R27" library="microbuilder" deviceset="RESISTOR" device="_0603" value="120"/>
+<part name="U$97" library="microbuilder" deviceset="GND" device=""/>
+<part name="U$98" library="microbuilder" deviceset="3.3V" device=""/>
+<part name="U$99" library="microbuilder" deviceset="GND" device=""/>
+<part name="U$100" library="microbuilder" deviceset="GND" device=""/>
+<part name="U$101" library="microbuilder" deviceset="GND" device=""/>
+<part name="U$102" library="microbuilder" deviceset="GND" device=""/>
+<part name="U$103" library="microbuilder" deviceset="GND" device=""/>
+<part name="U$104" library="microbuilder" deviceset="GND" device=""/>
+<part name="U$105" library="microbuilder" deviceset="GND" device=""/>
+<part name="U$106" library="microbuilder" deviceset="3.3V" device=""/>
+<part name="U$107" library="microbuilder" deviceset="3.3V" device=""/>
+<part name="U$108" library="microbuilder" deviceset="3.3V" device=""/>
+<part name="U$109" library="microbuilder" deviceset="3.3V" device=""/>
 </parts>
 <sheets>
@@
 <instance part="U$70" gate="G$1" x="45.72" y="-30.48" rot="R270"/>
 <instance part="U$71" gate="G$1" x="45.72" y="-48.26" rot="R270"/>
+<instance part="U$97" gate="G$1" x="27.94" y="12.7" rot="R90"/>
+<instance part="U$98" gate="G$1" x="7.62" y="12.7" rot="R90"/>
+<instance part="U$99" gate="G$1" x="53.34" y="-12.7" rot="R90"/>
+<instance part="U$100" gate="G$1" x="53.34" y="-30.48" rot="R90"/>
+<instance part="U$101" gate="G$1" x="53.34" y="-48.26" rot="R90"/>
+<instance part="U$102" gate="G$1" x="15.24" y="-71.12" rot="R90"/>
+<instance part="U$103" gate="G$1" x="15.24" y="-50.8" rot="R90"/>
+<instance part="U$104" gate="G$1" x="15.24" y="-30.48" rot="R90"/>
+<instance part="U$105" gate="G$1" x="15.24" y="-12.7" rot="R90"/>
+<instance part="U$106" gate="G$1" x="0" y="-12.7" rot="R90"/>
+<instance part="U$107" gate="G$1" x="0" y="-30.48" rot="R90"/>
+<instance part="U$108" gate="G$1" x="0" y="-50.8" rot="R90"/>
+<instance part="U$109" gate="G$1" x="0" y="-71.12" rot="R90"/>
 </instances>
 <busses>
@@
 <junction x="177.8" y="-30.48"/>
 </segment>
+<segment>
+<pinref part="U$42" gate="G$1" pin="A"/>
+<pinref part="U$97" gate="G$1" pin="GND"/>
+<wire x1="25.4" y1="12.7" x2="22.86" y2="12.7" width="0.1524" layer="91"/>
+</segment>
+<segment>
+<pinref part="U$69" gate="G$1" pin="A"/>
+<pinref part="U$99" gate="G$1" pin="GND"/>
+</segment>
+<segment>
+<pinref part="U$70" gate="G$1" pin="A"/>
+<pinref part="U$100" gate="G$1" pin="GND"/>
+</segment>
+<segment>
+<pinref part="U$71" gate="G$1" pin="A"/>
+<pinref part="U$101" gate="G$1" pin="GND"/>
+</segment>
+<segment>
+<pinref part="U$68" gate="G$1" pin="A"/>
+<pinref part="U$102" gate="G$1" pin="GND"/>
+</segment>
+<segment>
+<pinref part="U$67" gate="G$1" pin="A"/>
+<pinref part="U$103" gate="G$1" pin="GND"/>
+</segment>
+<segment>
+<pinref part="U$66" gate="G$1" pin="A"/>
+<pinref part="U$104" gate="G$1" pin="GND"/>
+</segment>
+<segment>
+<pinref part="U$65" gate="G$1" pin="A"/>
+<pinref part="U$105" gate="G$1" pin="GND"/>
+</segment>
 </net>
 <net name="N$9" class="0">
@@
 </segment>
 </net>
-<net name="N$32" class="0">
+<net name="BTN_LED7" class="0">
 <segment>
 <pinref part="U$47" gate="G$1" pin="LED1+"/>
@@
 </segment>
 </net>
-<net name="N$33" class="0">
+<net name="BTN_LED8" class="0">
 <segment>
 <pinref part="U$47" gate="G$1" pin="LED2+"/>
@@
 </segment>
 </net>
-<net name="N$37" class="0">
+<net name="BTN_LED9" class="0">
 <segment>
 <pinref part="U$51" gate="G$1" pin="LED1+"/>
@@
 </segment>
 </net>
-<net name="N$38" class="0">
+<net name="BTN_LED10" class="0">
 <segment>
 <pinref part="U$51" gate="G$1" pin="LED2+"/>
@@
 </segment>
 </net>
-<net name="N$47" class="0">
+<net name="BTN_LED11" class="0">
 <segment>
 <pinref part="U$59" gate="G$1" pin="LED1+"/>
@@
 </segment>
 </net>
-<net name="N$48" class="0">
+<net name="BTN_LED12" class="0">
 <segment>
 <pinref part="U$59" gate="G$1" pin="LED2+"/>
@@
 </segment>
 </net>
+<net name="3.3V" class="0">
+<segment>
+<pinref part="U$42" gate="G$1" pin="E"/>
+<pinref part="U$98" gate="G$1" pin="3.3V"/>
+<wire x1="10.16" y1="12.7" x2="12.7" y2="12.7" width="0.1524" layer="91"/>
+</segment>
+<segment>
+<pinref part="U$65" gate="G$1" pin="E"/>
+<pinref part="U$106" gate="G$1" pin="3.3V"/>
+</segment>
+<segment>
+<pinref part="U$66" gate="G$1" pin="E"/>
+<pinref part="U$107" gate="G$1" pin="3.3V"/>
+</segment>
+<segment>
+<pinref part="U$67" gate="G$1" pin="E"/>
+<pinref part="U$108" gate="G$1" pin="3.3V"/>
+</segment>
+<segment>
+<pinref part="U$68" gate="G$1" pin="E"/>
+<pinref part="U$109" gate="G$1" pin="3.3V"/>
+</segment>
+</net>

Commit message: wip
Parts:
- removed IC2: 74LS595D, SparkFun-DigitalIC:74LS595D
- removed JP4: (no value), microbuilder:HEADER-1X670MIL
- added R28, R29: 0, microbuilder:RESISTOR_0603
- added U$117: SSD1306-ALI, keves:SSD1306-ALI
Connections:
- removed net N$60: D1B.A, IC3.QA
- removed net N$61: D1A.A, IC3.QB
- removed net N$62: R24.1, U$87.C
- removed net N$63: IC4.QG
- removed net N$64: IC4.QH
- removed net N$66: R23.1, U$87.D
- removed net N$67: R22.1, U$87.E
- removed net N$68: R21.1, U$87.F
- removed net N$69: R20.1, U$87.G
- removed net N$70: R19.1, U$87.H
- new net BTN_UNUSED1: IC4.QB
- new net BTN_UUSED2: IC4.QA
- new net DIN_1: R26.1, U$63.CH_A, U$87.A
- new net DIN_2: R25.1, U$63.CH_B, U$87.B
- new net DIN_3: R24.1, U$63.SW2, U$87.C
- new net DIN_4: R23.1, U$64.CH_A, U$87.D
- new net DIN_5: R22.1, U$64.CH_B, U$87.E
- new net DIN_6: R21.1, U$64.SW2, U$87.F
- new net DIN_7: C15.P$2, R20.1, U$36.SW2_A, U$36.SW2_B, U$87.G
- new net DIN_8: C17.P$2, R19.1, U$47.SW2_A, U$47.SW2_B, U$87.H
- new net N$13: R29.2, U$1.PB9
- new net N$27: R28.2, U$1.PB8
- new net N$32: U$42.S
- new net N$33: U$65.S
- new net N$37: U$69.S
- new net N$38: U$70.S
- new net N$47: U$71.S
- new net N$48: U$68.S
- net 3.3V: now also U$117.VCC, U$69.E, U$70.E, U$71.E; no longer JP4.1
- net BTN_LED1: now also IC3.QA; no longer IC3.QC
- net BTN_LED10: now also IC4.QC; no longer IC4.QD
- net BTN_LED3: now also IC3.QF; no longer IC3.QE
- net BTN_LED4: now also IC3.QH; no longer IC3.QF
- net BTN_LED5: now also IC3.QE; no longer IC3.QG
- net BTN_LED6: now also IC4.QD, U$51.LED1+; no longer IC3.QH, U$36.LED2+
- net BTN_LED7: now also IC4.QG; no longer IC4.QA
- net BTN_LED8: now also IC4.QH; no longer IC4.QB
- net BTN_LED9: now also IC3.QG, U$36.LED2+; no longer IC4.QC, U$51.LED1+
- net CAN_RX: now also R29.1
- net CAN_TX: now also R28.1
- net GND: now also U$117.GND, U$63.COMMON, U$63.SW1, U$64.COMMON, U$64.SW1; no longer JP4.2
- net LCD_CLK: now also U$117.CLK; no longer JP4.3
- net LCD_DC: now also U$117.DC; no longer JP4.6
- net LCD_MOSI: now also U$117.MOSI; no longer JP4.4
- net LCS_CS: now also U$117.CS; no longer JP4.5
- net N$11: now also D1B.A, IC3.QB; no longer C15.P$2, U$36.SW2_A, U$36.SW2_B
- net N$31: now also D1A.A, IC3.QC; no longer C17.P$2, U$47.SW2_A, U$47.SW2_B
- net N$42: now also U$66.S; no longer R26.1, U$87.A
- net N$43: now also U$67.S; no longer R25.1, U$87.B
Other:
- moved on the sheet: U$63, U$64

Commit message: wip
Parts:
- removed SWD: (no value), microbuilder:HEADER-1X576MIL
- removed U$87: 74165D, SparkFun-DigitalIC:74165D
- added IC2: 74LS595D, SparkFun-DigitalIC:74LS595D
- added JP4: (no value), microbuilder:HEADER-1X2ROUND
- C1, C2: value 18pf -> 0.1uF
- C10, C11, C9: value 10uF 603-CC206KKX5R7BB106 -> 0.1uF; device SparkFun-Passives:CAP1206 -> microbuilder:CAP_CERAMIC0603
- C13, C7: value 0.1uF -> 2.2uF 810-CGJ4J2X7R1A225K; device microbuilder:CAP_CERAMIC0603 -> microbuilder:CAP_CERAMIC0805
- C15, C17, C18: value 0.1uF -> 10uF 603-CC206KKX5R7BB106; device microbuilder:CAP_CERAMIC0603 -> SparkFun-Passives:CAP1206
- C4: value 2.2uF 810-CGJ4J2X7R1A225K -> 0.1uF; device microbuilder:CAP_CERAMIC0805 -> microbuilder:CAP_CERAMIC0603
- C5: value 0.1uF -> 18pf
- C6: value 2.2uF 810-CGJ4J2X7R1A225K -> 18pf; device microbuilder:CAP_CERAMIC0805 -> microbuilder:CAP_CERAMIC0603
- IC4: value 74LS595D -> 74165D; device SparkFun-DigitalIC:74LS595D -> SparkFun-DigitalIC:74165D
- JP2: device microbuilder:HEADER-1X2ROUND -> microbuilder:HEADER-1X576MIL
- R10, R13, R14: value 330 -> 0; device microbuilder:RESISTOR0603 -> microbuilder:RESISTOR_0603
- R11: value 330 -> 120; device microbuilder:RESISTOR0603 -> microbuilder:RESISTOR_0603
- R12, R4, R5, R6, R7, R8, R9: value 330 -> 10k; device microbuilder:RESISTOR0603 -> microbuilder:RESISTOR_0603
- R15, R16: value 330 -> 22
- R17, R19, R20, R21, R22, R23, R24, R25, R26: value 10k -> 330; device microbuilder:RESISTOR_0603 -> microbuilder:RESISTOR0603
- R18, R28, R29: value 0 -> 330; device microbuilder:RESISTOR_0603 -> microbuilder:RESISTOR0603
- R2, R3: value 22 -> 10k; device microbuilder:RESISTOR0603 -> microbuilder:RESISTOR_0603
- R27: value 120 -> 330; device microbuilder:RESISTOR_0603 -> microbuilder:RESISTOR0603
- renumbered U$1 to CPU1, U$117 to LCD1, U$36 to BTN1, U$42 to FADER1, U$43 to BTN2, U$47 to BTN4, U$51 to BTN5, U$55 to BTN3, U$59 to BTN6, U$63 to ROTENC1, U$64 to ROTENC2, U$65 to POT1, U$66 to POT2, U$67 to POT3, U$68 to POT4, U$69 to POT5, U$70 to POT6, U$71 to POT7, USB to X1
Connections:
- net 3.3V: now also C1.P$2, C10.P$1, C11.P$1, C12.P$2, C17.2, C2.P$1, C3.P$2, C4.P$2, C9.P$2, IC2.SCL, IC2.VCC, JP2.1, JP4.1, R1.2, R2.2, R3.2, R5.2, R6.2, R7.2, R8.2, R9.2; no longer C10.2, C21.P$2, C22.P$2, C23.P$1, C24.P$2, C25.P$1, C3.P$1, C5.P$2, C7.P$2, IC4.SCL, JP3.1, R19.2, R20.2, R21.2, R22.2, R23.2, R24.2, R25.2, R26.2, SWD.1, U$87.VCC
- net 5.0V: now also C15.2, JP3.1; no longer C9.2, JP2.1
- net AVDD: now also C18.2, C19.P$1; no longer C11.2, C12.P$1
- net BTN_LED1: now also IC2.QA; no longer IC3.QA
- net BTN_LED10: now also IC1.QC; no longer IC4.QC
- net BTN_LED11: now also IC1.QE; no longer IC4.QE
- net BTN_LED12: now also IC1.QF; no longer IC4.QF
- net BTN_LED2: now also IC2.QD; no longer IC3.QD
- net BTN_LED3: now also IC2.QF; no longer IC3.QF
- net BTN_LED4: now also IC2.QH; no longer IC3.QH
- net BTN_LED5: now also IC2.QE; no longer IC3.QE
- net BTN_LED6: now also IC1.QD; no longer IC4.QD
- net BTN_LED7: now also IC1.QG; no longer IC4.QG
- net BTN_LED8: now also IC1.QH; no longer IC4.QH
- net BTN_LED9: now also IC2.QG; no longer IC3.QG
- net BTN_UNUSED1: now also IC1.QB; no longer IC4.QB
- net BTN_UUSED2: now also IC1.QA; no longer IC4.QA
- net CAN_H: now also R11.1; no longer R27.1
- net CAN_L: now also R11.2; no longer R27.2
- net CAN_RX: now also R13.1; no longer R29.1
- net CAN_TX: now also R14.1; no longer R28.1
- net DIN_1: now also IC4.A, R2.1, ROTENC2.CH_B; no longer R26.1, ROTENC1.CH_A, U$87.A
- net DIN_2: now also IC4.B, R3.1, ROTENC1.CH_A; no longer R25.1, ROTENC1.CH_B, U$87.B
- net DIN_3: now also IC4.C, R4.1; no longer R24.1, U$87.C
- net DIN_4: now also IC4.D, R5.1; no longer R23.1, U$87.D
- net DIN_5: now also IC4.E, R6.1, ROTENC1.CH_B; no longer R22.1, ROTENC2.CH_B, U$87.E
- net DIN_6: now also IC4.F, R7.1; no longer R21.1, U$87.F
- net DIN_7: now also C20.P$2, IC4.G, R8.1; no longer C15.P$2, R20.1, U$87.G
- net DIN_8: now also C23.P$2, IC4.H, R9.1; no longer BTN4.SW2_A, C17.P$2, R19.1, U$87.H
- net GND: now also C10.P$2, C11.P$2, C12.P$1, C15.1, C16.P$2, C17.1, C18.1, C19.P$2, C2.P$2, C23.P$1, C25.P$1, C3.P$1, C4.P$1, C6.P$1, C7.P$2, C9.P$1, IC2.G, IC2.GND, IC4.CLK_INH, JP2.5, JP4.2, R19.2, R20.2, R21.2, R22.2, R23.2, R24.2, R25.2, R26.2, R27.2, R28.2, R29.2; no longer BTN2.SW1_A, BTN4.SW1_A, BTN6.SW1_A, C10.1, C11.1, C12.P$2, C15.P$1, C16.P$1, C17.P$1, C18.P$1, C19.P$1, C2.P$1, C23.P$2, C25.P$2, C3.P$2, C4.P$2, C6.P$2, C7.P$1, C9.1, IC4.G, JP2.2, R1.2, R11.2, R13.2, R14.2, R15.2, R16.2, R5.2, R6.2, R7.2, R8.2, R9.2, SWD.5, U$87.CLK_INH, U$87.GND
- net N$1: now also C6.P$2; no longer C2.P$2
- net N$10: now also R19.1; no longer R6.1
- net N$11: now also IC2.QB; no longer IC3.QB
- net N$12: now also IC1.SER, IC2.QH*; no longer IC3.QH*, IC4.SER
- net N$13: now also R13.2; no longer R29.2
- net N$2: now also C5.P$2; no longer C1.P$2
- net N$24: now also R20.1; no longer R7.1
- net N$25: now also R21.1; no longer R8.1
- net N$26: now also C21.P$2; no longer BTN2.SW2_A, C16.P$2
- net N$27: now also R14.2; no longer R28.2
- net N$28: now also IC4.SER, R1.1; no longer R17.1, U$87.SER
- net N$29: now also R24.1; no longer R9.1
- net N$3: now also C13.P$1; no longer C6.P$1
- net N$30: now also R25.1; no longer R10.1
- net N$31: now also IC2.QC; no longer IC3.QC
- net N$34: now also R26.1; no longer R11.1
- net N$35: now also R27.1; no longer R12.1
- net N$36: now also C24.P$2; no longer C18.P$2
- net N$39: now also R22.1; no longer R13.1
- net N$4: now also C7.P$1; no longer C4.P$1
- net N$40: now also R23.1; no longer R14.1
- net N$41: now also C22.P$2; no longer C19.P$2
- net N$44: now also R28.1; no longer R15.1
- net N$45: now also R29.1; no longer R16.1
- net N$46: now also C25.P$2; no longer BTN6.SW2_A, C20.P$2
- net N$49: now also IC3.QA; no longer IC1.QA
- net N$5: now also R17.1; no longer R4.1
- net N$50: now also IC3.QB; no longer IC1.QB
- net N$51: now also IC3.QC; no longer IC1.QC
- net N$52: now also IC3.QD; no longer IC1.QD
- net N$53: now also IC3.QE; no longer IC1.QE
- net N$54: now also IC3.QF; no longer IC1.QF
- net N$55: now also IC3.QG; no longer IC1.QG
- net N$56: now also IC3.QH; no longer IC1.QH
- net N$57: now also IC2.SER, IC3.QH*; no longer IC1.QH*, IC3.SER
- net N$6: now also R12.1; no longer R1.1
- net N$65: now also IC1.QH*; no longer IC4.QH*
- net N$7: now also R15.2; no longer R2.2
- net N$73: now also R10.1; no longer R18.1
- net N$8: now also R16.2; no longer R3.2
- net N$9: now also R18.1; no longer R5.1
- net NRST: now also B2.S, B2.S1, C16.P$1, JP2.4; no longer B1.S, B1.S1, C13.P$1, SWD.4
- net PB2: now also B1.S, B1.S1; no longer B2.S, B2.S1
- net SPI2_CLK: now also IC2.SCK, IC4.CLK; no longer IC4.SCK, U$87.CLK
- net SPI2_MISO: now also IC4.QH; no longer U$87.QH
- net SPI2_MOSI: now also IC3.SER; no longer IC1.SER
- net SPI2_RC1: now also IC2.RCK; no longer IC4.RCK
- net SPI2_RC2: now also IC4.SH/!LD; no longer U$87.SH/!LD
- net SWCK: now also JP2.2; no longer SWD.2
- net SWDIO: now also JP2.3; no longer SWD.3
- net USB_DM: now also R15.1; no longer R2.1
- net USB_DP: now also R16.1; no longer R3.1

Commit message: wip
Connections:
- removed net N$32: FADER1.S
- removed net N$33: POT1.S
- removed net N$37: POT5.S
- removed net N$38: POT6.S
- removed net N$42: POT2.S
- removed net N$43: POT3.S
- removed net N$47: POT7.S
- removed net N$48: POT4.S
- new net ADC0: CPU1.PA0, POT5.S
- new net ADC1: CPU1.PA1, POT6.S
- new net ADC2: CPU1.PA2/UART2_TX, POT7.S
- new net ADC3: CPU1.PA3/UART2_RX, POT4.S
- new net ADC4: CPU1.PA4/SPI1_NSS, POT3.S
- new net ADC5: CPU1.PA5/SPI1_SCK, POT2.S
- new net ADC6: CPU1.PA6/SPI1_MISO, POT1.S
- new net ADC7: CPU1.PA7/SPI1_MOSI, FADER1.S
- new net DIN_TODO: BTN1.SW2_A, BTN1.SW2_B, C20.P$2
- new net DIN_TODO2: BTN4.SW2_B, C23.P$2
- net DIN_1: now also ROTENC2.CH_A; no longer ROTENC2.CH_B
- net DIN_2: now also ROTENC2.CH_B; no longer ROTENC1.CH_A
- net DIN_3: now also ROTENC2.SW2; no longer ROTENC1.SW2
- net DIN_4: no longer ROTENC2.CH_A
- net DIN_5: now also ROTENC1.SW2; no longer ROTENC1.CH_B
- net DIN_6: now also ROTENC1.CH_A; no longer ROTENC2.SW2
- net DIN_7: now also ROTENC1.CH_B; no longer BTN1.SW2_A, BTN1.SW2_B, C20.P$2
- net DIN_8: no longer BTN4.SW2_B, C23.P$2
Other:
- moved on the sheet: C8
