File: midimixer-channel.sch (EAGLE design)
At the start: 95 parts, among them IC1 74LS595D, IC2 74LS595D, IC3 74LS595D, IC4 74165D, U1 LM1117IMPX-3.3/NOPB, Y1 8MHz 695-HCM49-8-U

Commit message: wip
Parts:
- JTAG: value (none) -> jtag
- renumbered JP2 to JTAG
Connections:
- removed net LCS_CS: LCD1.CS
- new net LCD_CS: CPU1.PB6, LCD1.CS
- new net LCD_MISO_UNUSED: CPU1.PB4/JTRST
- net LCD_CLK: now also CPU1.PB3/JTDO
- net LCD_DC: now also CPU1.PB7
- net LCD_MOSI: now also CPU1.PB5
- net NRST: now also JTAG.2; no longer JTAG.4
- net SWCK: now also JTAG.3; no longer JTAG.2
- net SWDIO: now also JTAG.4; no longer JTAG.3
Changed lines of the file:
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@@
 <part name="JP1" library="microbuilder" deviceset="JUMPER2" device=""/>
 <part name="U$20" library="microbuilder" deviceset="5.0V" device=""/>
-<part name="JP2" library="microbuilder" deviceset="HEADER-1X5" device="76MIL"/>
+<part name="JTAG" library="microbuilder" deviceset="HEADER-1X5" device="76MIL" value="jtag"/>
 <part name="U$21" library="microbuilder" deviceset="3.3V" device=""/>
 <part name="U$22" library="microbuilder" deviceset="GND" device=""/>
@@
 <instance part="JP1" gate="A" x="129.54" y="124.46"/>
 <instance part="U$20" gate="G$1" x="121.92" y="121.92" rot="R90"/>
-<instance part="JP2" gate="A" x="180.34" y="111.76"/>
+<instance part="JTAG" gate="A" x="180.34" y="111.76"/>
 <instance part="U$21" gate="G$1" x="167.64" y="116.84" rot="R90"/>
 <instance part="U$22" gate="G$1" x="167.64" y="106.68" rot="R270"/>
@@
 </segment>
 <segment>
-<pinref part="JP2" gate="A" pin="1"/>
+<pinref part="JTAG" gate="A" pin="1"/>
 <pinref part="U$21" gate="G$1" pin="3.3V"/>
 <wire x1="170.18" y1="116.84" x2="177.8" y2="116.84" width="0.1524" layer="91"/>
@@
 </segment>
 <segment>
-<pinref part="JP2" gate="A" pin="5"/>
+<pinref part="JTAG" gate="A" pin="5"/>
 <pinref part="U$22" gate="G$1" pin="GND"/>
 <wire x1="177.8" y1="106.68" x2="170.18" y2="106.68" width="0.2032" layer="91"/>
@@
 <wire x1="15.24" y1="96.52" x2="12.7" y2="96.52" width="0.2032" layer="91"/>
 <label x="12.7" y="96.52" size="1.778" layer="95"/>
-</segment>
-<segment>
-<pinref part="JP2" gate="A" pin="4"/>
-<wire x1="177.8" y1="109.22" x2="170.18" y2="109.22" width="0.2032" layer="91"/>
-<label x="165.1" y="109.22" size="1.778" layer="95"/>
 </segment>
 <segment>
@@
 <wire x1="147.32" y1="33.02" x2="139.7" y2="33.02" width="0.2032" layer="91"/>
 <label x="139.7" y="33.02" size="1.778" layer="95"/>
+</segment>
+<segment>
+<pinref part="JTAG" gate="A" pin="2"/>
+<wire x1="177.8" y1="114.3" x2="170.18" y2="114.3" width="0.2032" layer="91"/>
+<label x="162.56" y="114.3" size="1.778" layer="95"/>
 </segment>
 </net>
@@
 </segment>
 <segment>
-<pinref part="JP2" gate="A" pin="3"/>
-<wire x1="177.8" y1="111.76" x2="170.18" y2="111.76" width="0.2032" layer="91"/>
-<label x="162.56" y="111.76" size="1.778" layer="95"/>
+<pinref part="JTAG" gate="A" pin="4"/>
+<wire x1="177.8" y1="109.22" x2="170.18" y2="109.22" width="0.2032" layer="91"/>
+<label x="165.1" y="109.22" size="1.778" layer="95"/>
 </segment>
 </net>
@@
 </segment>
 <segment>
-<pinref part="JP2" gate="A" pin="2"/>
-<wire x1="177.8" y1="114.3" x2="170.18" y2="114.3" width="0.2032" layer="91"/>
-<label x="162.56" y="114.3" size="1.778" layer="95"/>
+<pinref part="JTAG" gate="A" pin="3"/>
+<wire x1="177.8" y1="111.76" x2="170.18" y2="111.76" width="0.2032" layer="91"/>
+<label x="162.56" y="111.76" size="1.778" layer="95"/>
 </segment>
 </net>
@@
 <pinref part="LCD1" gate="G$1" pin="CLK"/>
 </segment>
+<segment>
+<pinref part="CPU1" gate="G$1" pin="PB3/JTDO"/>
+<wire x1="81.28" y1="88.9" x2="96.52" y2="88.9" width="0.2032" layer="91"/>
+<label x="88.9" y="88.9" size="1.778" layer="95"/>
+</segment>
 </net>
 <net name="LCD_MOSI" class="0">
@@
 <pinref part="LCD1" gate="G$1" pin="MOSI"/>
 </segment>
-</net>
-<net name="LCS_CS" class="0">
-<segment>
-<wire x1="132.08" y1="-5.08" x2="116.84" y2="-5.08" width="0.2032" layer="91"/>
-<label x="114.3" y="-5.08" size="1.778" layer="95"/>
-<pinref part="LCD1" gate="G$1" pin="CS"/>
+<segment>
+<pinref part="CPU1" gate="G$1" pin="PB5"/>
+<wire x1="81.28" y1="93.98" x2="96.52" y2="93.98" width="0.2032" layer="91"/>
+<label x="88.9" y="93.98" size="1.778" layer="95"/>
 </segment>
 </net>
@@
 <label x="114.3" y="-7.62" size="1.778" layer="95"/>
 <pinref part="LCD1" gate="G$1" pin="DC"/>
+</segment>
+<segment>
+<pinref part="CPU1" gate="G$1" pin="PB7"/>
+<wire x1="81.28" y1="99.06" x2="96.52" y2="99.06" width="0.2032" layer="91"/>
+<label x="88.9" y="99.06" size="1.778" layer="95"/>
 </segment>
 </net>
@@
 </segment>
 </net>
+<net name="LCD_MISO_UNUSED" class="0">
+<segment>
+<pinref part="CPU1" gate="G$1" pin="PB4/JTRST"/>
+<wire x1="81.28" y1="91.44" x2="96.52" y2="91.44" width="0.2032" layer="91"/>
+<label x="88.9" y="91.44" size="1.778" layer="95"/>
+</segment>
+</net>
+<net name="LCD_CS" class="0">
+<segment>
+<pinref part="CPU1" gate="G$1" pin="PB6"/>
+<wire x1="81.28" y1="96.52" x2="96.52" y2="96.52" width="0.2032" layer="91"/>
+<label x="88.9" y="96.52" size="1.778" layer="95"/>
+</segment>
+<segment>
+<wire x1="132.08" y1="-5.08" x2="116.84" y2="-5.08" width="0.2032" layer="91"/>
+<label x="114.3" y="-5.08" size="1.778" layer="95"/>
+<pinref part="LCD1" gate="G$1" pin="CS"/>
+</segment>
+</net>
