File: midimixer-channel.sch (EAGLE design)
At the start: 95 parts, among them IC1 74LS595D, IC2 74LS595D, IC3 74LS595D, IC4 74165D, U1 LM1117IMPX-3.3/NOPB, Y1 8MHz 695-HCM49-8-U

Commit message: wip
Parts:
- added JP2, JP5: (no value), microbuilder:HEADER-1X4ROUND
Connections:
- net 5.0V: now also JP2.1, JP5.1
- net CAN_H: now also JP2.2, JP5.2
- net CAN_L: now also JP2.3, JP5.3
- net GND: now also JP2.4, JP5.4
Changed lines of the file:
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@@
 <part name="U$116" library="microbuilder" deviceset="GND" device=""/>
 <part name="LCD1" library="keves" deviceset="SSD1306-ALI" device=""/>
+<part name="JP2" library="microbuilder" deviceset="HEADER-1X4" device="ROUND"/>
+<part name="U$1" library="microbuilder" deviceset="5.0V" device=""/>
+<part name="U$36" library="microbuilder" deviceset="GND" device=""/>
+<part name="JP5" library="microbuilder" deviceset="HEADER-1X4" device="ROUND"/>
 </parts>
 <sheets>
@@
 <instance part="R13" gate="G$1" x="109.22" y="106.68" rot="R180"/>
 <instance part="LCD1" gate="G$1" x="139.7" y="5.08"/>
+<instance part="JP2" gate="A" x="-12.7" y="-2.54" rot="R180"/>
+<instance part="U$1" gate="G$1" x="5.08" y="-7.62" rot="R270"/>
+<instance part="U$36" gate="G$1" x="5.08" y="0" rot="R90"/>
+<instance part="JP5" gate="A" x="-2.54" y="-2.54" rot="R180"/>
 </instances>
 <busses>
@@
 <wire x1="30.48" y1="-15.24" x2="27.94" y2="-15.24" width="0.1524" layer="91"/>
 </segment>
+<segment>
+<pinref part="JP2" gate="A" pin="4"/>
+<pinref part="U$36" gate="G$1" pin="GND"/>
+<wire x1="2.54" y1="0" x2="0" y2="0" width="0.1524" layer="91"/>
+<pinref part="JP5" gate="A" pin="4"/>
+<junction x="0" y="0"/>
+<wire x1="0" y1="0" x2="-10.16" y2="0" width="0.1524" layer="91"/>
+</segment>
 </net>
 <net name="NRST" class="0">
@@
 <junction x="132.08" y="60.96"/>
 <wire x1="132.08" y1="60.96" x2="137.16" y2="60.96" width="0.1524" layer="91"/>
+</segment>
+<segment>
+<pinref part="JP2" gate="A" pin="1"/>
+<pinref part="U$1" gate="G$1" pin="5.0V"/>
+<wire x1="2.54" y1="-7.62" x2="0" y2="-7.62" width="0.1524" layer="91"/>
+<pinref part="JP5" gate="A" pin="1"/>
+<junction x="0" y="-7.62"/>
+<wire x1="0" y1="-7.62" x2="-10.16" y2="-7.62" width="0.1524" layer="91"/>
 </segment>
 </net>
@@
 <label x="86.36" y="-10.16" size="1.778" layer="95"/>
 </segment>
+<segment>
+<pinref part="JP2" gate="A" pin="3"/>
+<wire x1="0" y1="-2.54" x2="15.24" y2="-2.54" width="0.2032" layer="91"/>
+<label x="12.7" y="-2.54" size="1.778" layer="95"/>
+<pinref part="JP5" gate="A" pin="3"/>
+<junction x="0" y="-2.54"/>
+<wire x1="0" y1="-2.54" x2="-10.16" y2="-2.54" width="0.1524" layer="91"/>
+</segment>
 </net>
 <net name="CAN_H" class="0">
@@
 <label x="86.36" y="0" size="1.778" layer="95"/>
 </segment>
+<segment>
+<pinref part="JP2" gate="A" pin="2"/>
+<wire x1="0" y1="-5.08" x2="15.24" y2="-5.08" width="0.2032" layer="91"/>
+<label x="12.7" y="-5.08" size="1.778" layer="95"/>
+<pinref part="JP5" gate="A" pin="2"/>
+<junction x="0" y="-5.08"/>
+<wire x1="0" y1="-5.08" x2="-10.16" y2="-5.08" width="0.1524" layer="91"/>
+</segment>
 </net>
 <net name="CAN_TX" class="0">
+<segment>
+<pinref part="R14" gate="G$1" pin="1"/>
+<wire x1="114.3" y1="104.14" x2="119.38" y2="104.14" width="0.2032" layer="91"/>
+<label x="116.84" y="104.14" size="1.778" layer="95"/>
+</segment>
 <segment>
 <pinref part="D2" gate="G$1" pin="TXD"/>
@@
 <label x="27.94" y="-2.54" size="1.778" layer="95"/>
 </segment>
-<segment>
-<pinref part="R14" gate="G$1" pin="1"/>
-<wire x1="114.3" y1="104.14" x2="119.38" y2="104.14" width="0.2032" layer="91"/>
-<label x="116.84" y="104.14" size="1.778" layer="95"/>
-</segment>
-</net>
+</net>
