File: midimixer-channel.brd (EAGLE design)
At the start: 50.8 x 277.8 mm, 90 parts, among them IC1 74LS595D, IC2 74LS595D, IC3 74LS595D, IC4 74LS595D, U1 LM1117IMPX-3.3/NOPB, Y1 8MHz 695-HCM49-8-U

Commit message: wip
Parts:
- added C25: 0.1uF, microbuilder:0603
- added D2: SN65HVD230, omc:SO8
- added R18: 0, microbuilder:_0603
- added R27: 120, microbuilder:_0603
Connections:
- removed net N$13: IC1.14
- removed net N$27: U$87.9
- removed net N$58: IC1.11, IC3.11, IC4.11, U$87.2
- removed net N$59: IC1.12, IC3.12, IC4.12, U$87.1
- new net CAN_H: D2.7, R27.1
- new net CAN_L: D2.6, R27.2
- new net CAN_RX: D2.4
- new net CAN_TX: D2.1
- new net N$73: D2.8, R18.1
- new net SPI2_CLK: IC1.11, IC3.11, IC4.11, U$1.34, U$87.2
- new net SPI2_MISO: U$1.35, U$87.9
- new net SPI2_MOSI: IC1.14, U$1.36
- new net SPI2_RC1: IC1.12, IC3.12, IC4.12, U$1.33
- new net SPI2_RC2: U$1.37, U$87.1
- net 3.3V: now also C25.1, D2.3
- net GND: now also C25.2, D2.2, R18.2
Changed lines of the file:
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@@
 <layer number="23" name="tOrigins" color="15" fill="1" visible="yes" active="yes"/>
 <layer number="24" name="bOrigins" color="15" fill="1" visible="yes" active="yes"/>
-<layer number="25" name="tNames" color="7" fill="1" visible="yes" active="yes"/>
-<layer number="26" name="bNames" color="7" fill="1" visible="yes" active="yes"/>
-<layer number="27" name="tValues" color="7" fill="1" visible="yes" active="yes"/>
-<layer number="28" name="bValues" color="7" fill="1" visible="yes" active="yes"/>
+<layer number="25" name="tNames" color="7" fill="1" visible="no" active="yes"/>
+<layer number="26" name="bNames" color="7" fill="1" visible="no" active="yes"/>
+<layer number="27" name="tValues" color="7" fill="1" visible="no" active="yes"/>
+<layer number="28" name="bValues" color="7" fill="1" visible="no" active="yes"/>
 <layer number="29" name="tStop" color="7" fill="3" visible="no" active="yes"/>
 <layer number="30" name="bStop" color="7" fill="6" visible="no" active="yes"/>
@@
 <layer number="230" name="230bmp" color="7" fill="1" visible="no" active="yes"/>
 <layer number="231" name="231bmp" color="7" fill="1" visible="no" active="yes"/>
+<layer number="232" name="Eagle3D_PG2" color="14" fill="2" visible="yes" active="yes"/>
+<layer number="233" name="Eagle3D_PG3" color="14" fill="4" visible="yes" active="yes"/>
 <layer number="248" name="Housing" color="7" fill="1" visible="no" active="yes"/>
 <layer number="249" name="Edge" color="7" fill="1" visible="no" active="yes"/>
@@
 <element name="R25" library="microbuilder" package="_0603" value="10k" x="-52.07" y="-218.44"/>
 <element name="R26" library="microbuilder" package="_0603" value="10k" x="-52.07" y="-223.52"/>
+<element name="D2" library="omc" package="SO8" value="SN65HVD230" x="-50.8" y="-229.87"/>
+<element name="C25" library="microbuilder" package="0603" value="0.1uF" x="-53.34" y="-234.95"/>
+<element name="R18" library="microbuilder" package="_0603" value="0" x="-52.07" y="-238.76"/>
+<element name="R27" library="microbuilder" package="_0603" value="120" x="-52.07" y="-243.84"/>
 </elements>
 <signals>
@@
 <contactref element="R24" pad="2"/>
 <contactref element="R25" pad="2"/>
+<contactref element="C25" pad="1"/>
+<contactref element="D2" pad="3"/>
 <wire x1="-51.308" y1="-193.04" x2="-51.308" y2="-198.12" width="0" layer="19" extent="1-1"/>
 <wire x1="-51.308" y1="-187.96" x2="-51.308" y2="-193.04" width="0" layer="19" extent="1-1"/>
@@
 <wire x1="-51.308" y1="-218.44" x2="-51.308" y2="-213.36" width="0" layer="19" extent="1-1"/>
 <wire x1="-51.308" y1="-223.52" x2="-51.308" y2="-218.44" width="0" layer="19" extent="1-1"/>
+<wire x1="-50.165" y1="-232.67" x2="-51.308" y2="-223.52" width="0" layer="19" extent="1-1"/>
+<wire x1="-54.19" y1="-234.95" x2="-50.165" y2="-232.67" width="0" layer="19" extent="1-1"/>
 <wire x1="-51.308" y1="-177.8" x2="-51.308" y2="-187.96" width="0" layer="19" extent="1-1"/>
 <wire x1="-52.49" y1="-173.99" x2="-51.308" y2="-177.8" width="0" layer="19" extent="1-1"/>
@@
 <contactref element="C24" pad="1"/>
 <contactref element="U$87" pad="15"/>
+<contactref element="D2" pad="2"/>
+<contactref element="C25" pad="2"/>
+<contactref element="R18" pad="2"/>
 <wire x1="-50.165" y1="-166.11" x2="-54.19" y2="-173.99" width="0" layer="19" extent="1-1"/>
 <wire x1="-52.49" y1="-162.56" x2="-50.165" y2="-166.11" width="0" layer="19" extent="1-1"/>
@@
 <wire x1="20.06" y1="106.045" x2="25.66" y2="99.695" width="0" layer="19" extent="1-1"/>
 <wire x1="25.66" y1="111.125" x2="20.06" y2="106.045" width="0" layer="19" extent="1-1"/>
+<wire x1="-51.435" y1="-232.67" x2="-54.19" y2="-173.99" width="0" layer="19" extent="1-1"/>
+<wire x1="-52.49" y1="-234.95" x2="-51.435" y2="-232.67" width="0" layer="19" extent="1-1"/>
+<wire x1="-51.308" y1="-238.76" x2="-52.49" y2="-234.95" width="0" layer="19" extent="1-1"/>
 </signal>
 <signal name="NRST">
@@
 <wire x1="25.66" y1="100.965" x2="25.66" y2="106.045" width="0" layer="19" extent="1-1"/>
 </signal>
-<signal name="N$58">
+<signal name="SPI2_CLK">
 <contactref element="IC3" pad="11"/>
 <contactref element="IC1" pad="11"/>
 <contactref element="IC4" pad="11"/>
 <contactref element="U$87" pad="2"/>
-<wire x1="34.55" y1="33.655" x2="-50.165" y2="-171.71" width="0" layer="19" extent="1-1"/>
+<contactref element="U$1" pad="34"/>
+<wire x1="41.35" y1="24.8" x2="-50.165" y2="-171.71" width="0" layer="19" extent="1-1"/>
+<wire x1="34.55" y1="33.655" x2="41.35" y2="24.8" width="0" layer="19" extent="1-1"/>
 <wire x1="25.66" y1="97.155" x2="34.55" y2="33.655" width="0" layer="19" extent="1-1"/>
 <wire x1="25.66" y1="108.585" x2="25.66" y2="97.155" width="0" layer="19" extent="1-1"/>
 </signal>
-<signal name="N$59">
+<signal name="SPI2_RC1">
 <contactref element="IC1" pad="12"/>
 <contactref element="IC3" pad="12"/>
 <contactref element="IC4" pad="12"/>
-<contactref element="U$87" pad="1"/>
-<wire x1="34.55" y1="34.925" x2="-51.435" y2="-171.71" width="0" layer="19" extent="1-1"/>
-<wire x1="25.66" y1="98.425" x2="34.55" y2="34.925" width="0" layer="19" extent="1-1"/>
-<wire x1="25.66" y1="109.855" x2="25.66" y2="98.425" width="0" layer="19" extent="1-1"/>
+<contactref element="U$1" pad="33"/>
+<wire x1="25.66" y1="98.425" x2="25.66" y2="109.855" width="0" layer="19" extent="1-1"/>
+<wire x1="34.55" y1="34.925" x2="25.66" y2="98.425" width="0" layer="19" extent="1-1"/>
+<wire x1="41.85" y1="24.8" x2="34.55" y2="34.925" width="0" layer="19" extent="1-1"/>
 </signal>
 <signal name="N$60">
@@
 <contactref element="IC4" pad="9"/>
 </signal>
-<signal name="N$13">
+<signal name="SPI2_MOSI">
 <contactref element="IC1" pad="14"/>
-</signal>
-<signal name="N$27">
+<contactref element="U$1" pad="36"/>
+<wire x1="40.35" y1="24.8" x2="25.66" y2="112.395" width="0" layer="19" extent="1-1"/>
+</signal>
+<signal name="SPI2_MISO">
 <contactref element="U$87" pad="9"/>
+<contactref element="U$1" pad="35"/>
+<wire x1="40.85" y1="24.8" x2="-42.545" y2="-166.11" width="0" layer="19" extent="1-1"/>
 </signal>
 <signal name="N$28">
@@
 <wire x1="-45.085" y1="-171.71" x2="-52.832" y2="-187.96" width="0" layer="19" extent="1-1"/>
 </signal>
+<signal name="N$73">
+<contactref element="D2" pad="8"/>
+<contactref element="R18" pad="1"/>
+<wire x1="-52.705" y1="-227.07" x2="-52.832" y2="-238.76" width="0" layer="19" extent="1-1"/>
+</signal>
+<signal name="CAN_L">
+<contactref element="D2" pad="6"/>
+<contactref element="R27" pad="2"/>
+<wire x1="-50.165" y1="-227.07" x2="-51.308" y2="-243.84" width="0" layer="19" extent="1-1"/>
+</signal>
+<signal name="CAN_H">
+<contactref element="D2" pad="7"/>
+<contactref element="R27" pad="1"/>
+<wire x1="-51.435" y1="-227.07" x2="-52.832" y2="-243.84" width="0" layer="19" extent="1-1"/>
+</signal>
+<signal name="CAN_TX">
+<contactref element="D2" pad="1"/>
+</signal>
+<signal name="CAN_RX">
+<contactref element="D2" pad="4"/>
+</signal>
+<signal name="SPI2_RC2">
+<contactref element="U$87" pad="1"/>
+<contactref element="U$1" pad="37"/>
+<wire x1="39.85" y1="24.8" x2="-51.435" y2="-171.71" width="0" layer="19" extent="1-1"/>
+</signal>
 </signals>

Commit message: wip
Connections:
- removed net N$32: U$47.LED1+
- removed net N$33: U$47.LED2+
- removed net N$37: U$51.LED1+
- removed net N$38: U$51.LED2+
- removed net N$47: U$59.LED1+
- removed net N$48: U$59.LED2+
- net 3.3V: now also U$42.P3, U$65.P3, U$66.P3, U$67.P3, U$68.P3
- net BTN_LED10: now also U$51.LED2+
- net BTN_LED11: now also U$59.LED1+
- net BTN_LED12: now also U$59.LED2+
- net BTN_LED7: now also U$47.LED1+
- net BTN_LED8: now also U$47.LED2+
- net BTN_LED9: now also U$51.LED1+
- net GND: now also U$42.P1, U$65.P1, U$66.P1, U$67.P1, U$68.P1, U$69.P1, U$70.P1, U$71.P1
Changed lines of the file:
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@@
 <contactref element="C25" pad="1"/>
 <contactref element="D2" pad="3"/>
+<contactref element="U$42" pad="P3"/>
+<contactref element="U$65" pad="P3"/>
+<contactref element="U$66" pad="P3"/>
+<contactref element="U$67" pad="P3"/>
+<contactref element="U$68" pad="P3"/>
 <wire x1="-51.308" y1="-193.04" x2="-51.308" y2="-198.12" width="0" layer="19" extent="1-1"/>
 <wire x1="-51.308" y1="-187.96" x2="-51.308" y2="-193.04" width="0" layer="19" extent="1-1"/>
@@
 <wire x1="43.85" y1="22.8" x2="34.35" y2="24.8" width="0" layer="19" extent="1-1"/>
 <wire x1="43.85" y1="16.3" x2="43.85" y2="22.8" width="0" layer="19" extent="1-1"/>
-<wire x1="25.66" y1="95.885" x2="34.55" y2="40.005" width="0" layer="19" extent="1-1"/>
+<wire x1="10.95" y1="81.2" x2="34.55" y2="40.005" width="0" layer="19" extent="1-1"/>
+<wire x1="25.66" y1="95.885" x2="10.95" y2="81.2" width="0" layer="19" extent="1-1"/>
 <wire x1="25.66" y1="103.505" x2="25.66" y2="95.885" width="0" layer="19" extent="1-1"/>
 <wire x1="25.66" y1="107.315" x2="25.66" y2="103.505" width="0" layer="19" extent="1-1"/>
 <wire x1="25.66" y1="114.935" x2="25.66" y2="107.315" width="0" layer="19" extent="1-1"/>
+<wire x1="13.95" y1="114.3" x2="25.66" y2="114.935" width="0" layer="19" extent="1-1"/>
+<wire x1="39.35" y1="88.9" x2="25.66" y2="95.885" width="0" layer="19" extent="1-1"/>
+<wire x1="13.95" y1="139.7" x2="13.95" y2="114.3" width="0" layer="19" extent="1-1"/>
+<wire x1="13.95" y1="165.1" x2="13.95" y2="139.7" width="0" layer="19" extent="1-1"/>
 </signal>
 <signal name="N$1">
@@
 <contactref element="C25" pad="2"/>
 <contactref element="R18" pad="2"/>
+<contactref element="U$42" pad="P1"/>
+<contactref element="U$69" pad="P1"/>
+<contactref element="U$70" pad="P1"/>
+<contactref element="U$71" pad="P1"/>
+<contactref element="U$68" pad="P1"/>
+<contactref element="U$67" pad="P1"/>
+<contactref element="U$66" pad="P1"/>
+<contactref element="U$65" pad="P1"/>
 <wire x1="-50.165" y1="-166.11" x2="-54.19" y2="-173.99" width="0" layer="19" extent="1-1"/>
 <wire x1="-52.49" y1="-162.56" x2="-50.165" y2="-166.11" width="0" layer="19" extent="1-1"/>
@@
 <wire x1="-14.91" y1="-22.86" x2="-7.64" y2="-20.15" width="0" layer="19" extent="1-1"/>
 <wire x1="11.85" y1="-16.51" x2="3.49" y2="-17.78" width="0" layer="19" extent="1-1"/>
-<wire x1="-32.17" y1="6.35" x2="-14.91" y2="-22.86" width="0" layer="19" extent="1-1"/>
-<wire x1="-32.17" y1="8.89" x2="-32.17" y2="6.35" width="0" layer="19" extent="1-1"/>
-<wire x1="-38.52" y1="6.35" x2="-32.17" y2="6.35" width="0" layer="19" extent="1-1"/>
-<wire x1="-38.52" y1="3.81" x2="-38.52" y2="6.35" width="0" layer="19" extent="1-1"/>
-<wire x1="-40.22" y1="8.89" x2="-38.52" y2="6.35" width="0" layer="19" extent="1-1"/>
-<wire x1="-30.06" y1="21.59" x2="-32.17" y2="8.89" width="0" layer="19" extent="1-1"/>
-<wire x1="-32.17" y1="36.83" x2="-30.06" y2="21.59" width="0" layer="19" extent="1-1"/>
-<wire x1="-32.17" y1="39.37" x2="-32.17" y2="36.83" width="0" layer="19" extent="1-1"/>
-<wire x1="-25.82" y1="36.83" x2="-32.17" y2="36.83" width="0" layer="19" extent="1-1"/>
-<wire x1="-38.52" y1="36.83" x2="-32.17" y2="36.83" width="0" layer="19" extent="1-1"/>
-<wire x1="-40.22" y1="39.37" x2="-38.52" y2="36.83" width="0" layer="19" extent="1-1"/>
-<wire x1="-30.06" y1="52.07" x2="-32.17" y2="39.37" width="0" layer="19" extent="1-1"/>
-<wire x1="-38.52" y1="67.31" x2="-30.06" y2="52.07" width="0" layer="19" extent="1-1"/>
-<wire x1="-40.22" y1="69.85" x2="-38.52" y2="67.31" width="0" layer="19" extent="1-1"/>
-<wire x1="-32.17" y1="69.85" x2="-38.52" y2="67.31" width="0" layer="19" extent="1-1"/>
-<wire x1="32.35" y1="15.8" x2="11.85" y2="-16.51" width="0" layer="19" extent="1-1"/>
+<wire x1="10.95" y1="7.7" x2="1.69" y2="-10.16" width="0" layer="19" extent="1-1"/>
+<wire x1="32.35" y1="15.8" x2="10.95" y2="7.7" width="0" layer="19" extent="1-1"/>
 <wire x1="39.85" y1="13.3" x2="32.35" y2="15.8" width="0" layer="19" extent="1-1"/>
 <wire x1="43.85" y1="15.8" x2="39.85" y2="13.3" width="0" layer="19" extent="1-1"/>
@@
 <wire x1="28.65" y1="73.95" x2="34.85" y2="73.95" width="0" layer="19" extent="1-1"/>
 <wire x1="22.15" y1="73.95" x2="28.65" y2="73.95" width="0" layer="19" extent="1-1"/>
-<wire x1="5.08" y1="81.28" x2="22.15" y2="73.95" width="0" layer="19" extent="1-1"/>
-<wire x1="5.08" y1="97.79" x2="5.08" y2="81.28" width="0" layer="19" extent="1-1"/>
-<wire x1="20.06" y1="94.615" x2="5.08" y2="97.79" width="0" layer="19" extent="1-1"/>
-<wire x1="25.66" y1="99.695" x2="20.06" y2="94.615" width="0" layer="19" extent="1-1"/>
+<wire x1="34.35" y1="88.9" x2="34.85" y2="73.95" width="0" layer="19" extent="1-1"/>
+<wire x1="25.66" y1="99.695" x2="34.35" y2="88.9" width="0" layer="19" extent="1-1"/>
+<wire x1="20.06" y1="94.615" x2="25.66" y2="99.695" width="0" layer="19" extent="1-1"/>
 <wire x1="20.06" y1="106.045" x2="25.66" y2="99.695" width="0" layer="19" extent="1-1"/>
 <wire x1="25.66" y1="111.125" x2="20.06" y2="106.045" width="0" layer="19" extent="1-1"/>
+<wire x1="34.35" y1="114.3" x2="25.66" y2="111.125" width="0" layer="19" extent="1-1"/>
+<wire x1="8.95" y1="114.3" x2="20.06" y2="106.045" width="0" layer="19" extent="1-1"/>
+<wire x1="5.08" y1="97.79" x2="20.06" y2="94.615" width="0" layer="19" extent="1-1"/>
+<wire x1="5.08" y1="81.28" x2="5.08" y2="97.79" width="0" layer="19" extent="1-1"/>
+<wire x1="34.35" y1="139.7" x2="34.35" y2="114.3" width="0" layer="19" extent="1-1"/>
+<wire x1="34.35" y1="165.1" x2="34.35" y2="139.7" width="0" layer="19" extent="1-1"/>
+<wire x1="8.95" y1="165.1" x2="34.35" y2="165.1" width="0" layer="19" extent="1-1"/>
+<wire x1="8.95" y1="139.7" x2="8.95" y2="114.3" width="0" layer="19" extent="1-1"/>
+<wire x1="-32.17" y1="6.35" x2="-14.91" y2="-22.86" width="0" layer="19" extent="1-1"/>
+<wire x1="-32.17" y1="8.89" x2="-32.17" y2="6.35" width="0" layer="19" extent="1-1"/>
+<wire x1="-38.52" y1="6.35" x2="-32.17" y2="6.35" width="0" layer="19" extent="1-1"/>
+<wire x1="-38.52" y1="3.81" x2="-38.52" y2="6.35" width="0" layer="19" extent="1-1"/>
+<wire x1="-40.22" y1="8.89" x2="-38.52" y2="6.35" width="0" layer="19" extent="1-1"/>
+<wire x1="-30.06" y1="21.59" x2="-32.17" y2="8.89" width="0" layer="19" extent="1-1"/>
+<wire x1="-32.17" y1="36.83" x2="-30.06" y2="21.59" width="0" layer="19" extent="1-1"/>
+<wire x1="-32.17" y1="39.37" x2="-32.17" y2="36.83" width="0" layer="19" extent="1-1"/>
+<wire x1="-25.82" y1="36.83" x2="-32.17" y2="36.83" width="0" layer="19" extent="1-1"/>
+<wire x1="-38.52" y1="36.83" x2="-32.17" y2="36.83" width="0" layer="19" extent="1-1"/>
+<wire x1="-40.22" y1="39.37" x2="-38.52" y2="36.83" width="0" layer="19" extent="1-1"/>
+<wire x1="-30.06" y1="52.07" x2="-32.17" y2="39.37" width="0" layer="19" extent="1-1"/>
+<wire x1="-38.52" y1="67.31" x2="-30.06" y2="52.07" width="0" layer="19" extent="1-1"/>
+<wire x1="-40.22" y1="69.85" x2="-38.52" y2="67.31" width="0" layer="19" extent="1-1"/>
+<wire x1="-32.17" y1="69.85" x2="-38.52" y2="67.31" width="0" layer="19" extent="1-1"/>
 <wire x1="-51.435" y1="-232.67" x2="-54.19" y2="-173.99" width="0" layer="19" extent="1-1"/>
 <wire x1="-52.49" y1="-234.95" x2="-51.435" y2="-232.67" width="0" layer="19" extent="1-1"/>
@@
 <wire x1="-28.36" y1="52.07" x2="22.15" y2="50.51" width="0" layer="19" extent="1-1"/>
 </signal>
-<signal name="N$32">
-<contactref element="U$47" pad="LED1+"/>
-</signal>
-<signal name="N$33">
-<contactref element="U$47" pad="LED2+"/>
-</signal>
 <signal name="N$34">
 <contactref element="U$51" pad="LED1-"/>
@@
 <wire x1="-38.52" y1="39.37" x2="34.85" y2="50.51" width="0" layer="19" extent="1-1"/>
 </signal>
-<signal name="N$37">
-<contactref element="U$51" pad="LED1+"/>
-</signal>
-<signal name="N$38">
-<contactref element="U$51" pad="LED2+"/>
-</signal>
 <signal name="N$39">
 <contactref element="U$55" pad="LED1-"/>
@@
 <wire x1="22.15" y1="64.48" x2="28.65" y2="64.48" width="0" layer="19" extent="1-1"/>
 <wire x1="-38.52" y1="8.89" x2="22.15" y2="64.48" width="0" layer="19" extent="1-1"/>
-</signal>
-<signal name="N$47">
-<contactref element="U$59" pad="LED1+"/>
-</signal>
-<signal name="N$48">
-<contactref element="U$59" pad="LED2+"/>
 </signal>
 <signal name="VCC">
@@
 <signal name="BTN_LED7">
 <contactref element="IC4" pad="15"/>
+<contactref element="U$47" pad="LED1+"/>
+<wire x1="34.55" y1="38.735" x2="25.4" y2="51.86" width="0" layer="19" extent="1-1"/>
 </signal>
 <signal name="BTN_LED8">
 <contactref element="IC4" pad="1"/>
+<contactref element="U$47" pad="LED2+"/>
+<wire x1="28.95" y1="40.005" x2="25.4" y2="44.66" width="0" layer="19" extent="1-1"/>
 </signal>
 <signal name="BTN_LED9">
 <contactref element="IC4" pad="2"/>
+<contactref element="U$51" pad="LED1+"/>
+<wire x1="28.95" y1="38.735" x2="38.1" y2="51.86" width="0" layer="19" extent="1-1"/>
 </signal>
 <signal name="BTN_LED10">
 <contactref element="IC4" pad="3"/>
+<contactref element="U$51" pad="LED2+"/>
+<wire x1="28.95" y1="37.465" x2="38.1" y2="44.66" width="0" layer="19" extent="1-1"/>
 </signal>
 <signal name="BTN_LED11">
 <contactref element="IC4" pad="4"/>
+<contactref element="U$59" pad="LED1+"/>
+<wire x1="28.95" y1="36.195" x2="25.4" y2="65.83" width="0" layer="19" extent="1-1"/>
 </signal>
 <signal name="BTN_LED12">
 <contactref element="IC4" pad="5"/>
+<contactref element="U$59" pad="LED2+"/>
+<wire x1="28.95" y1="34.925" x2="25.4" y2="58.63" width="0" layer="19" extent="1-1"/>
 </signal>
 <signal name="N$63">

Commit message: wip
Parts:
- removed IC2: 74LS595D, SparkFun-DigitalIC:SO16
- removed JP4: (no value), microbuilder:1X06_ROUND_70
- added R28, R29: 0, microbuilder:_0603
- added U$117: SSD1306-ALI, keves:SSD1306-ALI
- moved C23 277.4 mm to (24.3, 103.8), turned to 180 degrees
- moved C21 264.1 mm to (28.3, 93.7), turned to 180 degrees
- moved C22 216.0 mm to (37.2, 36.1), turned to 270 degrees
- moved C2 54.9 mm to (48.3, 17.8), turned to 90 degrees
- moved C8 51.3 mm to (40.6, 6.35), turned to 270 degrees
- moved C1 50.0 mm to (48.3, 10.2), turned to 270 degrees
- moved C3 49.6 mm to (34.3, 22.9)
- moved R1 49.5 mm to (35.6, 5.08), turned to 270 degrees
- moved C4 49.0 mm to (27.9, 24.1), turned to 180 degrees
- moved C7 43.0 mm to (26.7, 10.2), turned to 90 degrees
- moved Y1 41.5 mm to (44.5, 14.0), turned to 270 degrees
- moved C5 41.0 mm to (27.9, 21.6)
- moved C6 40.5 mm to (24.1, 11.4), turned to 270 degrees
- moved IC1 13.0 mm to (22.4, 97.5)
- moved IC3 12.2 mm to (23.6, 86.9)
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Connections:
- removed net N$60: D1.2, IC3.15
- removed net N$61: D1.1, IC3.1
- removed net N$62: R24.1, U$87.13
- removed net N$63: IC4.6
- removed net N$64: IC4.7
- removed net N$66: R23.1, U$87.14
- removed net N$67: R22.1, U$87.3
- removed net N$68: R21.1, U$87.4
- removed net N$69: R20.1, U$87.5
- removed net N$70: R19.1, U$87.6
- removed net VCC: IC2.16
- new net BTN_UNUSED1: IC4.1
- new net BTN_UUSED2: IC4.15
- new net DIN_1: R26.1, U$63.A, U$87.11
- new net DIN_2: R25.1, U$63.B, U$87.12
- new net DIN_3: R24.1, U$63.S2, U$87.13
- new net DIN_4: R23.1, U$64.A, U$87.14
- new net DIN_5: R22.1, U$64.B, U$87.3
- new net DIN_6: R21.1, U$64.S2, U$87.4
- new net DIN_7: C15.2, R20.1, U$36.SW3, U$36.SW4, U$87.5
- new net DIN_8: C17.2, R19.1, U$47.SW3, U$47.SW4, U$87.6
- new net N$13: R29.2, U$1.62
- new net N$27: R28.2, U$1.61
- new net N$32: U$42.P2
- new net N$33: U$65.P2
- new net N$37: U$69.P2
- new net N$38: U$70.P2
- new net N$47: U$71.P2
- new net N$48: U$68.P2
- net 3.3V: now also U$117.P$1, U$69.P3, U$70.P3, U$71.P3; no longer JP4.1
- net BTN_LED1: now also IC3.15; no longer IC3.2
- net BTN_LED10: now also IC4.2; no longer IC4.3
- net BTN_LED3: now also IC3.5; no longer IC3.4
- net BTN_LED4: now also IC3.7; no longer IC3.5
- net BTN_LED5: now also IC3.4; no longer IC3.6
- net BTN_LED6: now also IC4.3, U$51.LED1+; no longer IC3.7, U$36.LED2+
- net BTN_LED7: now also IC4.6; no longer IC4.15
- net BTN_LED8: now also IC4.7; no longer IC4.1
- net BTN_LED9: now also IC3.6, U$36.LED2+; no longer IC4.2, U$51.LED1+
- net CAN_RX: now also R29.1
- net CAN_TX: now also R28.1
- net GND: now also U$117.P$2, U$63.C, U$63.S1, U$64.C, U$64.S1; no longer IC2.8, JP4.2
- net LCD_CLK: now also U$117.P$3; no longer JP4.3
- net LCD_DC: now also U$117.P$6; no longer JP4.6
- net LCD_MOSI: now also U$117.P$4; no longer JP4.4
- net LCS_CS: now also U$117.P$5; no longer JP4.5
- net N$11: now also D1.2, IC3.1; no longer C15.2, U$36.SW3, U$36.SW4
- net N$31: now also D1.1, IC3.2; no longer C17.2, U$47.SW3, U$47.SW4
- net N$42: now also U$66.P2; no longer R26.1, U$87.11
- net N$43: now also U$67.P2; no longer R25.1, U$87.12
Routing:
- net SPI2_MOSI: track 0.00 -> 71.9 mm, vias 0 -> 1
- net SPI2_RC1: track 0.00 -> 67.6 mm, vias 0 -> 2
- net SPI2_CLK: track 0.00 -> 65.7 mm, vias 0 -> 3
- net N$12: track 0.00 -> 52.2 mm, vias 0 -> 2
- net BTN_LED9: track 0.00 -> 40.2 mm
- net BTN_LED5: track 0.00 -> 35.6 mm
- net BTN_LED2: track 0.00 -> 29.2 mm
- net BTN_LED11: track 0.00 -> 28.0 mm
- net BTN_LED12: track 0.00 -> 20.3 mm
- net 3.3V: track 0.00 -> 17.9 mm, vias 0 -> 5
- net BTN_LED1: track 0.00 -> 16.9 mm
- net BTN_LED4: track 0.00 -> 13.7 mm
- net BTN_LED6: track 0.00 -> 13.6 mm
- net BTN_LED7: track 0.00 -> 13.0 mm
- net N$49: track 0.00 -> 12.6 mm
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- added copper zone on layer 16, net 3.3V
- added copper zone on layer 1, net GND
Other:
- board size 50.8 x 277.8 mm -> 50.8 x 241.3 mm
