File: midimixer-channel.brd (EAGLE design)
At the start: 50.8 x 241.3 mm, 95 parts, among them IC1 74LS595D, IC3 74LS595D, IC4 74LS595D, U1 LM1117IMPX-3.3/NOPB, Y1 8MHz 695-HCM49-8-U

Commit message: wip
Parts:
- removed SWD: (no value), microbuilder:1X05_ROUND_76
- removed U$87: 74165D, SparkFun-DigitalIC:SO16
- added IC2: 74LS595D, SparkFun-DigitalIC:SO16
- added JP4: (no value), microbuilder:1X02_ROUND
- C1, C2: value 18pf -> 0.1uF
- C10, C11, C9: value 10uF 603-CC206KKX5R7BB106 -> 0.1uF; device SparkFun-Passives:1206 -> microbuilder:0603
- C13, C7: value 0.1uF -> 2.2uF 810-CGJ4J2X7R1A225K; device microbuilder:0603 -> microbuilder:0805
- C15, C17, C18: value 0.1uF -> 10uF 603-CC206KKX5R7BB106; device microbuilder:0603 -> SparkFun-Passives:1206
- C4: value 2.2uF 810-CGJ4J2X7R1A225K -> 0.1uF; device microbuilder:0805 -> microbuilder:0603
- C5: value 0.1uF -> 18pf
- C6: value 2.2uF 810-CGJ4J2X7R1A225K -> 18pf; device microbuilder:0805 -> microbuilder:0603
- IC4: value 74LS595D -> 74165D
- JP2: device microbuilder:1X02_ROUND -> microbuilder:1X05_ROUND_76
- R10, R13, R14: value 330 -> 0; device microbuilder:0603 -> microbuilder:_0603
- R11: value 330 -> 120; device microbuilder:0603 -> microbuilder:_0603
- R12, R4, R5, R6, R7, R8, R9: value 330 -> 10k; device microbuilder:0603 -> microbuilder:_0603
- R15, R16: value 330 -> 22
- R17, R19, R20, R21, R22, R23, R24, R25, R26: value 10k -> 330; device microbuilder:_0603 -> microbuilder:0603
- R18, R28, R29: value 0 -> 330; device microbuilder:_0603 -> microbuilder:0603
- R2, R3: value 22 -> 10k; device microbuilder:0603 -> microbuilder:_0603
- R27: value 120 -> 330; device microbuilder:_0603 -> microbuilder:0603
- moved R29 325.8 mm to (23.9, 62.9), flipped to the bottom, turned to 90 degrees
- moved R28 316.5 mm to (28.8, 57.0), flipped to the bottom, turned to 270 degrees
- moved R18 315.0 mm to (39.5, 62.6), flipped to the bottom, turned to 270 degrees
- moved C25 310.7 mm to (22.7, 66.3), flipped to the bottom
- moved R27 305.1 mm to (36.2, 48.3), flipped to the bottom, turned to 90 degrees
- moved R6 301.1 mm to (16.0, 192.7), flipped to the bottom, turned to 180 degrees
- moved R5 297.2 mm to (9.27, 192.8), flipped to the bottom
- moved R23 297.2 mm to (36.7, 75.3), flipped to the bottom, turned to 270 degrees
- moved R22 293.1 mm to (39.2, 75.3), flipped to the bottom, turned to 270 degrees
- moved R26 284.7 mm to (38.7, 46.4), flipped to the bottom
- moved R21 283.8 mm to (24.0, 75.3), flipped to the bottom, turned to 270 degrees
- moved R11 281.0 mm to (-52.1, -243.8)
- moved R10 278.8 mm to (-52.1, -238.8)
- moved R25 278.3 mm to (23.9, 49.3), flipped to the bottom, turned to 90 degrees
- moved R24 278.0 mm to (29.6, 52.3), flipped to the bottom
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- renumbered U$1 to CPU1, U$117 to LCD1, U$36 to BTN1, U$42 to FADER1, U$43 to BTN2, U$47 to BTN4, U$51 to BTN5, U$55 to BTN3, U$59 to BTN6, U$63 to ROTENC1, U$64 to ROTENC2, U$65 to POT1, U$66 to POT2, U$67 to POT3, U$68 to POT4, U$69 to POT5, U$70 to POT6, U$71 to POT7, USB to X1
Connections:
- net 3.3V: now also C1.2, C10.1, C11.1, C12.2, C17.2, C2.1, C3.2, C4.2, C9.2, IC2.10, IC2.16, JP2.1, JP4.1, R1.2, R2.2, R3.2, R5.2, R6.2, R7.2, R8.2, R9.2; no longer C10.2, C21.2, C22.2, C23.1, C24.2, C25.1, C3.1, C5.2, C7.2, IC4.10, JP3.1, R19.2, R20.2, R21.2, R22.2, R23.2, R24.2, R25.2, R26.2, SWD.1, U$87.16
- net 5.0V: now also C15.2, JP3.1; no longer C9.2, JP2.1
- net AVDD: now also C18.2, C19.1; no longer C11.2, C12.1
- net BTN_LED1: now also IC2.15; no longer IC3.15
- net BTN_LED10: now also IC1.2; no longer IC4.2
- net BTN_LED11: now also IC1.4; no longer IC4.4
- net BTN_LED12: now also IC1.5; no longer IC4.5
- net BTN_LED2: now also IC2.3; no longer IC3.3
- net BTN_LED3: now also IC2.5; no longer IC3.5
- net BTN_LED4: now also IC2.7; no longer IC3.7
- net BTN_LED5: now also IC2.4; no longer IC3.4
- net BTN_LED6: now also IC1.3; no longer IC4.3
- net BTN_LED7: now also IC1.6; no longer IC4.6
- net BTN_LED8: now also IC1.7; no longer IC4.7
- net BTN_LED9: now also IC2.6; no longer IC3.6
- net BTN_UNUSED1: now also IC1.1; no longer IC4.1
- net BTN_UUSED2: now also IC1.15; no longer IC4.15
- net CAN_H: now also R11.1; no longer R27.1
- net CAN_L: now also R11.2; no longer R27.2
- net CAN_RX: now also R13.1; no longer R29.1
- net CAN_TX: now also R14.1; no longer R28.1
- net DIN_1: now also IC4.11, R2.1, ROTENC2.B; no longer R26.1, ROTENC1.A, U$87.11
- net DIN_2: now also IC4.12, R3.1, ROTENC1.A; no longer R25.1, ROTENC1.B, U$87.12
- net DIN_3: now also IC4.13, R4.1; no longer R24.1, U$87.13
- net DIN_4: now also IC4.14, R5.1; no longer R23.1, U$87.14
- net DIN_5: now also IC4.3, R6.1, ROTENC1.B; no longer R22.1, ROTENC2.B, U$87.3
- net DIN_6: now also IC4.4, R7.1; no longer R21.1, U$87.4
- net DIN_7: now also C20.2, IC4.5, R8.1; no longer C15.2, R20.1, U$87.5
- net DIN_8: now also C23.2, IC4.6, R9.1; no longer BTN4.SW3, C17.2, R19.1, U$87.6
- net GND: now also C10.2, C11.2, C12.1, C16.2, C19.2, C2.2, C23.1, C25.1, C3.1, C4.1, C6.1, C7.2, IC2.13, IC2.8, IC4.15, JP2.5, JP4.2, R19.2, R20.2, R21.2, R22.2, R23.2, R24.2, R25.2, R26.2, R27.2, R28.2, R29.2; no longer BTN2.SW1, BTN4.SW1, BTN6.SW1, C10.1, C11.1, C12.2, C16.1, C19.1, C2.1, C23.2, C25.2, C3.2, C4.2, C6.2, C7.1, IC4.13, JP2.2, R1.2, R11.2, R13.2, R14.2, R15.2, R16.2, R5.2, R6.2, R7.2, R8.2, R9.2, SWD.5, U$87.15, U$87.8
- net N$1: now also C6.2; no longer C2.2
- net N$10: now also R19.1; no longer R6.1
- net N$11: now also IC2.1; no longer IC3.1
- net N$12: now also IC1.14, IC2.9; no longer IC3.9, IC4.14
- net N$13: now also R13.2; no longer R29.2
- net N$2: now also C5.2; no longer C1.2
- net N$24: now also R20.1; no longer R7.1
- net N$25: now also R21.1; no longer R8.1
- net N$26: now also C21.2; no longer BTN2.SW3, C16.2
- net N$27: now also R14.2; no longer R28.2
- net N$28: now also IC4.10, R1.1; no longer R17.1, U$87.10
- net N$29: now also R24.1; no longer R9.1
- net N$3: now also C13.1; no longer C6.1
- net N$30: now also R25.1; no longer R10.1
- net N$31: now also IC2.2; no longer IC3.2
- net N$34: now also R26.1; no longer R11.1
- net N$35: now also R27.1; no longer R12.1
- net N$36: now also C24.2; no longer C18.2
- net N$39: now also R22.1; no longer R13.1
- net N$4: now also C7.1; no longer C4.1
- net N$40: now also R23.1; no longer R14.1
- net N$41: now also C22.2; no longer C19.2
- net N$44: now also R28.1; no longer R15.1
- net N$45: now also R29.1; no longer R16.1
- net N$46: now also C25.2; no longer BTN6.SW3, C20.2
- net N$49: now also IC3.15; no longer IC1.15
- net N$5: now also R17.1; no longer R4.1
- net N$50: now also IC3.1; no longer IC1.1
- net N$51: now also IC3.2; no longer IC1.2
- net N$52: now also IC3.3; no longer IC1.3
- net N$53: now also IC3.4; no longer IC1.4
- net N$54: now also IC3.5; no longer IC1.5
- net N$55: now also IC3.6; no longer IC1.6
- net N$56: now also IC3.7; no longer IC1.7
- net N$57: now also IC2.14, IC3.9; no longer IC1.9, IC3.14
- net N$6: now also R12.1; no longer R1.1
- net N$65: now also IC1.9; no longer IC4.9
- net N$7: now also R15.2; no longer R2.2
- net N$73: now also R10.1; no longer R18.1
- net N$8: now also R16.2; no longer R3.2
- net N$9: now also R18.1; no longer R5.1
- net NRST: now also B2.B, B2.B', C16.1, JP2.4; no longer B1.B, B1.B', C13.1, SWD.4
- net PB2: now also B1.B, B1.B'; no longer B2.B, B2.B'
- net SPI2_CLK: now also IC2.11, IC4.2; no longer IC4.11, U$87.2
- net SPI2_MISO: now also IC4.9; no longer U$87.9
- net SPI2_MOSI: now also IC3.14; no longer IC1.14
- net SPI2_RC1: now also IC2.12; no longer IC4.12
- net SPI2_RC2: now also IC4.1; no longer U$87.1
- net SWCK: now also JP2.2; no longer SWD.2
- net SWDIO: now also JP2.3; no longer SWD.3
- net USB_DM: now also R15.1; no longer R2.1
- net USB_DP: now also R16.1; no longer R3.1
Routing:
- net GND: track 0.00 -> 65.0 mm, vias 0 -> 2
- net DIN_7: track 0.00 -> 8.91 mm
- net N$41: track 0.00 -> 8.48 mm
- net N$36: track 0.00 -> 6.71 mm
- net N$44: track 0.00 -> 5.07 mm
- net N$24: track 0.00 -> 4.84 mm
- net N$29: track 0.00 -> 4.66 mm
- net N$34: track 0.00 -> 2.90 mm
- net N$9: track 0.00 -> 2.71 mm
- net N$10: track 0.00 -> 2.50 mm
- net N$39: track 0.00 -> 2.47 mm
- net SPI2_CLK: track 65.7 -> 68.1 mm
- net SPI2_RC1: track 67.6 -> 70.0 mm
- net N$26: track 0.00 -> 2.23 mm
- net N$40: track 0.00 -> 2.22 mm
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
Commit message: wip
Parts:
- moved R8 395.2 mm to (43.2, 190.5), flipped to the bottom, turned to 180 degrees
- moved R9 375.8 mm to (22.6, 180.3), flipped to the bottom
- moved C1 365.9 mm to (8.26, 186.7), flipped to the bottom, turned to 90 degrees
- moved R1 363.0 mm to (7.11, 180.3), flipped to the bottom
- moved D2 252.5 mm to (-14.7, 20.1)
- moved R11 252.5 mm to (-16.0, 6.10)
- moved R13 252.5 mm to (-16.0, -4.06)
- moved C10 252.5 mm to (-17.3, 15.0)
- moved R10 252.5 mm to (-16.0, 11.2)
- moved R14 252.5 mm to (-16.0, 1.02)
- moved H2 244.0 mm to (-11.0, 88.1)
- moved H4 216.7 mm to (-24.8, 75.3)
- moved C14 180.1 mm to (-4.95, 81.0), turned to 180 degrees
- moved C16 165.2 mm to (-4.95, 73.4), turned to 180 degrees
- moved B1 154.2 mm to (-7.49, 68.3), turned to 180 degrees
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Connections:
- removed net N$32: FADER1.P2
- removed net N$33: POT1.P2
- removed net N$37: POT5.P2
- removed net N$38: POT6.P2
- removed net N$42: POT2.P2
- removed net N$43: POT3.P2
- removed net N$47: POT7.P2
- removed net N$48: POT4.P2
- new net ADC0: CPU1.14, POT5.P2
- new net ADC1: CPU1.15, POT6.P2
- new net ADC2: CPU1.16, POT7.P2
- new net ADC3: CPU1.17, POT4.P2
- new net ADC4: CPU1.20, POT3.P2
- new net ADC5: CPU1.21, POT2.P2
- new net ADC6: CPU1.22, POT1.P2
- new net ADC7: CPU1.23, FADER1.P2
- new net DIN_TODO: BTN1.SW3, BTN1.SW4, C20.2
- new net DIN_TODO2: BTN4.SW4, C23.2
- net DIN_1: now also ROTENC2.A; no longer ROTENC2.B
- net DIN_2: now also ROTENC2.B; no longer ROTENC1.A
- net DIN_3: now also ROTENC2.S2; no longer ROTENC1.S2
- net DIN_4: no longer ROTENC2.A
- net DIN_5: now also ROTENC1.S2; no longer ROTENC1.B
- net DIN_6: now also ROTENC1.A; no longer ROTENC2.S2
- net DIN_7: now also ROTENC1.B; no longer BTN1.SW3, BTN1.SW4, C20.2
- net DIN_8: no longer BTN4.SW4, C23.2
Routing:
- net SPI2_RC2: track 0.00 -> 193.0 mm, vias 0 -> 1
- net SPI2_MISO: track 0.00 -> 183.9 mm, vias 0 -> 1
- net ADC3: track 0.00 -> 168.4 mm
- net ADC0: track 0.00 -> 163.1 mm
- net ADC4: track 0.00 -> 148.5 mm
- net ADC1: track 0.00 -> 127.8 mm
- net ADC5: track 0.00 -> 123.3 mm
- net SPI2_CLK: track 68.1 -> 187.8 mm
- net ADC2: track 0.00 -> 101.4 mm
- net ADC6: track 0.00 -> 79.2 mm
- net DIN_5: track 0.00 -> 39.6 mm
- net DIN_6: track 0.00 -> 25.2 mm
- net DIN_3: track 0.00 -> 23.6 mm
- net DIN_7: track 8.91 -> 32.3 mm
- net 3.3V: track 17.9 -> 39.9 mm, vias 5 -> 11
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
Commit message: wip
Parts:
- removed JP2: (no value), microbuilder:1X05_ROUND_76
- added JTAG: jtag, microbuilder:1X05_ROUND_76
- moved R13 42.2 mm to (25.1, 5.33)
- moved R14 41.6 mm to (25.1, 7.11)
- moved C10 39.4 mm to (20.1, 2.29), flipped to the bottom
- moved D2 37.6 mm to (20.1, 5.84), flipped to the bottom, turned to 270 degrees
- moved R10 34.1 mm to (18.0, 9.40), flipped to the bottom, turned to 180 degrees
- moved R11 31.0 mm to (15.0, 4.83), flipped to the bottom, turned to 270 degrees
- moved R12 2.97 mm to (34.5, 7.87), turned to 180 degrees
Connections:
- removed net LCS_CS: LCD1.P$5
- new net LCD_CS: CPU1.58, LCD1.P$5
- new net LCD_MISO_UNUSED: CPU1.56
- net 3.3V: now also JTAG.1; no longer JP2.1
- net GND: now also JTAG.5; no longer JP2.5
- net LCD_CLK: now also CPU1.55
- net LCD_DC: now also CPU1.59
- net LCD_MOSI: now also CPU1.57
- net NRST: now also JTAG.2; no longer JP2.4
- net SWCK: now also JTAG.3; no longer JP2.2
- net SWDIO: now also JTAG.4; no longer JP2.3
Routing:
- net LCD_CLK: track 0.00 -> 246.7 mm, vias 0 -> 2
- net LCD_MOSI: track 0.00 -> 246.0 mm, vias 0 -> 2
- net LCD_CS: track 0.00 -> 245.0 mm, vias 0 -> 2
- net LCD_DC: track 0.00 -> 243.4 mm, vias 0 -> 2
- net NRST: track 0.00 -> 14.8 mm, vias 0 -> 1
- net N$13: track 0.00 -> 14.4 mm
- net N$27: track 0.00 -> 13.5 mm
- net SWDIO: track 0.00 -> 12.4 mm, vias 0 -> 1
- net GND: track 74.9 -> 85.4 mm, vias 4 -> 6
- net SWCK: track 0.00 -> 8.85 mm, vias 0 -> 1
- net CAN_TX: track 0.00 -> 4.42 mm, vias 0 -> 1
- net CAN_RX: track 0.00 -> 3.56 mm, vias 0 -> 1
- net CAN_L: track 0.00 -> 2.75 mm
- net CAN_H: track 0.00 -> 2.65 mm
- net N$6: track 0.00 -> 1.92 mm
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
Commit message: wip
Parts:
- added JP2, JP5: (no value), microbuilder:1X04_ROUND
- moved C19 53.0 mm to (35.3, 18.5), flipped to the bottom, turned to 90 degrees
- moved R17 49.8 mm to (35.3, 31.8)
- moved C18 48.7 mm to (33.3, 19.1), flipped to the bottom, turned to 270 degrees
- moved LED1 48.0 mm to (38.9, 31.8), turned to 270 degrees
- moved L1 43.5 mm to (31.5, 18.5), flipped to the bottom, turned to 270 degrees
- moved C17 35.9 mm to (5.84, 11.7), flipped to the bottom, turned to 90 degrees
- moved C15 25.9 mm to (2.29, 17.5), flipped to the bottom, turned to 270 degrees
- moved U1 24.0 mm to (7.37, 19.1), flipped to the bottom, turned to 0 degrees
Connections:
- net 5.0V: now also JP2.1, JP5.1
- net CAN_H: now also JP2.2, JP5.2
- net CAN_L: now also JP2.3, JP5.3
- net GND: now also JP2.4, JP5.4
Routing:
- net 5.0V: track 0.00 -> 21.7 mm
- net CAN_L: track 2.75 -> 21.7 mm, vias 0 -> 2
- net CAN_H: track 2.65 -> 21.0 mm, vias 0 -> 2
- net GND: track 85.4 -> 99.3 mm, vias 6 -> 10
- net AVDD: track 0.00 -> 8.65 mm, vias 0 -> 1
- net N$5: track 0.00 -> 1.96 mm
- net 3.3V: track 39.9 -> 41.9 mm, vias 11 -> 12
- net LCD_CLK: track 246.7 -> 245.1 mm
- net LCD_MOSI: track 246.0 -> 244.5 mm
- net LCD_CS: track 245.0 -> 244.3 mm
